File: Boards/BITS/bits.brd (EAGLE design)
At the start: 41.4 x 43.5 mm, 25 parts, among them T1 Si1013, X1 22-23-2021, X2 53398-10, X3 22-23-2031, X4 22-23-2041

Commit message: Cleaned up the BITS schematic
Parts:
- removed U$1: MICROSD, adafruit:MICROSD
- added C11: 10 uF, resistor:C0603
- added C2: .1 uF, resistor:C0603
- added C3: 10 uF, resistor:C1210
- added C4: .18 uF, resistor:C0603
- added C5: 2.2 uF, resistor:C1210
- added D3: DO-214AC, HASP:DO-214AC
- added JP1: (no value), pinhead:1X02
- added L1: CDRH104R, library:CDRH104R
- added R17, R20, R21: 23.3k, resistor:R0603
- added R18: 75k, resistor:R0603
- added R19: 13.3k, resistor:R0603
- added U$4: MICRO_SD, NR_connectors:MICRO_SD_HINGED
- added U1: LMR16020, HASP:SO8
Connections:
- new net IN1: C3.1, C5.1, JP1.2, R21.2, U1.P$2
- new net N$29: R17.2, U1.P$4
- new net N$31: C2.2, U1.P$1
- new net N$32: C2.1, D3.P$2, L1.P$1, U1.P$8
- new net N$33: R18.1, R19.2, U1.P$5
- new net N$34: R20.2, R21.1, U1.P$3
- new net REG_OUT: C11.1, C4.1, L1.P$2, R18.2
- net +3V3: now also U$4.VDD, U$4.VSS; no longer U$1.4
- net GND: now also C11.2, C3.2, C4.2, C5.2, D3.P$1, JP1.1, R17.1, R19.1, R20.1, U$4.CD1, U$4.GND1, U$4.GND2, U$4.GND3, U$4.GND4, U1.P$7, U1.PAD; no longer U$1.6, U$1.MT1, U$1.MT2
- net MISO: now also U$4.DAT0; no longer U$1.7
- net MOSI: now also U$4.CMD; no longer U$1.3
- net SCK: now also U$4.CLK; no longer U$1.5
- net SD_CS: now also U$4.CD; no longer U$1.2
Routing:
- net +3V3: track 66.2 -> 7.12 mm, vias 1 -> 0
- net SCK: track 37.7 -> 36.1 mm
- net SD_CS: track 32.3 -> 31.8 mm
- net GND: vias 22 -> 31
Other:
- board size 41.4 x 43.5 mm -> 71.4 x 86.6 mm
- board text added: "10V"
- board text added: "5V"
- board text added: "GND"
- board text added: "HASP Input Regulator"
- board text added: "V. 2 5-2017"
- board text added: "Vin"
