File: Boards/BITS/bits.brd (EAGLE design)
At the start: 45 x 45 mm, 38 parts, among them T1 SI1013, U1 LMR16020, X1 22-23-2021, X2 53398-10, X3 22-23-2031, X4 22-23-2041

Commit message: Integrate the BITS XBee
Parts:
- removed X4: 22-23-2041, con-molex:22-23-2041
- added XB1: XBEE-PRO, maxstream:XBEE-PRO
Connections:
- net +3V3: now also XB1.1; no longer X4.3
- net DIN: now also XB1.3; no longer X4.1
- net DOUT: now also XB1.2; no longer X4.2
- net GND: now also XB1.10; no longer X4.4
Changed lines of the file:
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@@
 <attribute name="VALUE" x="-1.603375" y="39.497" size="1.016" layer="27" ratio="10" rot="R270"/>
-</element>
-<element name="X4" library="con-molex" package="22-23-2041" value="22-23-2041" x="11.509375" y="4.191" smashed="yes" rot="R180">
-<attribute name="MF" value="MOLEX" x="11.509375" y="4.191" size="1.778" layer="27" rot="R180" display="off"/>
-<attribute name="MPN" value="22-23-2041" x="11.509375" y="4.191" size="1.778" layer="27" rot="R180" display="off"/>
-<attribute name="NAME" x="16.589375" y="0.381" size="1.016" layer="25" ratio="10" rot="R180"/>
-<attribute name="OC_FARNELL" value="1462920" x="11.509375" y="4.191" size="1.778" layer="27" rot="R180" display="off"/>
-<attribute name="OC_NEWARK" value="38C0355" x="11.509375" y="4.191" size="1.778" layer="27" rot="R180" display="off"/>
-<attribute name="VALUE" x="16.589375" y="9.271" size="1.016" layer="27" ratio="10" rot="R180"/>
 </element>
 <element name="U$7" library="ubloxLib" package="MAX-M8" value="MAX-M8" x="34.464625" y="34.401125" smashed="yes" rot="R180"/>
@@
 </element>
 <element name="T1" library="cmdLibs" package="SC-75" value="SI1013" x="26.876375" y="32.35325" smashed="yes" rot="R90"/>
+<element name="XB1" library="maxstream" library_urn="urn:adsk.eagle:library:270" package="XBEE-PRO" package3d_urn="urn:adsk.eagle:package:18008/1" value="XBEE-PRO" x="-64" y="19" smashed="yes">
+<attribute name="MF" value="" x="-64" y="19" size="1.778" layer="27" display="off"/>
+<attribute name="MPN" value="XBP24-AWI-001" x="-64" y="19" size="1.778" layer="27" display="off"/>
+<attribute name="NAME" x="-75.43" y="32.97" size="1.27" layer="25"/>
+<attribute name="OC_FARNELL" value="1337916" x="-64" y="19" size="1.778" layer="27" display="off"/>
+<attribute name="OC_NEWARK" value="42M2667" x="-64" y="19" size="1.778" layer="27" display="off"/>
+<attribute name="VALUE" x="-75.43" y="-0.3" size="1.27" layer="27"/>
+</element>
 </elements>
 <signals>
@@
 <contactref element="X1" pad="1"/>
 <contactref element="X3" pad="3"/>
-<contactref element="X4" pad="4"/>
 <contactref element="U$7" pad="10_GND"/>
 <contactref element="C1" pad="GND"/>
@@
 <contactref element="JP1" pad="1"/>
 <contactref element="R20" pad="1"/>
+<contactref element="XB1" pad="10"/>
+<wire x1="39.014625" y1="30.101125" x2="39.014625" y2="32.251125" width="0" layer="19" extent="1-1"/>
+<wire x1="39.624" y1="28.194" x2="39.014625" y2="30.101125" width="0" layer="19" extent="1-1"/>
+<wire x1="29.514625" y1="38.801125" x2="39.014625" y2="32.251125" width="0" layer="19" extent="1-1"/>
+<wire x1="18.122" y1="41.402" x2="29.514625" y2="38.801125" width="0" layer="19" extent="1-1"/>
+<wire x1="16.676" y1="34.417" x2="18.122" y2="41.402" width="0" layer="19" extent="1-1"/>
+<wire x1="14.31925" y1="24.783875" x2="16.676" y2="34.417" width="0" layer="19" extent="1-1"/>
+<wire x1="10.50925" y1="24.86325" x2="14.31925" y2="24.783875" width="0" layer="19" extent="1-1"/>
+<wire x1="18.1737" y1="24.336375" x2="14.31925" y2="24.783875" width="0" layer="19" extent="1-1"/>
+<wire x1="9.15125" y1="19.097625" x2="10.50925" y2="24.86325" width="0" layer="19" extent="1-1"/>
+<wire x1="19.337375" y1="17.429875" x2="18.1737" y2="24.336375" width="0" layer="19" extent="1-1"/>
+<wire x1="16.462375" y1="16.779875" x2="19.337375" y2="17.429875" width="0" layer="19" extent="1-1"/>
+<wire x1="16.247375" y1="12.112625" x2="16.462375" y2="16.779875" width="0" layer="19" extent="1-1"/>
+<wire x1="14.97875" y1="10.2235" x2="16.247375" y2="12.112625" width="0" layer="19" extent="1-1"/>
+<wire x1="18.533375" y1="9.652" x2="16.247375" y2="12.112625" width="0" layer="19" extent="1-1"/>
+<wire x1="22.455875" y1="13.001625" x2="18.533375" y2="9.652" width="0" layer="19" extent="1-1"/>
+<wire x1="28.482125" y1="15.698875" x2="22.455875" y2="13.001625" width="0" layer="19" extent="1-1"/>
+<wire x1="33.382125" y1="15.698875" x2="28.482125" y2="15.698875" width="0" layer="19" extent="1-1"/>
+<wire x1="36.432125" y1="15.798875" x2="33.382125" y2="15.698875" width="0" layer="19" extent="1-1"/>
+<wire x1="39.892375" y1="16.454625" x2="36.432125" y2="15.798875" width="0" layer="19" extent="1-1"/>
+<wire x1="32.131" y1="7.239" x2="33.382125" y2="15.698875" width="0" layer="19" extent="1-16"/>
 <wire x1="38.332125" y1="3.498875" x2="32.131" y2="7.239" width="0" layer="19" extent="1-16"/>
+<wire x1="24.982125" y1="3.498875" x2="32.131" y2="7.239" width="0" layer="19" extent="1-16"/>
+<wire x1="3.556" y1="30.0355" x2="10.50925" y2="24.86325" width="0" layer="19" extent="1-1"/>
+<wire x1="3.476625" y1="33.147" x2="3.556" y2="30.0355" width="0" layer="19" extent="1-1"/>
+<wire x1="6.604" y1="35.814" x2="3.476625" y2="33.147" width="0" layer="19" extent="1-1"/>
+<wire x1="8.14" y1="39.878" x2="6.604" y2="35.814" width="0" layer="19" extent="1-1"/>
+<wire x1="8.14" y1="41.91" x2="8.14" y2="39.878" width="0" layer="19" extent="1-1"/>
+<wire x1="6.02425" y1="9.869" x2="14.97875" y2="10.2235" width="0" layer="19" extent="1-1"/>
+<wire x1="-49.006125" y1="17.526" x2="3.556" y2="30.0355" width="0" layer="19" extent="1-1"/>
+<wire x1="-75" y1="10" x2="-49.006125" y2="17.526" width="0" layer="19" extent="1-1"/>
 </signal>
 <signal name="+3V3">
-<contactref element="X4" pad="3"/>
 <contactref element="X2" pad="9"/>
 <contactref element="L1" pad="P$2"/>
@@
 <contactref element="U$4" pad="VDD"/>
 <contactref element="D1" pad="A"/>
+<contactref element="XB1" pad="1"/>
 <wire x1="26.625375" y1="33.53325" x2="34.544" y2="43.434" width="0" layer="19" extent="1-1"/>
 <wire x1="34.401125" y1="21.574125" x2="26.625375" y2="33.53325" width="0" layer="19" extent="1-1"/>
@@
 <wire x1="13.27875" y1="10.2235" x2="20.755875" y2="13.001625" width="0" layer="19" extent="1-1"/>
 <wire x1="11.48625" y1="16.5735" x2="13.27875" y2="10.2235" width="0" layer="19" extent="1-1"/>
-<wire x1="10.239375" y1="4.191" x2="13.27875" y2="10.2235" width="0" layer="19" extent="1-1"/>
 <wire x1="6.02425" y1="11.119" x2="13.27875" y2="10.2235" width="0" layer="19" extent="1-1"/>
 <wire x1="29.282125" y1="2.998875" x2="20.755875" y2="13.001625" width="0" layer="19" extent="1-1"/>
@@
 <wire x1="7.936" y1="32.766" x2="11.48625" y2="16.5735" width="0" layer="19" extent="1-1"/>
 <wire x1="6.604" y1="33.274" x2="7.936" y2="32.766" width="0" layer="19" extent="1-1"/>
+<wire x1="-75" y1="28" x2="6.604" y2="33.274" width="0" layer="19" extent="1-1"/>
 </signal>
 <signal name="MOSI">
@@
 <signal name="DOUT">
 <contactref element="U$2" pad="9"/>
-<contactref element="X4" pad="2"/>
-<wire x1="12.779375" y1="4.191" x2="14.224" y2="28.194" width="0" layer="19" extent="1-1"/>
+<contactref element="XB1" pad="2"/>
+<wire x1="14.224" y1="28.194" x2="-75" y2="26" width="0" layer="19" extent="1-1"/>
 </signal>
 <signal name="DIN">
 <contactref element="U$2" pad="10"/>
-<contactref element="X4" pad="1"/>
-<wire x1="15.319375" y1="4.191" x2="11.684" y2="28.194" width="0" layer="19" extent="1-1"/>
+<contactref element="XB1" pad="3"/>
+<wire x1="11.684" y1="28.194" x2="-75" y2="24" width="0" layer="19" extent="1-1"/>
 </signal>
 <signal name="AGND">
@@
 </board>
 </drawing>
+<compatibility>
+<note version="8.2" severity="warning">
+Since Version 8.2, EAGLE supports online libraries. The ids
+of those online libraries will not be understood (or retained)
+with this version.
+</note>
+<note version="8.3" severity="warning">
+Since Version 8.3, EAGLE supports URNs for individual library
+assets (packages, symbols, and devices). The URNs of those assets
+will not be understood (or retained) with this version.
+</note>
+<note version="8.3" severity="warning">
+Since Version 8.3, EAGLE supports the association of 3D packages
+with devices in libraries, schematics, and board files. Those 3D
+packages will not be understood (or retained) with this version.
+</note>
+</compatibility>
 </eagle>
