File: Boards/BITS/bitsClassic.brd (EAGLE design)
At the start: 45 x 45 mm, 38 parts, among them T1 SI1013, U1 LMR16020, X1 22-23-2021, X2 53398-10, X3 22-23-2031

Commit message: routed bits board
Parts:
- removed JP1: (no value), pinhead:1X02
- removed R4: 18k, resistor:R0603
- removed R5: 10k, resistor:R0603
- removed X1: 22-23-2021, con-molex:22-23-2021
- removed X3: 22-23-2031, con-molex:22-23-2031
- added U$1: MOLEX_NANOFIT_2, cmdLibs:MOLEX_NANOFIT_2
- L1: value CDRH104R -> ASPI-6045S-560M-TCT-ND; device library:CDRH104R -> inductors:ABRACON
- R18: value 75k -> 45k
- R20: value 23.3k -> 31.6k
- R21: value 23.3k -> 190k
- moved XB1 96.4 mm to (32.4, 21.9)
- moved U$8 34.7 mm to (30.0, 2.40), turned to 0 degrees
- moved LED2 30.2 mm to (29.1, 17.4), turned to 270 degrees
- moved LED1 30.1 mm to (29.1, 19.6), turned to 270 degrees
- moved C4 28.4 mm to (19.7, 38.1)
- moved R10 26.2 mm to (26.1, 17.4), turned to 0 degrees
- moved R9 26.1 mm to (26.1, 19.6), turned to 0 degrees
- moved D1 24.9 mm to (33.2, 28.4), turned to 270 degrees
- moved U$7 24.8 mm to (29.9, 10.1), turned to 90 degrees
- moved C11 22.9 mm to (19.6, 35.8)
- moved R19 21.1 mm to (15.7, 30.4), turned to 90 degrees
- moved L1 21.0 mm to (14.9, 36.3), turned to 270 degrees
- moved R3 20.1 mm to (36.1, 34.3), turned to 0 degrees
- moved U$3 20.0 mm to (12.2, 7.96)
- moved R1 18.9 mm to (36.1, 32.1), turned to 0 degrees
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Connections:
- net N$32 renamed SW
- net N$33 renamed FB
- removed net BAT_CELL2: R4.1, R5.1, U$2.15/A1
- removed net CELL1: R1.1, X3.1
- removed net CELL2: R4.2, X3.2
- new net A: U$2.16/A2
- new net K: U$2.19/A5
- new net N$10: U$2.A11
- new net N$12: U$2.20/A6
- new net N$13: U$2.21/A7
- new net N$35: U$2.22/A8
- new net N$36: U$2.23/A9
- new net N$37: U$2.A10
- new net N$7: U$2.17/A3
- new net N$8: U$2.18/A4
- net +5V: no longer X1.2
- net BAT_CELL1: now also U$2.15/A1; no longer U$2.14/A0
- net DIN: now also U$2.1; no longer U$2.10
- net DOUT: now also U$2.0; no longer U$2.9
- net GND: now also U$1.P$2; no longer JP1.1, R5.2, X1.1, X3.3
- net GPSON: now also U$2.5; no longer U$2.6
- net IN1: now also R1.1, U$1.P$1; no longer JP1.2
- net LED2: now also U$2.3; no longer U$2.5
- net RING: now also U$2.14/A0; no longer U$2.16/A2
- net RXD: now also U$2.9; no longer U$2.0
- net SD_CS: now also U$2.2; no longer U$2.3
- net SLEEP: now also U$2.6; no longer U$2.2
- net TXD: now also U$2.10; no longer U$2.1
Routing:
- net +3V3: track 0.00 -> 103.9 mm, vias 0 -> 5
- net IN1: track 0.00 -> 95.4 mm, vias 0 -> 3
- net MOSI: track 0.00 -> 82.3 mm
- net SCK: track 0.00 -> 71.0 mm
- net RING: track 0.00 -> 63.2 mm
- net MISO: track 0.00 -> 59.1 mm
- net VBAT: track 0.00 -> 58.7 mm
- net V_BCKP: track 0.00 -> 42.3 mm
- net TXD: track 0.00 -> 39.2 mm
- net N$11: track 1.10 -> 39.2 mm
- net SLEEP: track 0.00 -> 36.6 mm
- net RXD: track 0.00 -> 33.1 mm
- net N$3: track 0.00 -> 25.2 mm
- net DOUT: track 0.00 -> 23.2 mm
- net DIN: track 0.00 -> 19.9 mm
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- added copper zone on layer 1, net +3V3
- added copper zone on layer 1, net FB
- added copper zone on layer 1, net GND
- added copper zone on layer 16, net GND
- added copper zone on layer 1, net IN1
- added copper zone on layer 1, net SW
Other:
- board size 45 x 45 mm -> 45 x 40 mm
- board text added: "BITS V3"
- board text added: "GND"
- board text added: "Vin"
