File: Boards/BITS/bitsClassic.sch (EAGLE design)
At the start: 38 parts, among them T1 SI1013, U1 LMR16020, X1 22-23-2021, X2 53398-10, X3 22-23-2031

Commit message: routed bits board
Parts:
- removed JP1: (no value), pinhead:PINHD-1X2
- removed R4: 18k, resistor:R-US_R0603
- removed R5: 10k, resistor:R-US_R0603
- removed X1: 22-23-2021, con-molex:22-23-2021
- removed X3: 22-23-2031, con-molex:22-23-2031
- added U$1: MOLEX_NANOFIT_2, cmdLibs:MOLEX_NANOFIT_2
- L1: value CDRH104R -> ASPI-6045S-560M-TCT-ND; device library:CDRH104R -> inductors:ASPI-6045S-560M-TCT-ND
- R18: value 75k -> 45k
- R20: value 23.3k -> 31.6k
- R21: value 23.3k -> 190k
Connections:
- net N$32 renamed SW
- net N$33 renamed FB
- removed net BAT_CELL2: R4.1, R5.1, U$2.15/A1/T
- removed net CELL1: R1.1, X3-1.S
- removed net CELL2: R4.2, X3-2.S
- new net A: U$2.16/A2/T
- new net K: U$2.19/A5/T/SCL0
- new net N$10: U$2.A11
- new net N$12: U$2.20/A6/PWM
- new net N$13: U$2.21/A7/PWM
- new net N$35: U$2.22/A8/T/PWM
- new net N$36: U$2.23/A9/T/PWM
- new net N$37: U$2.A10
- new net N$7: U$2.17/A3/T
- new net N$8: U$2.18/A4/T/SDA0
- net +5V: no longer X1-2.S
- net BAT_CELL1: now also U$2.15/A1/T; no longer U$2.14/A0
- net DIN: now also U$2.1/TX1/T; no longer U$2.10/TX2/PWM
- net DOUT: now also U$2.0/RX1/T; no longer U$2.9/RX2/PWM
- net GND: now also U$1.P2; no longer JP1.1, R5.2, X1-1.S, X3-3.S
- net GPSON: now also U$2.5/PWM; no longer U$2.6/PWM
- net IN1: now also R1.1, U$1.P1; no longer JP1.2
- net LED2: now also U$2.3/CAN-TX/PWM; no longer U$2.5/PWM
- net RING: now also U$2.14/A0; no longer U$2.16/A2/T
- net RXD: now also U$2.9/RX2/PWM; no longer U$2.0/RX1/T
- net SD_CS: now also U$2.2; no longer U$2.3/CAN-TX/PWM
- net SLEEP: now also U$2.6/PWM; no longer U$2.2
- net TXD: now also U$2.10/TX2/PWM; no longer U$2.1/TX1/T
Other:
- note added: "Voltage Moniter"
- note added: "XBEE"
- note removed: "Battery Voltage"
- note removed: "Cell Dividers"
- note removed: "Headers"
- note removed: "Power"
- moved on the sheet: LED1, LED2, R1, R10, R3, R9, X2-1, X2-10, X2-2, X2-3, X2-4, X2-5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
