File: Boards/BITS/bitsClassicEdit.brd (EAGLE design)
At the start: 45 x 40 mm, 34 parts, among them T1 SI1013, U1 LMR16020, X2 53398-10

Commit message: Created an alternate board
Parts:
- moved R3 36.8 mm to (12.9, 5.78), turned to 90 degrees
- moved R1 36.7 mm to (10.0, 6.26)
- moved U$3 24.5 mm to (9.33, 32.3), turned to 270 degrees
- moved U$4 15.1 mm to (9.92, 29.1), turned to 180 degrees
- moved U$1 14.9 mm to (10.3, 2.04), turned to 180 degrees
- moved C4 14.4 mm to (11.2, 26.4)
- moved D3 14.4 mm to (1.65, 24.6)
- moved R18 14.4 mm to (9.38, 18.7)
- moved C5 14.4 mm to (5.14, 8.12)
- moved C11 14.4 mm to (11.1, 24.2)
- moved C2 14.4 mm to (1.42, 11.4)
- moved C3 14.4 mm to (7.33, 11.2)
- moved L1 14.4 mm to (6.42, 24.6)
- moved R17 14.4 mm to (7.95, 16.0)
- moved R19 14.4 mm to (7.20, 18.7)
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Connections:
- removed net N$37: U$2.A10
- net BAT_CELL1: now also U$2.A10; no longer U$2.15/A1
Routing:
- net +3V3: track 103.9 -> 39.2 mm, vias 5 -> 2
- net MOSI: track 82.3 -> 18.6 mm
- net IN1: track 84.2 -> 20.9 mm, vias 2 -> 0
- net RING: track 63.2 -> 0.00 mm
- net SCK: track 71.0 -> 26.4 mm, vias 0 -> 1
- net V_BCKP: track 42.3 -> 0.00 mm
- net MISO: track 59.1 -> 18.1 mm
- net VBAT: track 58.7 -> 18.1 mm
- net TXD: track 39.2 -> 0.00 mm
- net SLEEP: track 36.6 -> 0.00 mm
- net RXD: track 33.1 -> 0.00 mm
- net N$11: track 39.2 -> 10.8 mm
- net BAT_CELL1: track 4.20 -> 30.8 mm, vias 0 -> 1
- net N$3: track 25.2 -> 1.99 mm
- net DOUT: track 23.2 -> 0.00 mm
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Other:
- board size 45 x 40 mm -> 45 x 45 mm

Commit message: bits board try 2
Parts:
- moved R19 9.98 mm to (12.5, 10.2)
- moved R17 9.93 mm to (13.0, 7.48)
- moved R20 9.10 mm to (10.5, 5.18)
- moved U1 8.60 mm to (8.59, 10.4)
- moved R7 7.84 mm to (34.6, 27.4), turned to 180 degrees
- moved D1 7.41 mm to (36.3, 25.6)
- moved D3 7.39 mm to (1.65, 17.2)
- moved R21 7.20 mm to (7.30, 5.16), turned to 180 degrees
- moved C11 7.04 mm to (11.5, 17.1)
- moved C4 6.89 mm to (11.4, 19.5)
- moved L1 6.60 mm to (6.31, 18.0)
- moved R2 6.52 mm to (29.3, 22.3)
- moved R18 5.25 mm to (12.0, 14.2)
- moved C1 4.60 mm to (34.4, 31.6), turned to 0 degrees
- moved C3 4.41 mm to (2.98, 10.4), turned to 180 degrees
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Connections:
- removed net N$35: U$2.22/A8
- removed net N$36: U$2.23/A9
- new net C: U$2.A10
- new net X: U$2.14/A0
- net BAT_CELL1: now also U$2.22/A8; no longer U$2.A10
- net DIN: now also U$2.10; no longer U$2.1
- net DOUT: now also U$2.9; no longer U$2.0
- net GPSON: now also U$2.4; no longer U$2.5
- net LED1: now also U$2.3; no longer U$2.4
- net LED2: now also U$2.2; no longer U$2.3
- net RING: now also U$2.23/A9; no longer U$2.14/A0
- net RXD: now also U$2.0; no longer U$2.9
- net SD_CS: now also U$2.6; no longer U$2.2
- net SLEEP: now also U$2.5; no longer U$2.6
- net TXD: now also U$2.1; no longer U$2.10
Routing:
- net +3V3: track 39.2 -> 106.0 mm, vias 2 -> 0
- net V_BCKP: track 0.00 -> 41.3 mm
- net RING: track 0.00 -> 35.9 mm
- net SD_CS: track 0.00 -> 27.2 mm
- net VBAT: track 18.1 -> 39.6 mm
- net IN1: track 20.9 -> 0.00 mm
- net N$9: track 1.83 -> 22.0 mm
- net N$3: track 1.99 -> 18.6 mm
- net TXD: track 0.00 -> 12.5 mm
- net RXD: track 0.00 -> 10.9 mm
- net SLEEP: track 0.00 -> 10.3 mm
- net RX3: track 17.2 -> 7.17 mm
- net N$11: track 10.8 -> 19.5 mm
- net MISO: track 18.1 -> 9.62 mm
- net BAT_CELL1: track 30.8 -> 39.1 mm, vias 1 -> 0
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- removed copper zone on layer 1, net FB

Commit message: All of the changes with CAD and electronics since switching to the microclasp connectors
Parts:
- added R4: (no value), resistor:R0603
- added U$5: (no value), NR_connectors:MICROCLASP
- U$1: value MOLEX_NANOFIT_2 -> (none); device cmdLibs:MOLEX_NANOFIT_2 -> NR_connectors:MICROCLASP
- moved C11 9.80 mm to (11.3, 26.9), turned to 90 degrees
- moved U$3 8.08 mm to (12.6, 38.1), turned to 0 degrees
- moved C4 7.73 mm to (13.5, 27.0), turned to 90 degrees
- moved R1 6.07 mm to (19.7, 4.00), turned to 90 degrees
- moved L1 5.80 mm to (10.6, 22.0), turned to 180 degrees
- moved U1 4.17 mm to (8.62, 14.6)
- moved R19 3.64 mm to (12.7, 13.9)
- moved R17 3.46 mm to (13.8, 10.9)
- moved R20 3.33 mm to (10.6, 8.50)
- moved R21 3.33 mm to (7.32, 8.49)
- moved R18 2.99 mm to (12.7, 17.1)
- moved R3 2.67 mm to (13.8, 8.52)
- moved D3 1.87 mm to (3.40, 17.9), turned to 0 degrees
- moved C2 1.64 mm to (4.00, 14.9)
- moved C3 1.40 mm to (3.09, 11.8)
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Connections:
- removed net X: U$2.14/A0
- new net N$32: R4.1, U$5.P$1
- new net SWITCH_LED: R4.2, U$2.14/A0
- net GND: now also U$5.P$2
Routing:
- net N$32: track 0.00 -> 56.6 mm, vias 0 -> 2
- net VBAT: track 39.6 -> 25.2 mm
- net +3V3: track 106.0 -> 99.8 mm
- net SW: track 0.00 -> 3.74 mm
- net BAT_CELL1: track 39.1 -> 42.6 mm
- net N$31: track 6.56 -> 3.96 mm
- net SWITCH_LED: track 0.00 -> 2.50 mm
- net GND: track 2.52 -> 4.70 mm, vias 34 -> 31
- net N$34: track 3.86 -> 4.96 mm
- net N$29: track 1.70 -> 2.76 mm
- net RING: track 35.9 -> 35.4 mm
- net TXD: track 12.5 -> 12.0 mm
- net RXD: track 10.9 -> 10.4 mm
- net SLEEP: track 10.3 -> 9.79 mm

Commit message: fixes and design review slides
Parts:
- removed R4: (no value), resistor:R0603
- removed U$5: (no value), NR_connectors:MICROCLASP
- added R5: (no value), resistor:R0603
- R20: value 31.6k -> 39k
- R21: value 190k -> 195k
- U$1: value (none) -> MICROCLASP_4; device NR_connectors:MICROCLASP -> NR_connectors:4_PIN_MICROCLASP
- moved U$1 1.25 mm to (11.9, 3.43)
Connections:
- removed net N$32: R4.1, U$5.P$1
- new net N$33: R5.2, U$1.P$2
- net GND: now also U$1.P$3, U$1.P$4; no longer U$1.P$2, U$5.P$2
- net SWITCH_LED: now also R5.1; no longer R4.2
Routing:
- net N$32: track 56.6 -> 0.00 mm, vias 2 -> 0

Commit message: Updated boards
Parts:
- moved R5 34.4 mm to (20.1, 6.40), turned to 270 degrees
- moved R1 7.55 mm to (13.7, 8.62), turned to 0 degrees
- moved R3 3.45 mm to (17.2, 8.16)
- moved X2 0.23 mm to (17.2, 18.7)
Connections:
- removed net N$13: U$2.21/A7
- new net E: U$2.14/A0
- net SWITCH_LED: now also U$2.21/A7; no longer U$2.14/A0
Routing:
- net SWITCH_LED: track 2.48 -> 34.7 mm
- net N$33: track 0.00 -> 6.01 mm
- net IN1: track 0.00 -> 5.22 mm
- net BAT_CELL1: track 42.6 -> 38.9 mm
- net GND: track 4.70 -> 4.98 mm, vias 31 -> 32
Other:
- board text added: "BITS V3.1"
- board text removed: "BITS V3"
