File: Boards/Cell_Tracker/cell.sch (EAGLE design)
At the start: 32 parts, among them IC1 NCV78M05BDTRKG, T1 Si1013, U2 LMR16020

Commit message: Cell tracker V3 routed
Parts:
- removed C1: (no value), jmolterLib:DCK-3R3E204T614-E
- removed C2: 0.33uF, rcl:C-USC0603
- removed D1: (no value), diode:DIODE-SOD523
- removed IC1: NCV78M05BDTRKG, linear:NCV78M05BDTRKG
- removed R7: 22, rcl:R-US_R0603
- removed U$2: MICROSD, adafruit:MICROSD
- added U$3: MICRO_SD, NR_connectors:MICRO_SD
Connections:
- net N$14 renamed SW
- net N$15 renamed FB
- net N$16 renamed EN
- removed net +5V: IC1.VO, U$1.VIN
- removed net N$12: COIN.+, U$1.VBAT
- removed net N$13: C1.3V3, R7.2
- net +3V3: now also U$3.VDD, U$3.VSS; no longer D1.A, U$2.VDD
- net GND: now also U$3.CD1, U$3.G1, U$3.G2, U$3.G3, U$3.G4; no longer C1.GND, C2.2, IC1.GND, U$2.GND, U$2.GND1, U$2.VSS
- net MISO: now also U$3.DAT0; no longer U$2.DATA_OUT
- net MOSI: now also U$3.CMD; no longer U$2.DATA_IN
- net N$6: now also U$1.VIN; no longer C2.1, IC1.VI
- net SCK: now also U$3.CLK; no longer U$2.SCLK
- net SD_CS: now also U$3.CD; no longer U$2.CS
- net V_BCKP: now also COIN.+, U$1.VBAT; no longer D1.C, R7.1
Other:
- note removed: "Cell Tracker LTE-M"

Commit message: cleaned up cell schematic
Other:
- note added: "3V3 Regulator"
- note removed: "Regulator and LVC"
- moved on the sheet: C10, C6, C7, C8, C9, COIN, D2, JP3, L1, R1, R10, R11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
