File: Boards/Cell_Tracker/cell.brd (EAGLE design)
At the start: 43.2 x 41.9 mm, 28 parts, among them U2 LMR16020

Commit message: fixes and design review slides
Parts:
- removed R7: (no value), resistor:R0603
- removed U$5: (no value), NR_connectors:MICROCLASP
- added R8: (no value), resistor:R0603
- R10: value 190k -> 195k
- R9: value 31.6k -> 39k
- U$4: value (none) -> MICROCLASP_4; device NR_connectors:MICROCLASP -> NR_connectors:4_PIN_MICROCLASP
- moved U$4 6.59 mm to (39.8, 15.6), turned to 90 degrees
Connections:
- removed net N$12: R7.1, U$5.P$1
- new net N$13: R8.2, U$4.P$2
- net GND: now also U$4.P$3, U$4.P$4; no longer U$4.P$2, U$5.P$2
- net SWITCH_LED: now also R8.1; no longer R7.2
Routing:
- net N$12: track 5.04 -> 0.00 mm
- net SWITCH_LED: track 13.8 -> 12.9 mm
Changed lines of the file:
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@@
 <attribute name="VALUE" x="21.415375" y="1.349375" size="1.27" layer="27"/>
 </element>
-<element name="R9" library="resistor" package="R0603" value="31.6k" x="35.163125" y="10.795" smashed="yes" rot="R270">
+<element name="R9" library="resistor" package="R0603" value="39k" x="35.163125" y="10.795" smashed="yes" rot="R270">
 <attribute name="NAME" x="35.798125" y="11.43" size="1.27" layer="25" rot="R270"/>
 <attribute name="VALUE" x="33.258125" y="11.43" size="1.27" layer="27" rot="R270"/>
 </element>
-<element name="R10" library="resistor" package="R0603" value="190k" x="35.163125" y="7.699375" smashed="yes" rot="R270">
+<element name="R10" library="resistor" package="R0603" value="195k" x="35.163125" y="7.699375" smashed="yes" rot="R270">
 <attribute name="NAME" x="35.798125" y="8.334375" size="1.27" layer="25" rot="R270"/>
 <attribute name="VALUE" x="33.258125" y="8.334375" size="1.27" layer="27" rot="R270"/>
@@
 <attribute name="VALUE" x="22.098" y="24.638" size="0.254" layer="27"/>
 </element>
-<element name="U$4" library="NR_connectors" package="MICROCLASP" value="" x="39.766875" y="9.04875" rot="R270"/>
-<element name="U$5" library="NR_connectors" package="MICROCLASP" value="" x="39.766875" y="17.30375" rot="R270"/>
-<element name="R7" library="resistor" package="R0603" value="" x="34.29" y="17.30375" rot="R180"/>
+<element name="U$4" library="NR_connectors" package="4_PIN_MICROCLASP" value="MICROCLASP_4" x="39.766875" y="15.636875" rot="R90"/>
+<element name="R8" library="resistor" package="R0603" value="" x="32.940625" y="17.065625"/>
 </elements>
 <signals>
@@
 <vertex x="-2.54" y="44.45"/>
 <vertex x="36.03625" y="44.45"/>
-<vertex x="36.115625" y="21.59"/>
-<vertex x="45.799375" y="21.59"/>
+<vertex x="36.115625" y="18.335625"/>
+<vertex x="45.799375" y="18.335625"/>
 <vertex x="45.72" y="-2.54"/>
 <vertex x="-2.54" y="-2.54"/>
@@
 <vertex x="-1.27" y="43.18"/>
 <vertex x="36.03625" y="43.18"/>
-<vertex x="36.35375" y="21.59"/>
-<vertex x="44.7675" y="21.59"/>
+<vertex x="36.274375" y="18.335625"/>
+<vertex x="44.688125" y="18.335625"/>
 <vertex x="44.45" y="-1.27"/>
 <vertex x="-1.27" y="-1.27"/>
@@
 <wire x1="29.272625" y1="8.90675" x2="29.5275" y2="8.651875" width="0.3048" layer="1"/>
 <via x="30.559375" y="9.445625" extent="1-16" drill="0.254"/>
-<contactref element="U$4" pad="P$2"/>
-<contactref element="U$5" pad="P$2"/>
 <via x="6.111875" y="4.7625" extent="1-16" drill="0.5"/>
 <via x="11.1125" y="11.509375" extent="1-16" drill="0.5"/>
 <via x="19.52625" y="15.160625" extent="1-16" drill="0.5"/>
 <via x="32.7025" y="14.76375" extent="1-16" drill="0.5"/>
-<via x="39.131875" y="12.144375" extent="1-16" drill="0.5"/>
+<via x="37.7825" y="14.366875" extent="1-16" drill="0.5"/>
 <via x="32.305625" y="23.256875" extent="1-16" drill="0.5"/>
 <via x="5.715" y="16.03375" extent="1-16" drill="0.5"/>
 <via x="31.4325" y="3.254375" extent="1-16" drill="0.4064"/>
+<contactref element="U$4" pad="P$3"/>
+<contactref element="U$4" pad="P$4"/>
+<wire x1="25.04175" y1="31.60275" x2="28.971875" y2="38.179375" width="0" layer="19" extent="1-1"/>
+<wire x1="28.41625" y1="29.5275" x2="25.04175" y2="31.60275" width="0" layer="19" extent="1-1"/>
+<wire x1="29.05125" y1="24.209375" x2="28.41625" y2="29.5275" width="0" layer="19" extent="1-1"/>
+<wire x1="32.305625" y1="23.256875" x2="29.05125" y2="24.209375" width="0" layer="19" extent="1-1"/>
+<wire x1="34.54175" y1="22.90275" x2="32.305625" y2="23.256875" width="0" layer="19" extent="1-1"/>
+<wire x1="34.54175" y1="25.05275" x2="34.54175" y2="22.90275" width="0" layer="19" extent="1-1"/>
+<wire x1="34.829625" y1="20.06625" x2="34.54175" y2="22.90275" width="0" layer="19" extent="1-1"/>
+<wire x1="35.131375" y1="14.7565" x2="34.829625" y2="20.06625" width="0" layer="19" extent="1-1"/>
+<wire x1="32.7025" y1="14.76375" x2="35.131375" y2="14.7565" width="0" layer="19" extent="1-1"/>
+<wire x1="30.8855" y1="13.446125" x2="32.7025" y2="14.76375" width="0" layer="19" extent="1-1"/>
+<wire x1="35.163125" y1="11.645" x2="35.131375" y2="14.7565" width="0" layer="19" extent="1-1"/>
+<wire x1="30.559375" y1="10.239375" x2="30.8855" y2="13.446125" width="0" layer="19" extent="1-1"/>
+<wire x1="30.559375" y1="9.445625" x2="30.559375" y2="10.239375" width="0" layer="19" extent="1-1"/>
+<wire x1="30.00375" y1="9.55675" x2="30.559375" y2="9.445625" width="0" layer="19" extent="1-1"/>
+<wire x1="29.5275" y1="9.445625" x2="30.00375" y2="9.55675" width="0" layer="19" extent="1-1"/>
+<wire x1="29.272625" y1="8.90675" x2="29.5275" y2="9.445625" width="0" layer="19" extent="1-1"/>
+<wire x1="30.559375" y1="8.651875" x2="30.559375" y2="9.445625" width="0" layer="19" extent="1-1"/>
+<wire x1="29.5275" y1="10.239375" x2="29.5275" y2="9.445625" width="0" layer="19" extent="1-1"/>
+<wire x1="37.7825" y1="14.366875" x2="35.163125" y2="11.645" width="0" layer="19" extent="1-1"/>
+<wire x1="31.4325" y1="3.254375" x2="30.559375" y2="8.651875" width="0" layer="19" extent="1-1"/>
+<wire x1="31.4325" y1="1.886125" x2="31.4325" y2="3.254375" width="0" layer="19" extent="1-1"/>
+<wire x1="34.591625" y1="1.886125" x2="31.4325" y2="1.886125" width="0" layer="19" extent="1-1"/>
+<wire x1="22.888575" y1="4.524375" x2="27.12875" y2="8.90675" width="0" layer="19" extent="1-1"/>
+<wire x1="19.1075" y1="2.578125" x2="22.888575" y2="4.524375" width="0" layer="19" extent="1-1"/>
+<wire x1="25.78" y1="17.23925" x2="30.8855" y2="13.446125" width="0" layer="19" extent="1-1"/>
+<wire x1="23.860125" y1="14.85175" x2="25.78" y2="17.23925" width="0" layer="19" extent="1-1"/>
+<wire x1="21.542375" y1="14.85175" x2="23.860125" y2="14.85175" width="0" layer="19" extent="1-1"/>
+<wire x1="19.52625" y1="15.160625" x2="21.542375" y2="14.85175" width="0" layer="19" extent="1-1"/>
+<wire x1="17.2075" y1="14.878125" x2="19.52625" y2="15.160625" width="0" layer="19" extent="1-1"/>
+<wire x1="14.1575" y1="14.778125" x2="17.2075" y2="14.878125" width="0" layer="19" extent="1-1"/>
+<wire x1="11.1125" y1="11.509375" x2="14.1575" y2="14.778125" width="0" layer="19" extent="1-1"/>
+<wire x1="9.2575" y1="14.778125" x2="11.1125" y2="11.509375" width="0" layer="19" extent="1-1"/>
+<wire x1="5.715" y1="16.03375" x2="9.2575" y2="14.778125" width="0" layer="19" extent="1-1"/>
+<wire x1="12.0715" y1="7.197625" x2="11.1125" y2="11.509375" width="0" layer="19" extent="16-16"/>
+<wire x1="6.111875" y1="4.7625" x2="12.0715" y2="7.197625" width="0" layer="19" extent="16-16"/>
+<wire x1="5.7575" y1="2.578125" x2="6.111875" y2="4.7625" width="0" layer="19" extent="1-1"/>
+<wire x1="14.049375" y1="29.924375" x2="25.04175" y2="31.60275" width="0" layer="19" extent="1-1"/>
+<wire x1="10.795" y1="28.41625" x2="14.049375" y2="29.924375" width="0" layer="19" extent="1-1"/>
+<wire x1="6.35" y1="28.813125" x2="10.795" y2="28.41625" width="0" layer="19" extent="1-1"/>
+<wire x1="1.809625" y1="27.68625" x2="6.35" y2="28.813125" width="0" layer="19" extent="1-1"/>
+<wire x1="13.6525" y1="37.465" x2="14.049375" y2="29.924375" width="0" layer="19" extent="1-1"/>
+<wire x1="5.916125" y1="40.461125" x2="13.6525" y2="37.465" width="0" layer="19" extent="1-1"/>
+<wire x1="5.318125" y1="37.1475" x2="5.916125" y2="40.461125" width="0" layer="19" extent="1-1"/>
+<wire x1="39.766875" y1="16.636875" x2="5.7575" y2="2.578125" width="0" layer="19" extent="1-1"/>
+<wire x1="39.766875" y1="18.636875" x2="39.766875" y2="16.636875" width="0" layer="19" extent="1-1"/>
 </signal>
 <signal name="+3V3">
@@
 <contactref element="U2" pad="P$2"/>
 <contactref element="R10" pad="2"/>
-<contactref element="U$4" pad="P$1"/>
 <polygon width="0.254" layer="1">
 <vertex x="38.655625" y="9.2075"/>
@@
 <wire x1="34.29" y1="8.334375" x2="34.29" y2="7.7225" width="0.254" layer="1"/>
 <wire x1="34.29" y1="7.7225" x2="35.163125" y2="6.849375" width="0.254" layer="1"/>
+<contactref element="U$4" pad="P$1"/>
+<wire x1="34.591625" y1="4.686125" x2="35.163125" y2="6.849375" width="0" layer="19" extent="1-1"/>
+<wire x1="31.4325" y1="4.686125" x2="34.591625" y2="4.686125" width="0" layer="19" extent="1-1"/>
+<wire x1="39.766875" y1="14.636875" x2="31.4325" y2="4.686125" width="0" layer="19" extent="1-1"/>
 </signal>
 <signal name="N$17">
@@
 <contactref element="U$1" pad="VIN"/>
 </signal>
-<signal name="N$12">
-<contactref element="R7" pad="1"/>
-<contactref element="U$5" pad="P$1"/>
-<wire x1="35.14" y1="17.30375" x2="38.766875" y2="17.30375" width="0.4064" layer="1"/>
-<wire x1="38.766875" y1="17.30375" x2="39.766875" y2="16.30375" width="0.4064" layer="1"/>
-</signal>
 <signal name="SWITCH_LED">
 <contactref element="U$1" pad="3"/>
-<contactref element="R7" pad="2"/>
-<wire x1="33.44" y1="17.30375" x2="33.44" y2="18.2" width="0.4064" layer="1"/>
 <wire x1="33.44" y1="18.2" x2="33.575625" y2="18.335625" width="0.4064" layer="1"/>
 <wire x1="33.575625" y1="18.335625" x2="33.575625" y2="20.875625" width="0.4064" layer="1"/>
@@
 <wire x1="25.55875" y1="21.2725" x2="24.669625" y2="20.383375" width="0.4064" layer="1"/>
 <wire x1="24.669625" y1="20.383375" x2="24.669625" y2="20.06625" width="0.4064" layer="1"/>
+<contactref element="R8" pad="1"/>
+<wire x1="32.090625" y1="17.065625" x2="24.669625" y2="20.06625" width="0" layer="19" extent="1-1"/>
 </signal>
 <signal name="N$15">
@@
 <contactref element="U$1" pad="6"/>
 </signal>
+<signal name="N$13">
+<contactref element="R8" pad="2"/>
+<contactref element="U$4" pad="P$2"/>
+<wire x1="39.766875" y1="12.636875" x2="33.790625" y2="17.065625" width="0" layer="19" extent="1-1"/>
+</signal>
 </signals>

Commit message: Updated boards
Parts:
- moved R9 8.02 mm to (35.3, 2.78), turned to 0 degrees
- moved R3 5.56 mm to (29.6, 14.0)
- moved U$4 3.80 mm to (37.9, 12.3)
- moved R8 3.29 mm to (31.8, 14.0), turned to 270 degrees
- moved R5 2.74 mm to (27.4, 14.0), turned to 270 degrees
- moved R10 2.70 mm to (35.3, 5.00), turned to 180 degrees
- moved C10 2.61 mm to (29.0, 4.16)
- moved C9 2.61 mm to (32.1, 4.16)
- moved C6 2.39 mm to (26.3, 3.95)
- moved D2 1.98 mm to (22.6, 4.52)
- moved R4 1.65 mm to (25.2, 14.0), turned to 90 degrees
- moved C8 0.87 mm to (23.0, 14.0)
- moved C7 0.71 mm to (20.8, 14.0)
Connections:
- removed net N$13: R8.2, U$4.P$2
- new net N$12: R8.2, U$4.P$1
- net VIN: now also U$4.P$2; no longer U$4.P$1
Routing:
- net EN: track 3.79 -> 15.9 mm
- net N$12: track 0.00 -> 6.86 mm
- net SWITCH_LED: track 12.9 -> 17.0 mm
- net VIN: track 3.49 -> 0.00 mm
- net N$9: track 5.84 -> 8.34 mm
- net +3V3: track 100.3 -> 102.4 mm
- net N$8: track 2.91 -> 4.46 mm
Other:
- board size 43.2 x 41.9 mm -> 41.9 x 41.9 mm
- board text added: "Cell Tracker 3.1"
- board text removed: "Cell Tracker 3.0"
