File: Boards/LVC/lvc.brd (EAGLE design)
At the start: 20.3 x 20.3 mm, 21 parts, among them Q1 SI7997DP, Q2 RK7002BMT116, U1 NCP300LSN33T1G, U2 L78L33ACUTR, U3 TLV170IDBVR

Commit message: a whole lot of finshed nonsense
Parts:
- removed J1, J2: (no value), pinhead:1X02
- added U$1, U$2: MOLEX_NANOFIT_2, cmdLibs:MOLEX_NANOFIT_2
- moved C4 1.27 mm to (16.0, 8.43)
- moved D2 1.27 mm to (15.1, 14.0)
- moved R4 1.27 mm to (13.3, 1.27)
- moved U1 1.27 mm to (13.3, 5.08)
- moved C2 1.27 mm to (7.62, 17.6)
- moved R6 1.27 mm to (4.68, 7.86)
- moved R5 1.27 mm to (2.51, 7.87)
- moved C1 1.27 mm to (15.2, 17.6)
- moved C3 1.27 mm to (6.37, 11.1)
- moved D1 1.27 mm to (9.53, 1.27)
- moved D3 1.27 mm to (7.78, 14.0)
- moved Q1 1.27 mm to (11.4, 11.3)
- moved Q2 1.27 mm to (19.1, 7.38)
- moved R10 1.27 mm to (5.76, 13.8)
- moved R11 1.27 mm to (6.91, 8.51)
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Connections:
- net GND: now also U$1.P$1, U$2.P$2; no longer J1.1, J2.2
- net VDD: now also U$2.P$1; no longer J2.1
- net VOUT: now also U$1.P$2; no longer J1.2
Routing:
- net GND: track 4.36 -> 1.86 mm, vias 11 -> 10
Other:
- board size 20.3 x 20.3 mm -> 22.9 x 24.1 mm

Commit message: All of the changes with CAD and electronics since switching to the microclasp connectors
Parts:
- removed U$1, U$2: MOLEX_NANOFIT_2, cmdLibs:MOLEX_NANOFIT_2
- added INPUT, LED_STATUS: (no value), NR_connectors:MICROCLASP
- added JP1, JP3: (no value), pinhead:1X02
- added JP2: (no value), pinhead:1X07
- moved D1 24.4 mm to (13.3, 25.4), turned to 180 degrees
- moved R4 24.4 mm to (9.53, 25.4), turned to 180 degrees
- moved R5 20.9 mm to (20.4, 18.8), turned to 90 degrees
- moved Q2 19.5 mm to (3.73, 19.3), turned to 180 degrees
- moved R6 17.4 mm to (18.2, 18.8), turned to 270 degrees
- moved U1 16.9 mm to (9.53, 21.6), turned to 180 degrees
- moved U3 16.9 mm to (13.3, 21.6), turned to 180 degrees
- moved C4 13.3 mm to (6.91, 18.2), turned to 270 degrees
- moved R11 13.2 mm to (16.0, 18.2), turned to 270 degrees
- moved C1 11.5 mm to (7.62, 9.05), turned to 270 degrees
- moved C2 11.5 mm to (15.2, 9.05), turned to 270 degrees
- moved R10 11.4 mm to (17.1, 12.9), turned to 90 degrees
- moved R2 11.4 mm to (5.76, 12.9), turned to 90 degrees
- moved C3 11.1 mm to (16.5, 15.6), turned to 180 degrees
- moved R3 11.1 mm to (6.37, 15.6), turned to 0 degrees
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Connections:
- removed net VOUT: C1.1, Q1.5, Q1.5L, Q1.6, U$1.P$2, U2.3
- new net MISO_6: JP2.2
- new net N$9: JP2.7
- new net RST: JP2.6
- new net SCK_7: JP2.3
- new net SCL_16: JP2.5
- new net SDA_17: JP2.4
- new net STATUS: JP2.1, LED_STATUS.P$2
- new net VREG: C1.1, JP1.2, JP3.2, Q1.5, Q1.5L, Q1.6, U2.3
- net GND: now also INPUT.P$2, JP1.1, JP3.1, LED_STATUS.P$1; no longer U$1.P$1, U$2.P$2
- net VDD: now also INPUT.P$1; no longer U$2.P$1
Routing:
- net V+: track 27.3 -> 0.00 mm
- net V_DIV_BUF: track 17.1 -> 0.00 mm
- net V_DIV: track 14.7 -> 0.00 mm
- net N$6: track 11.2 -> 0.00 mm
- net LOAD: track 10.4 -> 0.00 mm
- net N$5: track 8.99 -> 0.00 mm
- net N$7: track 4.83 -> 0.00 mm
- net LED: track 3.19 -> 1.15 mm
- net GND: vias 10 -> 8
- removed copper zone on layer 16, net GND
- removed copper zone on layer 1, net VDD
- removed copper zone on layer 1, net VOUT
Other:
- board size 22.9 x 24.1 mm -> 30.5 x 31.8 mm
- board text removed: "2 Cell ONLY"
- board text removed: "LVC Rev 6.1"

Commit message: fixes and design review slides
Parts:
- removed INPUT, LED_STATUS: (no value), NR_connectors:MICROCLASP
- added R1: (no value), resistor:R0603
- added U$1: MICROCLASP_4, NR_connectors:4_PIN_MICROCLASP
Connections:
- new net N$1: R1.2, U$1.P$2
- net GND: now also U$1.P$3, U$1.P$4; no longer INPUT.P$2, LED_STATUS.P$1
- net STATUS: now also R1.1; no longer LED_STATUS.P$2
- net VDD: now also U$1.P$1; no longer INPUT.P$1
Changed lines of the file:
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@@
 <element name="JP2" library="pinhead" package="1X07" value="" x="20.32" y="29.21" rot="R180"/>
 <element name="JP3" library="pinhead" package="1X02" value="" x="6.35" y="29.21"/>
-<element name="LED_STATUS" library="NR_connectors" package="MICROCLASP" value="" x="26.431875" y="23.01875" rot="R270"/>
-<element name="INPUT" library="NR_connectors" package="MICROCLASP" value="" x="26.590625" y="14.366875" rot="R270"/>
+<element name="U$1" library="NR_connectors" package="4_PIN_MICROCLASP" value="MICROCLASP_4" x="27.14625" y="15.08125" rot="R270"/>
+<element name="R1" library="resistor" package="R0603" value="" x="27.94" y="24.13" rot="R270"/>
 </elements>
 <signals>
@@
 <contactref element="JP1" pad="1"/>
 <contactref element="JP3" pad="1"/>
-<contactref element="LED_STATUS" pad="P$1"/>
-<contactref element="INPUT" pad="P$2"/>
-<wire x1="26.590625" y1="15.366875" x2="26.431875" y2="22.01875" width="0" layer="19" extent="1-1"/>
-<wire x1="18.335625" y1="16.8275" x2="26.590625" y2="15.366875" width="0" layer="19" extent="1-1"/>
+<contactref element="U$1" pad="P$3"/>
+<contactref element="U$1" pad="P$4"/>
+<wire x1="27.14625" y1="12.08125" x2="27.14625" y2="14.08125" width="0" layer="19" extent="1-1"/>
+<wire x1="5.08" y1="2.54" x2="27.14625" y2="12.08125" width="0" layer="19" extent="1-1"/>
+<wire x1="6.588125" y1="8.175625" x2="5.08" y2="2.54" width="0" layer="19" extent="1-1"/>
+<wire x1="5.635625" y1="10.239375" x2="6.61125" y2="8.19875" width="0" layer="19" extent="1-1"/>
+<wire x1="11.43" y1="10.963275" x2="7.62" y2="8.19875" width="0" layer="19" extent="1-1"/>
+<wire x1="15.24" y1="8.19875" x2="11.43" y2="10.963275" width="0" layer="19" extent="1-1"/>
+<wire x1="17.383125" y1="8.5725" x2="15.24" y2="8.19875" width="0" layer="19" extent="1-1"/>
+<wire x1="17.097375" y1="13.70875" x2="17.383125" y2="8.5725" width="0" layer="19" extent="1-1"/>
+<wire x1="15.644125" y1="15.5575" x2="17.097375" y2="13.70875" width="0" layer="19" extent="1-1"/>
+<wire x1="18.335625" y1="16.8275" x2="15.644125" y2="15.5575" width="0" layer="19" extent="1-1"/>
 <wire x1="18.176875" y1="17.961875" x2="18.335625" y2="16.8275" width="0" layer="19" extent="1-1"/>
 <wire x1="15.954375" y1="19.011" x2="18.176875" y2="17.961875" width="0" layer="19" extent="1-1"/>
-<wire x1="15.644125" y1="15.5575" x2="18.335625" y2="16.8275" width="0" layer="19" extent="1-1"/>
-<wire x1="17.097375" y1="13.70875" x2="15.644125" y2="15.5575" width="0" layer="19" extent="1-1"/>
 <wire x1="13.335" y1="22.89" x2="15.954375" y2="19.011" width="0" layer="19" extent="1-1"/>
 <wire x1="13.890625" y1="24.209375" x2="13.335" y2="22.89" width="0" layer="19" extent="1-1"/>
@@
 <wire x1="2.780625" y1="20.288125" x2="3.81" y2="21.59" width="0" layer="19" extent="1-1"/>
 <wire x1="6.905625" y1="17.390375" x2="2.780625" y2="20.288125" width="0" layer="19" extent="1-1"/>
-<wire x1="17.383125" y1="8.5725" x2="17.097375" y2="13.70875" width="0" layer="19" extent="1-1"/>
-<wire x1="15.24" y1="8.19875" x2="17.383125" y2="8.5725" width="0" layer="19" extent="1-1"/>
-<wire x1="11.43" y1="10.963275" x2="15.24" y2="8.19875" width="0" layer="19" extent="1-1"/>
-<wire x1="7.62" y1="8.19875" x2="11.43" y2="10.963275" width="0" layer="19" extent="1-1"/>
-<wire x1="5.635625" y1="10.239375" x2="6.61125" y2="8.19875" width="0" layer="19" extent="1-1"/>
-<wire x1="5.08" y1="2.54" x2="6.588125" y2="8.175625" width="0" layer="19" extent="1-1"/>
 </signal>
 <signal name="V+">
@@
 <contactref element="Q1" pad="8"/>
 <contactref element="Q1" pad="8L"/>
-<contactref element="INPUT" pad="P$1"/>
-<wire x1="13.335" y1="12.65875" x2="26.590625" y2="13.366875" width="0" layer="19" extent="1-1"/>
-<wire x1="12.04" y1="12.50375" x2="13.335" y2="12.65875" width="0" layer="19" extent="1-1"/>
+<contactref element="U$1" pad="P$1"/>
+<wire x1="12.04" y1="12.50375" x2="27.14625" y2="16.08125" width="0" layer="19" extent="1-1"/>
+<wire x1="13.335" y1="12.65875" x2="12.04" y2="12.50375" width="0" layer="19" extent="1-1"/>
 <wire x1="12.56" y1="14.76375" x2="13.335" y2="12.65875" width="0" layer="19" extent="1-1"/>
 </signal>
@@
 </signal>
 <signal name="STATUS">
-<contactref element="LED_STATUS" pad="P$2"/>
 <contactref element="JP2" pad="1"/>
-<wire x1="27.94" y1="29.21" x2="26.431875" y2="24.01875" width="0" layer="19" extent="1-1"/>
+<contactref element="R1" pad="1"/>
+<wire x1="27.94" y1="29.21" x2="27.94" y2="24.98" width="0" layer="19" extent="1-1"/>
+</signal>
+<signal name="N$1">
+<contactref element="U$1" pad="P$2"/>
+<contactref element="R1" pad="2"/>
+<wire x1="27.14625" y1="18.08125" x2="27.94" y2="23.28" width="0" layer="19" extent="1-1"/>
 </signal>
 </signals>

Commit message: Updated boards
Parts:
- removed JP1, JP3: (no value), pinhead:1X02
- added U$2, U$3: LITEAPRS, NR_connectors:LITEAPRS
- moved R2 17.5 mm to (19.4, 23.8), turned to 270 degrees
- moved D3 16.1 mm to (26.7, 23.8)
- moved C4 16.0 mm to (21.8, 23.9), turned to 90 degrees
- moved R10 13.1 mm to (24.3, 23.8)
- moved D2 12.9 mm to (17.9, 20.6), turned to 0 degrees
- moved R6 10.9 mm to (8.65, 24.1)
- moved R5 10.7 mm to (11.1, 24.1)
- moved R11 10.1 mm to (6.81, 13.9), turned to 180 degrees
- moved C3 9.76 mm to (6.76, 16.3), turned to 0 degrees
- moved Q2 9.27 mm to (12.4, 16.0), turned to 270 degrees
- moved R3 8.92 mm to (14.3, 19.7), turned to 180 degrees
- moved Q1 7.62 mm to (19.1, 15.2)
- moved D1 7.16 mm to (6.27, 24.2), turned to 270 degrees
- moved R4 5.91 mm to (11.0, 19.7), turned to 0 degrees
- moved U3 3.90 mm to (15.5, 24.8)
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Connections:
- net GND: now also U$2.P$2, U$3.P$2; no longer JP1.1, JP3.1
- net VREG: now also U$2.P$1, U$3.P$1; no longer JP1.2, JP3.2
Routing:
- net VREG: track 0.00 -> 49.8 mm
- net V+: track 0.00 -> 25.2 mm
- net V_DIV_BUF: track 0.00 -> 19.2 mm
- net N$6: track 0.00 -> 9.84 mm
- net V_DIV: track 0.00 -> 9.13 mm
- net N$5: track 0.00 -> 8.35 mm
- net STATUS: track 0.00 -> 6.98 mm
- net N$1: track 0.00 -> 6.64 mm
- net LOAD: track 0.00 -> 5.94 mm
- net N$7: track 0.00 -> 3.75 mm
- net LED: track 1.15 -> 3.98 mm
- net GND: track 1.86 -> 0.00 mm, vias 8 -> 0
- added copper zone on layer 16, net GND
- added copper zone on layer 1, net VDD
Other:
- board size 30.5 x 31.8 mm -> 31.4 x 33.5 mm
- board text added: "LED"
- board text added: "V2"
- board text added: "Vin"
- board text added: "Vreg"
- board text added: "liteAPRS LVC"
- board text removed: "IN"
- board text removed: "OUT"
- board text removed: "SN"
