File: Boards/LVC/lvc.sch (EAGLE design)
At the start: 21 parts, among them Q1 SI7997DP, Q2 RK7002BMT116, U1 NCP300LSN33T1G, U2 L78L33ACUTR, U3 TLV170IDBVR

Commit message: a whole lot of finshed nonsense
Parts:
- removed J1, J2: (no value), pinhead:PINHD-1X2
- added U$1, U$2: MOLEX_NANOFIT_2, cmdLibs:MOLEX_NANOFIT_2
Connections:
- net GND: now also U$1.P1, U$2.P2; no longer J1.1, J2.2
- net VDD: now also U$2.P1; no longer J2.1
- net VOUT: now also U$1.P2; no longer J1.2
Changed lines of the file:
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@@
 <part name="GND8" library="supply1" deviceset="GND" device=""/>
 <part name="R4" library="resistor" deviceset="R-US_" device="R0603" value="100k"/>
-<part name="J1" library="pinhead" deviceset="PINHD-1X2" device=""/>
-<part name="J2" library="pinhead" deviceset="PINHD-1X2" device=""/>
 <part name="GND9" library="supply1" deviceset="GND" device=""/>
 <part name="GND10" library="supply1" deviceset="GND" device=""/>
@@
 <part name="D3" library="LR_zener" deviceset="DZ2J120M0L" device=""/>
 <part name="Q2" library="LR_transistor" deviceset="RK7002BMT116" device=""/>
+<part name="U$1" library="cmdLibs" deviceset="MOLEX_NANOFIT_2" device=""/>
+<part name="U$2" library="cmdLibs" deviceset="MOLEX_NANOFIT_2" device=""/>
 </parts>
 <sheets>
@@
 <attribute name="VALUE" x="39.37" y="43.942" size="1.778" layer="96" rot="R180"/>
 </instance>
-<instance part="J1" gate="G$1" x="236.22" y="182.88" smashed="yes" rot="R180">
-<attribute name="NAME" x="238.76" y="177.292" size="1.778" layer="95" rot="R180"/>
-<attribute name="VALUE" x="259.08" y="187.96" size="1.778" layer="96" rot="R180"/>
-</instance>
-<instance part="J2" gate="G$1" x="241.3" y="154.94" smashed="yes">
-<attribute name="NAME" x="236.22" y="152.908" size="1.778" layer="95"/>
-<attribute name="VALUE" x="215.9" y="149.86" size="1.778" layer="96"/>
-</instance>
 <instance part="GND9" gate="1" x="248.92" y="147.32"/>
 <instance part="GND10" gate="1" x="228.6" y="172.72"/>
@@
 <instance part="D3" gate="A" x="243.84" y="93.98" rot="R180"/>
 <instance part="Q2" gate="G$1" x="48.26" y="55.88"/>
+<instance part="U$1" gate="G$1" x="243.84" y="180.34" rot="R180"/>
+<instance part="U$2" gate="G$1" x="233.68" y="157.48"/>
 </instances>
 <busses>
@@
 </segment>
 <segment>
-<pinref part="J2" gate="G$1" pin="2"/>
 <wire x1="238.76" y1="154.94" x2="248.92" y2="154.94" width="0.1524" layer="91"/>
 <wire x1="248.92" y1="154.94" x2="248.92" y2="149.86" width="0.1524" layer="91"/>
 <pinref part="GND9" gate="1" pin="GND"/>
+<pinref part="U$2" gate="G$1" pin="P2"/>
+<wire x1="238.76" y1="154.94" x2="238.76" y2="152.4" width="0.1524" layer="91"/>
+<wire x1="238.76" y1="152.4" x2="236.22" y2="152.4" width="0.1524" layer="91"/>
 </segment>
 <segment>
 <wire x1="228.6" y1="180.34" x2="228.6" y2="175.26" width="0.1524" layer="91"/>
 <pinref part="GND10" gate="1" pin="GND"/>
-<pinref part="J1" gate="G$1" pin="1"/>
 <wire x1="238.76" y1="180.34" x2="228.6" y2="180.34" width="0.1524" layer="91"/>
+<pinref part="U$1" gate="G$1" pin="P1"/>
+<wire x1="238.76" y1="180.34" x2="238.76" y2="177.8" width="0.1524" layer="91"/>
+<wire x1="238.76" y1="177.8" x2="241.3" y2="177.8" width="0.1524" layer="91"/>
 </segment>
 <segment>
@@
 <wire x1="228.6" y1="182.88" x2="228.6" y2="187.96" width="0.1524" layer="91"/>
 <label x="228.6" y="187.96" size="1.016" layer="95" rot="R90" xref="yes"/>
-<pinref part="J1" gate="G$1" pin="2"/>
 <wire x1="238.76" y1="182.88" x2="228.6" y2="182.88" width="0.1524" layer="91"/>
+<pinref part="U$1" gate="G$1" pin="P2"/>
+<wire x1="238.76" y1="182.88" x2="238.76" y2="185.42" width="0.1524" layer="91"/>
+<wire x1="238.76" y1="185.42" x2="241.3" y2="185.42" width="0.1524" layer="91"/>
 </segment>
 <segment>
@@
 <net name="VDD" class="0">
 <segment>
-<pinref part="J2" gate="G$1" pin="1"/>
 <pinref part="VDD1" gate="G$1" pin="VDD"/>
 <wire x1="238.76" y1="157.48" x2="248.92" y2="157.48" width="0.1524" layer="91"/>
 <wire x1="248.92" y1="157.48" x2="248.92" y2="162.56" width="0.1524" layer="91"/>
-</segment>
-<segment>
+<pinref part="U$2" gate="G$1" pin="P1"/>
+<wire x1="238.76" y1="157.48" x2="238.76" y2="160.02" width="0.1524" layer="91"/>
+<wire x1="238.76" y1="160.02" x2="236.22" y2="160.02" width="0.1524" layer="91"/>
+</segment>
+<segment>

Commit message: All of the changes with CAD and electronics since switching to the microclasp connectors
Parts:
- removed U$1, U$2: MOLEX_NANOFIT_2, cmdLibs:MOLEX_NANOFIT_2
- added INPUT, LED_STATUS: (no value), NR_connectors:MICROCLASP
- added JP1, JP3: (no value), pinhead:PINHD-1X2
- added JP2: (no value), pinhead:PINHD-1X7
Connections:
- removed net VOUT: C1.1, Q1A.D, U$1.P2, U2.VIN
- new net MISO_6: JP2.2
- new net N$9: JP2.7
- new net RST: JP2.6
- new net SCK_7: JP2.3
- new net SCL_16: JP2.5
- new net SDA_17: JP2.4
- new net STATUS: JP2.1, LED_STATUS.P$2
- new net VREG: C1.1, JP1.2, JP3.2, Q1A.D, U2.VIN
- net GND: now also INPUT.P$2, JP1.1, JP3.1, LED_STATUS.P$1; no longer U$1.P1, U$2.P2
- net VDD: now also INPUT.P$1; no longer U$2.P1
Other:
- note added: "Connectors"
- note removed: "Screw Terminals"
- moved on the sheet: C1, C2, C3, C4, D1, D2, D3, Q1A, Q1B, Q2, R10, R11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

Commit message: fixes and design review slides
Parts:
- removed INPUT, LED_STATUS: (no value), NR_connectors:MICROCLASP
- added R1: (no value), resistor:R-US_R0603
- added U$1: MICROCLASP_4, NR_connectors:MICROCLASP_4
Connections:
- new net N$1: R1.2, U$1.P$2
- net GND: now also U$1.P$3, U$1.P$4; no longer INPUT.P$2, LED_STATUS.P$1
- net STATUS: now also R1.1; no longer LED_STATUS.P$2
- net VDD: now also U$1.P$1; no longer INPUT.P$1
Other:
- note added: "Divider"
- note removed: "Dividers"
Changed lines of the file:
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@@
 <part name="GND8" library="supply1" deviceset="GND" device=""/>
 <part name="R4" library="resistor" deviceset="R-US_" device="R0603" value="100k"/>
-<part name="GND9" library="supply1" deviceset="GND" device=""/>
-<part name="GND10" library="supply1" deviceset="GND" device=""/>
 <part name="R5" library="resistor" deviceset="R-US_" device="R0603" value="1M"/>
 <part name="R6" library="resistor" deviceset="R-US_" device="R0603" value="1M"/>
@@
 <part name="GND13" library="supply1" deviceset="GND" device=""/>
 <part name="+3V1" library="supply1" deviceset="+3V3" device=""/>
-<part name="LED_STATUS" library="NR_connectors" deviceset="MICROCLASP" device=""/>
-<part name="INPUT" library="NR_connectors" deviceset="MICROCLASP" device=""/>
+<part name="U$1" library="NR_connectors" deviceset="MICROCLASP_4" device=""/>
+<part name="R1" library="resistor" deviceset="R-US_" device="R0603"/>
+<part name="GND9" library="supply1" deviceset="GND" device=""/>
 </parts>
 <sheets>
@@
 <text x="5.08" y="170.18" size="3.81" layer="97">Voltage Regulator</text>
 <text x="10.16" y="81.28" size="3.81" layer="97">Switching</text>
-<text x="147.32" y="167.64" size="3.81" layer="97">Dividers</text>
+<text x="147.32" y="167.64" size="3.81" layer="97">Divider</text>
 <wire x1="73.66" y1="5.08" x2="73.66" y2="91.44" width="0.1524" layer="97" style="shortdash"/>
 <wire x1="256.54" y1="91.44" x2="182.88" y2="91.44" width="0.1524" layer="97" style="shortdash"/>
@@
 <attribute name="VALUE" x="16.51" y="18.542" size="1.778" layer="96" rot="R180"/>
 </instance>
-<instance part="GND9" gate="1" x="236.22" y="144.78"/>
-<instance part="GND10" gate="1" x="195.58" y="144.78"/>
 <instance part="R5" gate="G$1" x="172.72" y="162.56" smashed="yes" rot="R270">
 <attribute name="NAME" x="173.99" y="164.0586" size="1.778" layer="95"/>
@@
 <attribute name="VALUE" x="159.258" y="72.39" size="1.778" layer="96"/>
 </instance>
-<instance part="VDD1" gate="G$1" x="238.76" y="154.94" rot="R270"/>
+<instance part="VDD1" gate="G$1" x="208.28" y="154.94" rot="R270"/>
 <instance part="VDD2" gate="G$1" x="171.958" y="46.99" smashed="yes" rot="R180">
 <attribute name="VALUE" x="174.498" y="44.45" size="1.778" layer="96" rot="R180"/>
@@
 <instance part="GND13" gate="1" x="198.12" y="109.22"/>
 <instance part="+3V1" gate="G$1" x="236.22" y="129.54" rot="R270"/>
-<instance part="LED_STATUS" gate="G$1" x="210.82" y="152.4" rot="R180"/>
-<instance part="INPUT" gate="G$1" x="220.98" y="154.94"/>
+<instance part="U$1" gate="G$1" x="187.96" y="149.86"/>
+<instance part="R1" gate="G$1" x="205.74" y="147.32" rot="R90"/>
+<instance part="GND9" gate="1" x="200.66" y="142.24"/>
 </instances>
 <busses>
@@
 <wire x1="17.78" y1="15.24" x2="17.78" y2="12.7" width="0.1524" layer="91"/>
 <pinref part="R4" gate="G$1" pin="2"/>
-</segment>
-<segment>
-<wire x1="231.14" y1="152.4" x2="236.22" y2="152.4" width="0.1524" layer="91"/>
-<wire x1="236.22" y1="152.4" x2="236.22" y2="147.32" width="0.1524" layer="91"/>
-<pinref part="GND9" gate="1" pin="GND"/>
-<pinref part="INPUT" gate="G$1" pin="P$2"/>
-</segment>
-<segment>
-<wire x1="195.58" y1="152.4" x2="195.58" y2="147.32" width="0.1524" layer="91"/>
-<pinref part="GND10" gate="1" pin="GND"/>
-<wire x1="200.66" y1="152.4" x2="195.58" y2="152.4" width="0.1524" layer="91"/>
-<pinref part="LED_STATUS" gate="G$1" pin="P$1"/>
 </segment>
 <segment>
@@
 <pinref part="GND13" gate="1" pin="GND"/>
 </segment>
+<segment>
+<pinref part="U$1" gate="G$1" pin="P$3"/>
+<wire x1="198.12" y1="149.86" x2="200.66" y2="149.86" width="0.1524" layer="91"/>
+<wire x1="200.66" y1="149.86" x2="200.66" y2="147.32" width="0.1524" layer="91"/>
+<pinref part="U$1" gate="G$1" pin="P$4"/>
+<wire x1="200.66" y1="147.32" x2="200.66" y2="144.78" width="0.1524" layer="91"/>
+<wire x1="198.12" y1="147.32" x2="200.66" y2="147.32" width="0.1524" layer="91"/>
+<pinref part="GND9" gate="1" pin="GND"/>
+</segment>
 </net>
 <net name="V+" class="0">
@@
 <segment>
 <pinref part="VDD1" gate="G$1" pin="VDD"/>
-<wire x1="231.14" y1="154.94" x2="236.22" y2="154.94" width="0.1524" layer="91"/>
-<pinref part="INPUT" gate="G$1" pin="P$1"/>
+<wire x1="198.12" y1="154.94" x2="205.74" y2="154.94" width="0.1524" layer="91"/>
+<pinref part="U$1" gate="G$1" pin="P$1"/>
 </segment>
 <segment>
@@
 <net name="STATUS" class="0">
 <segment>
-<label x="195.58" y="154.94" size="1.016" layer="95" rot="R180" xref="yes"/>
-<wire x1="200.66" y1="154.94" x2="195.58" y2="154.94" width="0.1524" layer="91"/>
-<pinref part="LED_STATUS" gate="G$1" pin="P$2"/>
-</segment>
-<segment>
 <pinref part="JP2" gate="A" pin="1"/>
 <wire x1="226.06" y1="114.3" x2="233.68" y2="114.3" width="0.1524" layer="91"/>
 <label x="233.68" y="114.3" size="1.016" layer="95" xref="yes"/>
 </segment>
-</net>
+<segment>
+<pinref part="R1" gate="G$1" pin="1"/>
+<wire x1="205.74" y1="142.24" x2="205.74" y2="139.7" width="0.1524" layer="91"/>
+<label x="205.74" y="139.7" size="1.016" layer="95" xref="yes"/>
+</segment>
+</net>
+<net name="N$1" class="0">
+<segment>
+<pinref part="U$1" gate="G$1" pin="P$2"/>
+<pinref part="R1" gate="G$1" pin="2"/>
+<wire x1="198.12" y1="152.4" x2="205.74" y2="152.4" width="0.1524" layer="91"/>
+</segment>
+</net>

Commit message: Updated boards
Parts:
- removed JP1, JP3: (no value), pinhead:PINHD-1X2
- added U$2, U$3: LITEAPRS, NR_connectors:LITEAPRS
Connections:
- net GND: now also U$2.P$2, U$3.P$2; no longer JP1.1, JP3.1
- net VREG: now also U$2.P$1, U$3.P$1; no longer JP1.2, JP3.2
Changed lines of the file:
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@@
 <part name="Q2" library="LR_transistor" deviceset="RK7002BMT116" device=""/>
 <part name="FRAME1" library="frames" deviceset="A4L-LOC" device=""/>
-<part name="JP1" library="pinhead" deviceset="PINHD-1X2" device=""/>
 <part name="JP2" library="pinhead" deviceset="PINHD-1X7" device=""/>
-<part name="JP3" library="pinhead" deviceset="PINHD-1X2" device=""/>
 <part name="GND2" library="supply1" deviceset="GND" device=""/>
 <part name="GND13" library="supply1" deviceset="GND" device=""/>
@@
 <part name="R1" library="resistor" deviceset="R-US_" device="R0603"/>
 <part name="GND9" library="supply1" deviceset="GND" device=""/>
+<part name="U$2" library="NR_connectors" deviceset="LITEAPRS" device=""/>
+<part name="U$3" library="NR_connectors" deviceset="LITEAPRS" device=""/>
 </parts>
 <sheets>
@@
 <instance part="Q2" gate="G$1" x="25.4" y="30.48"/>
 <instance part="FRAME1" gate="G$1" x="0" y="0"/>
-<instance part="JP1" gate="G$1" x="187.96" y="129.54" rot="R180"/>
 <instance part="JP2" gate="A" x="223.52" y="121.92" rot="R180"/>
-<instance part="JP3" gate="G$1" x="187.96" y="114.3" rot="R180"/>
 <instance part="GND2" gate="1" x="198.12" y="124.46"/>
 <instance part="GND13" gate="1" x="198.12" y="109.22"/>
@@
 <instance part="R1" gate="G$1" x="205.74" y="147.32" rot="R90"/>
 <instance part="GND9" gate="1" x="200.66" y="142.24"/>
+<instance part="U$2" gate="G$1" x="180.34" y="129.54"/>
+<instance part="U$3" gate="G$1" x="180.34" y="114.3"/>
 </instances>
 <busses>
@@
 </segment>
 <segment>
-<pinref part="JP1" gate="G$1" pin="1"/>
 <wire x1="190.5" y1="127" x2="198.12" y2="127" width="0.1524" layer="91"/>
 <pinref part="GND2" gate="1" pin="GND"/>
-</segment>
-<segment>
-<pinref part="JP3" gate="G$1" pin="1"/>
+<pinref part="U$2" gate="G$1" pin="P$2"/>
+</segment>
+<segment>
 <wire x1="190.5" y1="111.76" x2="198.12" y2="111.76" width="0.1524" layer="91"/>
 <pinref part="GND13" gate="1" pin="GND"/>
+<pinref part="U$3" gate="G$1" pin="P$2"/>
 </segment>
 <segment>
@@
 </segment>
 <segment>
-<pinref part="JP1" gate="G$1" pin="2"/>
 <wire x1="190.5" y1="129.54" x2="198.12" y2="129.54" width="0.1524" layer="91"/>
 <label x="198.12" y="129.54" size="1.016" layer="95" xref="yes"/>
-</segment>
-<segment>
-<pinref part="JP3" gate="G$1" pin="2"/>
+<pinref part="U$2" gate="G$1" pin="P$1"/>
+</segment>
+<segment>
 <wire x1="190.5" y1="114.3" x2="198.12" y2="114.3" width="0.1524" layer="91"/>
 <label x="198.12" y="114.3" size="1.016" layer="95" xref="yes"/>
-</segment>
-</net>
+<pinref part="U$3" gate="G$1" pin="P$1"/>
+</segment>
+</net>
