File: Boards/CellTracker_v3.2/cell.sch (EAGLE design)
At the start: 24 parts, among them U2 LMR16020

Commit message: Code+nearly completed boards
Parts:
- added C1: (no value), jmolterLib:DCK-3R3E204T614-E
- added D1: RB520S30T1G, diode:DIODE-SOD523
- added R7: 22, resistor:R-US_R0603
- C6: value 47 uF -> 0.1 uF
- R10: value 195k -> 140k
- R4: value 45k -> 340k
- R5: value 13.3k -> 100k
- R9: value 45k -> 30.1k
Connections:
- new net N$11: D1.C, R7.2
- new net N$5: C1.3V3, R7.1, U$7.6_V_BCKP
- net +3V3: now also D1.A; no longer U$7.6_V_BCKP
- net GND: now also C1.GND
Other:
- moved on the sheet: C10, C6, C7, C8, C9, D2, L1, R10, R2, R3, R4, R5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
