File: Boards/BITS3.2/bits3.2.sch (EAGLE design)
At the start: 32 parts, among them U1 LMR16020, X2 53398-10

Commit message: Code+nearly completed boards
Parts:
- C2: value .1 uF -> 0.1uF
- R1: value 18k -> 180k
- R3: value 10k -> 100k
- U$2: value TEENSY_3.1-3.2_ALL_PINS -> TEENSY_3.1-3.2_OUTER_ROW; device Teensy_3_and_LC_Series_Boards_v1.4:TEENSY_3.1-3.2_ALL_PINS -> Teensy_3_and_LC_Series_Boards_v1.4:TEENSY_3.1-3.2_OUTER_ROW
Connections:
- net LED1: now also U$2.4/CAN-RX-PWM; no longer U$2.4/CAN-RX/PWM
Other:
- moved on the sheet: R18
Changed lines of the file:
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@@
 </classes>
 <parts>
-<part name="U$2" library="Teensy_3_and_LC_Series_Boards_v1.4" deviceset="TEENSY_3.1-3.2_ALL_PINS" device=""/>
+<part name="U$2" library="Teensy_3_and_LC_Series_Boards_v1.4" deviceset="TEENSY_3.1-3.2_OUTER_ROW" device=""/>
 <part name="GND2" library="supply1" deviceset="GND" device=""/>
 <part name="X2" library="con-molex" deviceset="53?-10" device="398"/>
-<part name="R1" library="resistor" deviceset="R-US_" device="R0603" value="18k"/>
-<part name="R3" library="resistor" deviceset="R-US_" device="R0603" value="10k"/>
+<part name="R1" library="resistor" deviceset="R-US_" device="R0603" value="180k"/>
+<part name="R3" library="resistor" deviceset="R-US_" device="R0603" value="100k"/>
 <part name="GND4" library="supply1" deviceset="GND" device=""/>
 <part name="R9" library="resistor" deviceset="R-US_" device="R0603" value="470"/>
@@
 <part name="R18" library="resistor" deviceset="R-US_" device="R0603" value="45k"/>
 <part name="R19" library="resistor" deviceset="R-US_" device="R0603" value="13.3k"/>
-<part name="C2" library="resistor" deviceset="C-US" device="C0603" value=".1 uF"/>
+<part name="C2" library="resistor" deviceset="C-US" device="C0603" value="0.1uF"/>
 <part name="C3" library="resistor" deviceset="C-US" device="C1210" value="10 uF"/>
 <part name="C4" library="resistor" deviceset="C-US" device="C0603" value=".18 uF"/>
@@
 <attribute name="VALUE" x="212.852" y="145.542" size="1.016" layer="95"/>
 </instance>
-<instance part="R18" gate="G$1" x="233.68" y="142.24" smashed="yes" rot="R90">
-<attribute name="NAME" x="232.1814" y="140.462" size="1.27" layer="95" rot="R90"/>
-<attribute name="VALUE" x="236.474" y="140.716" size="1.27" layer="96" rot="R90"/>
+<instance part="R18" gate="G$1" x="233.68" y="139.7" smashed="yes" rot="R90">
+<attribute name="NAME" x="232.1814" y="137.922" size="1.27" layer="95" rot="R90"/>
+<attribute name="VALUE" x="236.474" y="138.176" size="1.27" layer="96" rot="R90"/>
 </instance>
 <instance part="R19" gate="G$1" x="233.68" y="124.46" smashed="yes" rot="R90">
@@
 <pinref part="+3V6" gate="G$1" pin="+3V3"/>
 <wire x1="251.46" y1="147.32" x2="251.46" y2="152.4" width="0.1524" layer="91"/>
-<pinref part="R18" gate="G$1" pin="2"/>
-<pinref part="L1" gate="G$1" pin="P$2"/>
-<wire x1="231.14" y1="147.32" x2="233.68" y2="147.32" width="0.1524" layer="91"/>
-<wire x1="233.68" y1="147.32" x2="241.3" y2="147.32" width="0.1524" layer="91"/>
-<junction x="233.68" y="147.32"/>
 <pinref part="C4" gate="G$1" pin="1"/>
 <wire x1="241.3" y1="147.32" x2="248.92" y2="147.32" width="0.1524" layer="91"/>
 <wire x1="248.92" y1="147.32" x2="251.46" y2="147.32" width="0.1524" layer="91"/>
 <wire x1="241.3" y1="144.78" x2="241.3" y2="147.32" width="0.1524" layer="91"/>
-<junction x="241.3" y="147.32"/>
 <pinref part="C11" gate="G$1" pin="1"/>
 <wire x1="248.92" y1="144.78" x2="248.92" y2="147.32" width="0.1524" layer="91"/>
 <junction x="248.92" y="147.32"/>
+<junction x="233.68" y="147.32"/>
+<pinref part="L1" gate="G$1" pin="P$2"/>
+<wire x1="231.14" y1="147.32" x2="233.68" y2="147.32" width="0.1524" layer="91"/>
+<pinref part="R18" gate="G$1" pin="2"/>
+<wire x1="233.68" y1="144.78" x2="233.68" y2="147.32" width="0.1524" layer="91"/>
+<wire x1="233.68" y1="147.32" x2="241.3" y2="147.32" width="0.1524" layer="91"/>
+<junction x="241.3" y="147.32"/>
 </segment>
 <segment>
@@
 </segment>
 <segment>
-<pinref part="U$2" gate="G$1" pin="4/CAN-RX/PWM"/>
+<pinref part="U$2" gate="G$1" pin="4/CAN-RX-PWM"/>
 <wire x1="20.32" y1="226.06" x2="17.78" y2="226.06" width="0.1524" layer="91"/>
 <label x="17.78" y="226.06" size="1.27" layer="95" rot="R180" xref="yes"/>
@@
 <wire x1="233.68" y1="132.08" x2="233.68" y2="129.54" width="0.1524" layer="91"/>
 <pinref part="R18" gate="G$1" pin="1"/>
-<wire x1="233.68" y1="137.16" x2="233.68" y2="132.08" width="0.1524" layer="91"/>
+<wire x1="233.68" y1="134.62" x2="233.68" y2="132.08" width="0.1524" layer="91"/>
 <junction x="233.68" y="132.08"/>
 <pinref part="U1" gate="G$1" pin="FB"/>

Commit message: More stuff, close, not done
Parts:
- added X1: 53261-04, con-molex:53261-04
Connections:
- new net N$8: X1-2.S
- new net N$9: X1-3.S
- net +3V3: now also X1-1.S
- net GND: now also X1-4.S
Other:
- note added: "Isolated Conn"
- note added: "Voltage Divider"
- note removed: "Voltage Moniter"
- moved on the sheet: C11, C2, C3, C4, C5, D1, D3, L1, LED1, LED2, R1, R10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
