File: Boards/BITS3.2/bits3.2.brd (EAGLE design)
At the start: 45 x 45 mm, 32 parts, among them U1 LMR16020, X2 53398-10

Commit message: Code+nearly completed boards
Parts:
- C2: value .1 uF -> 0.1uF
- R1: value 18k -> 180k
- R3: value 10k -> 100k
- U$2: value TEENSY_3.1-3.2_ALL_PINS -> TEENSY_3.1-3.2_OUTER_ROW; device Teensy_3_and_LC_Series_Boards_v1.4:TEENSY_3.0-3.2&LC_ALL_PINS -> Teensy_3_and_LC_Series_Boards_v1.4:TEENSY_3.0-3.2&LC_OUTER_ROW
- moved U$7 3.00 mm to (33.0, 10.3)
- moved U$8 2.26 mm to (29.8, -0.53), turned to 270 degrees
- moved D1 0.93 mm to (36.0, 24.4), turned to 270 degrees
Connections:
- removed net AREF: U$2.AREF
- removed net VUSB: U$2.VUSB
Routing:
- net V_BCKP: track 23.9 -> 16.2 mm, vias 0 -> 2
- net +3V3: track 65.0 -> 62.0 mm, vias 1 -> 2
- net N$4: track 4.90 -> 6.15 mm
- net N$1: track 4.05 -> 2.89 mm
- net N$3: track 6.64 -> 7.66 mm
Other:
- board size 45 x 45 mm -> 45 x 49.7 mm

Commit message: More stuff, close, not done
Parts:
- added X1: 53261-04, con-molex:53261-04
Connections:
- new net N$8: X1.2
- new net N$9: X1.3
- net +3V3: now also X1.1
- net GND: now also X1.4
Changed lines of the file:
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@@
 <attribute name="VALUE" x="18.161" y="7.0358" size="1.27" layer="27" rot="R270"/>
+</element>
+<element name="X1" library="con-molex" library_urn="urn:adsk.eagle:library:165" package="53261-04" value="53261-04" x="-1.524" y="-9.652" smashed="yes">
+<attribute name="MF" value="MOLEX" x="-1.524" y="-9.652" size="1.778" layer="27" display="off"/>
+<attribute name="MPN" value="" x="-1.524" y="-9.652" size="1.778" layer="27" display="off"/>
+<attribute name="NAME" x="-4.649" y="-6.777" size="1.27" layer="25"/>
+<attribute name="OC_FARNELL" value="1125374" x="-1.524" y="-9.652" size="1.778" layer="27" display="off"/>
+<attribute name="OC_NEWARK" value="unknown" x="-1.524" y="-9.652" size="1.778" layer="27" display="off"/>
+<attribute name="VALUE" x="-4.274" y="-10.152" size="1.27" layer="27"/>
 </element>
 </elements>
@@
 <via x="15.494" y="40.386" extent="1-16" drill="0.35"/>
 <via x="30.226" y="18.288" extent="1-16" drill="0.35"/>
+<contactref element="X1" pad="4"/>
+<wire x1="31.374" y1="39.836" x2="37.3126" y2="38.3032" width="0" layer="19" extent="1-1"/>
+<wire x1="26.8732" y1="42.926" x2="31.374" y2="39.836" width="0" layer="19" extent="1-1"/>
+<wire x1="27.686" y1="35.2298" x2="31.374" y2="39.836" width="0" layer="19" extent="1-1"/>
+<wire x1="29.6418" y1="29.5402" x2="27.686" y2="35.2298" width="0" layer="19" extent="1-1"/>
+<wire x1="33.659175" y1="30.085825" x2="29.6418" y2="29.5402" width="0" layer="19" extent="1-1"/>
+<wire x1="36.8808" y1="27.051" x2="33.659175" y2="30.085825" width="0" layer="19" extent="1-1"/>
+<wire x1="41.021" y1="27.9908" x2="36.8808" y2="27.051" width="0" layer="19" extent="1-1"/>
+<wire x1="35.179" y1="22.5298" x2="36.8808" y2="27.051" width="0" layer="19" extent="1-1"/>
+<wire x1="35.7124" y1="18.1356" x2="35.179" y2="22.5298" width="0" layer="19" extent="1-1"/>
+<wire x1="37.366125" y1="15.225375" x2="35.7124" y2="18.1356" width="0" layer="19" extent="1-1"/>
+<wire x1="36.6776" y1="12.954" x2="37.366125" y2="15.225375" width="0" layer="19" extent="1-1"/>
+<wire x1="30.226" y1="18.288" x2="35.7124" y2="18.1356" width="0" layer="19" extent="1-1"/>
+<wire x1="28.6808" y1="19.122" x2="30.226" y2="18.288" width="0" layer="19" extent="1-1"/>
+<wire x1="27.4628" y1="19.7662" x2="28.6808" y2="19.122" width="0" layer="19" extent="1-1"/>
+<wire x1="29.2608" y1="20.5994" x2="28.6808" y2="19.122" width="0" layer="19" extent="1-1"/>
+<wire x1="25.5524" y1="23.495" x2="27.4628" y2="19.7662" width="0" layer="19" extent="1-1"/>
+<wire x1="41.3512" y1="19.4818" x2="35.7124" y2="18.1356" width="0" layer="19" extent="1-1"/>
+<wire x1="21.525" y1="17.225" x2="27.4628" y2="19.7662" width="0" layer="19" extent="1-1"/>
+<wire x1="22.0472" y1="15.367" x2="21.525" y2="17.225" width="0" layer="19" extent="1-1"/>
+<wire x1="19.4056" y1="18.5674" x2="21.525" y2="17.225" width="0" layer="19" extent="1-1"/>
+<wire x1="16.5608" y1="21.7678" x2="19.4056" y2="18.5674" width="0" layer="19" extent="1-1"/>
+<wire x1="16.8124" y1="24.0768" x2="16.5608" y2="21.7678" width="0" layer="19" extent="1-1"/>
+<wire x1="13.5185" y1="27.82355" x2="14.72475" y2="24.3054" width="0" layer="19" extent="1-1"/>
+<wire x1="11.330775" y1="27.791475" x2="13.5185" y2="27.82355" width="0" layer="19" extent="1-1"/>
+<wire x1="11.321875" y1="29.774925" x2="11.330775" y2="27.791475" width="0" layer="19" extent="1-1"/>
+<wire x1="8.271875" y1="29.674925" x2="11.321875" y2="29.774925" width="0" layer="19" extent="1-1"/>
+<wire x1="16.221875" y1="29.774925" x2="13.5185" y2="27.82355" width="0" layer="19" extent="1-1"/>
+<wire x1="17.0942" y1="34.1376" x2="16.221875" y2="29.774925" width="0" layer="19" extent="1-1"/>
+<wire x1="16.8402" y1="14.7828" x2="19.4056" y2="18.5674" width="0" layer="19" extent="1-1"/>
+<wire x1="14.63755" y1="10.862975" x2="16.8402" y2="14.7828" width="0" layer="19" extent="1-1"/>
+<wire x1="12.6658" y1="13.018775" x2="14.63755" y2="10.862975" width="0" layer="19" extent="1-1"/>
+<wire x1="9.631525" y1="14.104975" x2="12.6658" y2="13.018775" width="0" layer="19" extent="1-1"/>
+<wire x1="9.631525" y1="15.120975" x2="9.631525" y2="14.104975" width="0" layer="19" extent="1-1"/>
+<wire x1="8.615525" y1="15.120975" x2="9.631525" y2="15.120975" width="0" layer="19" extent="1-1"/>
+<wire x1="8.615525" y1="14.612975" x2="8.615525" y2="15.120975" width="0" layer="19" extent="1-1"/>
+<wire x1="8.615525" y1="14.104975" x2="8.615525" y2="14.612975" width="0" layer="19" extent="1-1"/>
+<wire x1="7.965525" y1="15.486975" x2="8.615525" y2="15.120975" width="0" layer="19" extent="1-1"/>
+<wire x1="7.599525" y1="14.104975" x2="8.615525" y2="14.104975" width="0" layer="19" extent="1-1"/>
+<wire x1="11.408625" y1="8.503575" x2="14.63755" y2="10.862975" width="0" layer="19" extent="1-1"/>
+<wire x1="18.0608" y1="8.1636" x2="14.63755" y2="10.862975" width="0" layer="19" extent="1-1"/>
+<wire x1="17.5514" y1="5.1816" x2="18.0608" y2="8.1636" width="0" layer="19" extent="1-1"/>
+<wire x1="21.0566" y1="10.1854" x2="18.0608" y2="8.1636" width="0" layer="19" extent="1-1"/>
+<wire x1="17.3736" y1="1.2954" x2="17.5514" y2="5.1816" width="0" layer="19" extent="1-1"/>
+<wire x1="21.6662" y1="5.2832" x2="17.5514" y2="5.1816" width="0" layer="19" extent="1-1"/>
+<wire x1="23.754" y1="6.816" x2="21.6662" y2="5.2832" width="0" layer="19" extent="1-1"/>
+<wire x1="26.416" y1="7.0612" x2="23.754" y2="6.816" width="0" layer="19" extent="1-1"/>
+<wire x1="28.666125" y1="5.725375" x2="26.416" y2="7.0612" width="0" layer="19" extent="1-1"/>
+<wire x1="30.816125" y1="5.725375" x2="28.666125" y2="5.725375" width="0" layer="19" extent="1-1"/>
+<wire x1="10.938" y1="3.429" x2="11.408625" y2="8.503575" width="0" layer="19" extent="1-1"/>
+<wire x1="8.938" y1="3.429" x2="10.938" y2="3.429" width="0" layer="19" extent="1-1"/>
+<wire x1="4.3434" y1="5.6642" x2="8.938" y2="3.429" width="0" layer="19" extent="1-1"/>
+<wire x1="1.68115" y1="8.47165" x2="4.3434" y2="5.6642" width="0" layer="19" extent="1-1"/>
+<wire x1="1.686125" y1="11.82605" x2="1.68115" y2="8.47165" width="0" layer="19" extent="1-1"/>
+<wire x1="26.543" y1="12.3698" x2="26.416" y2="7.0612" width="0" layer="19" extent="1-1"/>
+<wire x1="1.7005" y1="17.859025" x2="1.686125" y2="11.82605" width="0" layer="19" extent="1-1"/>
+<wire x1="15.494" y1="40.386" x2="17.0942" y2="34.1376" width="0" layer="19" extent="1-1"/>
+<wire x1="15.421875" y1="42.474925" x2="15.494" y2="40.386" width="0" layer="19" extent="1-1"/>
+<wire x1="19.721875" y1="41.974925" x2="15.421875" y2="42.474925" width="0" layer="19" extent="1-1"/>
+<wire x1="2.6416" y1="34.7472" x2="8.271875" y2="29.674925" width="0" layer="19" extent="1-1"/>
+<wire x1="6.371875" y1="41.974925" x2="2.6416" y2="34.7472" width="0" layer="19" extent="1-1"/>
+<wire x1="-3.399" y1="-12.152" x2="4.3434" y2="5.6642" width="0" layer="19" extent="1-1"/>
 </signal>
 <signal name="+3V3">
@@
 <wire x1="40.04454375" y1="14.00085" x2="38.994" y2="12.95030625" width="0.4064" layer="16"/>
 <wire x1="40.04454375" y1="17.41115" x2="40.04454375" y2="14.00085" width="0.4064" layer="16"/>
+<contactref element="X1" pad="1"/>
+<wire x1="11.330775" y1="26.091475" x2="13.5185" y2="26.12355" width="0" layer="19" extent="1-1"/>
+<wire x1="14.72475" y1="23.0554" x2="13.5185" y2="26.12355" width="0" layer="19" extent="1-1"/>
+<wire x1="11.955875" y1="21.956075" x2="14.72475" y2="23.0554" width="0" layer="19" extent="1-1"/>
+<wire x1="12.7027" y1="17.97535" x2="11.955875" y2="21.956075" width="0" layer="19" extent="1-1"/>
+<wire x1="0.351" y1="-12.152" x2="12.7027" y2="17.97535" width="0" layer="19" extent="1-1"/>
 </signal>
 <signal name="MOSI">
@@
 <contactref element="U$2" pad="VBAT"/>
 </signal>
+<signal name="N$8">
+<contactref element="X1" pad="2"/>
+</signal>
+<signal name="N$9">
+<contactref element="X1" pad="3"/>
+</signal>
 </signals>
 <mfgpreviewcolors>
@@
 </board>
 </drawing>
+<compatibility>
+<note version="8.2" severity="warning">
+Since Version 8.2, EAGLE supports online libraries. The ids
+of those online libraries will not be understood (or retained)
+with this version.
+</note>
+</compatibility>
 </eagle>

Commit message: Finishing touches for Cell3.2
Parts:
- moved X1 42.7 mm to (3.05, 32.8), flipped to the bottom, turned to 270 degrees
- turned U$1 to 0 degrees
Connections:
- removed net N$8: X1.2
- removed net N$9: X1.3
- new net IN_B: U$2.15/A1, X1.3
- new net OUT_A: U$2.14/A0, X1.2
Routing:
- net OUT_A: track 0.00 -> 39.7 mm
- net IN_B: track 0.00 -> 34.7 mm
- net +3V3: track 62.0 -> 70.3 mm, vias 2 -> 3
- net IN1: track 5.22 -> 0.28 mm
- net N$33: track 6.01 -> 10.0 mm
- net N$7: track 4.96 -> 2.79 mm

Commit message: Finalizing BITS v3.2
Parts:
- removed LED2: Green, led:CHIP-LED0603
- removed R10: 470, resistor:R0603
- moved C5 53.1 mm to (55.3, -1.24), turned to 270 degrees
- moved C3 50.6 mm to (51.9, -1.23), turned to 270 degrees
- moved U$1 48.6 mm to (60.3, 7.62), turned to 90 degrees
- moved R21 48.3 mm to (55.3, 3.01), turned to 270 degrees
- moved C2 47.4 mm to (48.8, -0.32), turned to 90 degrees
- moved D3 46.5 mm to (45.9, -0.92), turned to 90 degrees
- moved R20 44.7 mm to (55.3, 6.24), turned to 270 degrees
- moved X1 44.0 mm to (31.0, -1.27), turned to 180 degrees
- moved U$8 43.2 mm to (64.3, 25.5), turned to 0 degrees
- moved U1 41.8 mm to (49.1, 4.30), turned to 90 degrees
- moved R1 41.4 mm to (55.1, 9.41), turned to 90 degrees
- moved R17 39.1 mm to (52.9, 9.47), turned to 270 degrees
- moved R3 38.7 mm to (55.6, 12.9), turned to 270 degrees
- moved R5 38.4 mm to (57.4, 15.7), turned to 0 degrees
- moved R19 37.6 mm to (49.9, 8.35), turned to 180 degrees
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Connections:
- removed net LED2: R10.1, U$2.3
- removed net N$5: LED2.A, R10.2
- net GND: no longer LED2.C
- net NETAV: now also U$2.3
Routing:
- net NETAV: track 0.00 -> 9.32 mm, vias 0 -> 1
- net TX3: track 11.3 -> 17.6 mm
- net RX3: track 10.9 -> 16.3 mm
- net N$3: track 7.66 -> 2.65 mm
- net +3V3: track 70.3 -> 74.5 mm
- net N$4: track 6.15 -> 2.07 mm
- net IN1: track 0.28 -> 4.28 mm
- net LED2: track 2.21 -> 0.00 mm
- net N$7: track 2.79 -> 4.96 mm
- net N$5: track 1.28 -> 0.00 mm
- net GND: track 4.98 -> 4.73 mm, vias 34 -> 38
Other:
- board size 45 x 49.7 mm -> 49.7 x 44.5 mm
- board text added: "2S LiPo"
- board text added: "3V3>"
- board text added: "</CMD>"
- board text added: "BITS v3.2"
- board text added: "BPP"
- board text added: "GND GND LED VIN"
- board text added: "GND>"
- board text added: "Isolated Conn GND IN_B OUT_A 3V3"
- board text removed: "BITS V3.2"
- board text removed: "GND"
- board text removed: "Vin"

Commit message: Final board export/cam, code libraries fld
Other:
- board size 49.7 x 44.5 mm -> 50 x 44.7 mm
Changed lines of the file:
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@@
 <board>
 <plain>
-<wire x1="62.208" y1="40.374" x2="21.008" y2="40.374" width="0.0254" layer="20"/>
 <hole x="60.604" y="-1.168" drill="2.5"/>
 <hole x="21.396" y="-1.168" drill="2.5"/>
@@
 <hole x="21.396" y="37.532" drill="2.5"/>
 <circle x="21.396" y="37.532" radius="2.5" width="0.0254" layer="21"/>
-<wire x1="18.754" y1="38.628" x2="18.754" y2="-2.372" width="0.0254" layer="20"/>
-<wire x1="20.754" y1="-4.118" x2="61.954" y2="-4.118" width="0.0254" layer="20"/>
-<wire x1="20.754" y1="-4.118" x2="18.754" y2="-2.372" width="0.0254" layer="20" curve="-90"/>
-<wire x1="18.754" y1="38.628" x2="21.008" y2="40.374" width="0.0254" layer="20" curve="-90"/>
-<wire x1="62.208" y1="40.374" x2="63.754" y2="38.682" width="0.0254" layer="20" curve="-90"/>
-<wire x1="63.754" y1="-2.318" x2="61.954" y2="-4.118" width="0.0254" layer="20" curve="-90"/>
 <text x="34.5102" y="-1.1052" size="2.54" layer="21" font="vector" align="center">BITS v3.2</text>
-<wire x1="63.754" y1="-2.286" x2="63.754" y2="22.606" width="0.0254" layer="20"/>
-<wire x1="63.754" y1="22.606" x2="65.151" y2="24.0792" width="0.0254" layer="20" curve="-90"/>
-<wire x1="65.151" y1="24.0792" x2="68.199" y2="24.0792" width="0.0254" layer="20"/>
-<wire x1="68.199" y1="24.0792" x2="68.4784" y2="24.3586" width="0.0254" layer="20" curve="90"/>
-<wire x1="68.4784" y1="24.3586" x2="68.4784" y2="26.6446" width="0.0254" layer="20"/>
-<wire x1="68.4784" y1="26.6446" x2="68.2752" y2="26.8986" width="0.0254" layer="20" curve="90"/>
-<wire x1="68.2752" y1="26.8986" x2="65.2272" y2="26.8986" width="0.0254" layer="20"/>
-<wire x1="65.2272" y1="26.8986" x2="63.754" y2="28.448" width="0.0254" layer="20" curve="-90"/>
-<wire x1="63.754" y1="28.448" x2="63.754" y2="38.862" width="0.0254" layer="20"/>
 <text x="52.324" y="38.608" size="0.8128" layer="22" rot="MR270">3V3&gt;</text>
 <text x="57.404" y="23.368" size="0.8128" layer="22" rot="MR270">GND&gt;</text>
 <text x="27.686" y="24.13" size="0.8128" layer="22" rot="MR0">3V3&gt;</text>
 <text x="24.638" y="27.432" size="0.8128" layer="22" rot="MR180">GND&gt;</text>
-<text x="29.972" y="6.858" size="0.8128" layer="22" rot="MR270">Isolated Conn
+<text x="26.416" y="10.668" size="0.8128" layer="22" rot="MR270">Isolated Conn
 GND
 IN_B
 OUT_A
 3V3</text>
-<text x="56.642" y="30.988" size="2.54" layer="22" ratio="4" rot="MR270">&lt;/CMD&gt;</text>
-<text x="53.34" y="26.416" size="1.778" layer="22" ratio="15" rot="MR270">BPP</text>
-<text x="63.246" y="21.59" size="1.27" layer="21" rot="R180">GND
+<text x="55.88" y="34.29" size="2.54" layer="22" ratio="4" rot="MR270">&lt;/CMD&gt;</text>
+<text x="52.832" y="29.718" size="1.778" layer="22" ratio="15" rot="MR270">BPP</text>
+<text x="61.722" y="18.542" size="0.8128" layer="21" rot="R180">GND
 GND
 LED
 VIN</text>
 <text x="56.134" y="12.954" size="1.778" layer="22" rot="MR270">2S LiPo</text>
+<wire x1="21.59" y1="-4.318" x2="60.706" y2="-4.318" width="0.0762" layer="20"/>
+<wire x1="60.706" y1="-4.318" x2="63.754" y2="-1.27" width="0.0762" layer="20" curve="90"/>
+<wire x1="63.754" y1="-1.27" x2="63.754" y2="14.224" width="0.0762" layer="20"/>
+<wire x1="63.754" y1="14.224" x2="62.992" y2="14.224" width="0.0762" layer="20"/>
+<wire x1="62.992" y1="14.224" x2="62.23" y2="14.986" width="0.0762" layer="20" curve="-90"/>
+<wire x1="62.23" y1="14.986" x2="62.23" y2="17.78" width="0.0762" layer="20"/>
+<wire x1="62.23" y1="17.78" x2="60.96" y2="19.05" width="0.0762" layer="20" curve="90"/>
+<wire x1="60.96" y1="19.05" x2="60.706" y2="19.05" width="0.0762" layer="20"/>
+<wire x1="60.706" y1="19.05" x2="59.436" y2="20.32" width="0.0762" layer="20" curve="-90"/>
+<wire x1="59.436" y1="20.32" x2="59.436" y2="22.606" width="0.0762" layer="20"/>
+<wire x1="59.436" y1="22.606" x2="60.452" y2="23.622" width="0.0762" layer="20" curve="-90"/>
+<wire x1="60.452" y1="23.622" x2="67.818" y2="23.622" width="0.0762" layer="20"/>
+<wire x1="67.818" y1="23.622" x2="68.58" y2="24.384" width="0.0762" layer="20" curve="90"/>
+<wire x1="68.58" y1="24.384" x2="68.58" y2="26.416" width="0.0762" layer="20"/>
+<wire x1="68.58" y1="26.416" x2="67.818" y2="27.178" width="0.0762" layer="20" curve="90"/>
+<wire x1="67.818" y1="27.178" x2="59.944" y2="27.178" width="0.0762" layer="20"/>
+<wire x1="59.944" y1="27.178" x2="59.69" y2="27.432" width="0.0762" layer="20" curve="-90"/>
+<wire x1="59.69" y1="27.432" x2="59.69" y2="33.782" width="0.0762" layer="20"/>
+<wire x1="59.69" y1="33.782" x2="60.706" y2="34.798" width="0.0762" layer="20" curve="-90"/>
+<wire x1="60.706" y1="34.798" x2="60.96" y2="34.798" width="0.0762" layer="20"/>
+<wire x1="60.96" y1="34.798" x2="63.5" y2="37.338" width="0.0762" layer="20" curve="90"/>
+<wire x1="63.5" y1="37.338" x2="60.452" y2="40.386" width="0.0762" layer="20" curve="90"/>
+<wire x1="60.452" y1="40.386" x2="21.336" y2="40.386" width="0.0762" layer="20"/>
+<wire x1="21.336" y1="40.386" x2="18.542" y2="37.592" width="0.0762" layer="20" curve="90"/>
+<wire x1="18.542" y1="37.592" x2="18.542" y2="-1.27" width="0.0762" layer="20"/>
+<wire x1="18.542" y1="-1.27" x2="21.59" y2="-4.318" width="0.0762" layer="20" curve="90"/>
 </plain>
 <attributes>

Commit message: Handling R values
Parts:
- R18: value 45k -> 170k
- R19: value 13.3k -> 50k
- R20: value 39k -> 30.1k
- R21: value 195k -> 140k
Changed lines of the file:
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@@
 <attribute name="VALUE" x="34.812925" y="11.317875" size="1.27" layer="25" rot="R270"/>
 </element>
-<element name="R18" library="resistor" package="R0603" value="45k" x="46.62865" y="8.3847" smashed="yes" rot="R180">
+<element name="R18" library="resistor" package="R0603" value="170k" x="46.62865" y="8.3847" smashed="yes" rot="R180">
 <attribute name="NAME" x="47.26365" y="7.7497" size="1.27" layer="25" rot="R180"/>
 <attribute name="VALUE" x="47.26365" y="10.2897" size="1.27" layer="27" rot="R180"/>
 </element>
-<element name="R19" library="resistor" package="R0603" value="13.3k" x="49.885225" y="8.3478" smashed="yes" rot="R180">
+<element name="R19" library="resistor" package="R0603" value="50k" x="49.885225" y="8.3478" smashed="yes" rot="R180">
 <attribute name="NAME" x="50.520225" y="7.7128" size="1.27" layer="25" rot="R180"/>
 <attribute name="VALUE" x="50.520225" y="10.2528" size="1.27" layer="27" rot="R180"/>
@@
 <attribute name="VALUE" x="49.069975" y="-4.0907" size="1.27" layer="27" rot="R90"/>
 </element>
-<element name="R20" library="resistor" package="R0603" value="39k" x="55.250425" y="6.240625" smashed="yes" rot="R270">
+<element name="R20" library="resistor" package="R0603" value="30.1k" x="55.250425" y="6.240625" smashed="yes" rot="R270">
 <attribute name="NAME" x="55.885425" y="6.875625" size="1.27" layer="25" rot="R270"/>
 <attribute name="VALUE" x="53.345425" y="6.875625" size="1.27" layer="27" rot="R270"/>
 </element>
-<element name="R21" library="resistor" package="R0603" value="195k" x="55.26315" y="3.005275" smashed="yes" rot="R270">
+<element name="R21" library="resistor" package="R0603" value="140k" x="55.26315" y="3.005275" smashed="yes" rot="R270">
 <attribute name="NAME" x="55.89815" y="3.640275" size="1.27" layer="25" rot="R270"/>
 <attribute name="VALUE" x="53.35815" y="3.640275" size="1.27" layer="27" rot="R270"/>

Commit message: minor R val changes, STEP generation
Parts:
- R18: value 170k -> 340k
- R19: value 50k -> 100k
Changed lines of the file:
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@@
 <attribute name="VALUE" x="34.812925" y="11.317875" size="1.27" layer="25" rot="R270"/>
 </element>
-<element name="R18" library="resistor" package="R0603" value="170k" x="46.62865" y="8.3847" smashed="yes" rot="R180">
+<element name="R18" library="resistor" package="R0603" value="340k" x="46.62865" y="8.3847" smashed="yes" rot="R180">
 <attribute name="NAME" x="47.26365" y="7.7497" size="1.27" layer="25" rot="R180"/>
 <attribute name="VALUE" x="47.26365" y="10.2897" size="1.27" layer="27" rot="R180"/>
 </element>
-<element name="R19" library="resistor" package="R0603" value="50k" x="49.885225" y="8.3478" smashed="yes" rot="R180">
+<element name="R19" library="resistor" package="R0603" value="100k" x="49.885225" y="8.3478" smashed="yes" rot="R180">
 <attribute name="NAME" x="50.520225" y="7.7128" size="1.27" layer="25" rot="R180"/>
 <attribute name="VALUE" x="50.520225" y="10.2528" size="1.27" layer="27" rot="R180"/>
