File: Boards/LVC_v2/lvc_v2.sch (EAGLE design)
At the start: 17 parts, among them U1 LMR16020

Commit message: routed lightAPRS LVC
Parts:
- removed U$2: LITEAPRS, NR_connectors:LITEAPRS
- added JP3: (no value), pinhead:PINHD-1X1
Connections:
- net GND: now also JP3.1; no longer U$2.P$2
Changed lines of the file:
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@@
 <part name="FRAME1" library="frames" deviceset="A4L-LOC" device=""/>
 <part name="JP2" library="pinhead" deviceset="PINHD-1X7" device=""/>
-<part name="GND2" library="supply1" deviceset="GND" device=""/>
 <part name="+3V1" library="supply1" deviceset="+3V3" device=""/>
-<part name="U$2" library="NR_connectors" deviceset="LITEAPRS" device=""/>
 <part name="R17" library="resistor" deviceset="R-US_" device="R0603" value="23.3k"/>
 <part name="L1" library="inductors" deviceset="ASPI-6045S-560M-TCT-ND" device=""/>
@@
 <part name="U$3" library="jmolterLib" deviceset="CL-SB-12B-01" device=""/>
 <part name="SUPPLY10" library="supply1" deviceset="GND" device=""/>
+<part name="SUPPLY11" library="supply1" deviceset="GND" device=""/>
+<part name="JP3" library="pinhead" library_urn="urn:adsk.eagle:library:325" deviceset="PINHD-1X1" device="" package3d_urn="urn:adsk.eagle:package:22485/2"/>
 </parts>
 <sheets>
@@
 <attribute name="VALUE" x="237.49" y="132.08" size="1.778" layer="96" rot="R180"/>
 </instance>
-<instance part="GND2" gate="1" x="205.74" y="121.92" smashed="yes">
-<attribute name="VALUE" x="203.2" y="119.38" size="1.778" layer="96"/>
-</instance>
 <instance part="+3V1" gate="G$1" x="243.84" y="127" smashed="yes" rot="R270">
 <attribute name="VALUE" x="238.76" y="129.54" size="1.778" layer="96"/>
 </instance>
-<instance part="U$2" gate="G$1" x="187.96" y="127" smashed="yes"/>
 <instance part="R17" gate="G$1" x="68.58" y="76.2" smashed="yes" rot="R90">
 <attribute name="NAME" x="67.0814" y="72.39" size="1.778" layer="95" rot="R90"/>
@@
 <instance part="SUPPLY10" gate="1" x="50.8" y="50.8" smashed="yes">
 <attribute name="VALUE" x="48.895" y="47.625" size="1.778" layer="96"/>
+</instance>
+<instance part="SUPPLY11" gate="1" x="213.36" y="109.22" smashed="yes">
+<attribute name="VALUE" x="210.947" y="106.553" size="1.778" layer="96"/>
+</instance>
+<instance part="JP3" gate="G$1" x="200.66" y="111.76" smashed="yes" rot="R180">
+<attribute name="NAME" x="207.01" y="108.585" size="1.778" layer="95" rot="R180"/>
+<attribute name="VALUE" x="207.01" y="116.84" size="1.778" layer="96" rot="R180"/>
 </instance>
 </instances>
@@
 <net name="GND" class="0">
 <segment>
-<wire x1="198.12" y1="124.46" x2="205.74" y2="124.46" width="0.1524" layer="91"/>
-<pinref part="GND2" gate="1" pin="GND"/>
-<pinref part="U$2" gate="G$1" pin="P$2"/>
-</segment>
-<segment>
 <pinref part="C3" gate="G$1" pin="2"/>
 <pinref part="SUPPLY2" gate="1" pin="GND"/>
@@
 <pinref part="SUPPLY10" gate="1" pin="GND"/>
 <wire x1="50.8" y1="60.96" x2="50.8" y2="53.34" width="0.1524" layer="91"/>
+</segment>
+<segment>
+<pinref part="JP3" gate="G$1" pin="1"/>
+<pinref part="SUPPLY11" gate="1" pin="GND"/>
+<wire x1="203.2" y1="111.76" x2="213.36" y2="111.76" width="0.1524" layer="91"/>
 </segment>
 </net>
@@
 which will not be processed correctly with this version.
 </note>
+<note version="8.2" severity="warning">
+Since Version 8.2, EAGLE supports online libraries. The ids
+of those online libraries will not be understood (or retained)
+with this version.
+</note>
+<note version="8.3" severity="warning">
+Since Version 8.3, EAGLE supports URNs for individual library
+assets (packages, symbols, and devices). The URNs of those assets
+will not be understood (or retained) with this version.
+</note>
+<note version="8.3" severity="warning">
+Since Version 8.3, EAGLE supports the association of 3D packages
+with devices in libraries, schematics, and board files. Those 3D
+packages will not be understood (or retained) with this version.
+</note>
 </compatibility>
