File: Boards/LoRa/SimplePayload/SimplePayload.sch (EAGLE design)
At the start: 10 parts, among them SW1 SPST_TACT-KMR2, U1 RFM95W, X1 32.768

Commit message: box fixes
Parts:
- added U$4: MICRO_SD, NR_connectors:MICRO_SD
Connections:
- new net SD_CS: U$4.CD
- net +3V3: now also U$4.VDD
- net GND: now also U$4.CD1, U$4.G1, U$4.G2, U$4.G3, U$4.G4, U$4.VSS
- net MISO: now also U$4.DAT0
- net MOSI: now also U$4.CMD
- net SCK: now also U$4.CLK
Other:
- note added: "SD Card"
Changed lines of the file:
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@@
 <layer number="112" name="tSilk" color="7" fill="1" visible="yes" active="yes"/>
 <layer number="113" name="ReferenceLS" color="7" fill="1" visible="yes" active="yes"/>
+<layer number="114" name="ANT" color="7" fill="1" visible="yes" active="yes"/>
+<layer number="115" name="usb" color="7" fill="1" visible="yes" active="yes"/>
 <layer number="116" name="Patch_BOT" color="7" fill="1" visible="yes" active="yes"/>
+<layer number="117" name="BACKMAAT1" color="7" fill="1" visible="yes" active="yes"/>
 <layer number="118" name="Rect_Pads" color="7" fill="1" visible="yes" active="yes"/>
+<layer number="119" name="KAP_TEKEN" color="7" fill="1" visible="yes" active="yes"/>
+<layer number="120" name="KAP_MAAT1" color="7" fill="1" visible="yes" active="yes"/>
 <layer number="121" name="sName" color="7" fill="1" visible="yes" active="yes"/>
 <layer number="122" name="_bPlace" color="7" fill="1" visible="yes" active="yes"/>
@@
 <layer number="128" name="_bValues" color="7" fill="1" visible="yes" active="yes"/>
 <layer number="129" name="Mask" color="7" fill="1" visible="yes" active="yes"/>
+<layer number="130" name="SMDSTROOK" color="7" fill="1" visible="yes" active="yes"/>
 <layer number="131" name="tAdjust" color="7" fill="1" visible="yes" active="yes"/>
 <layer number="132" name="bAdjust" color="7" fill="1" visible="yes" active="yes"/>
+<layer number="133" name="bottom_silk" color="7" fill="1" visible="yes" active="yes"/>
 <layer number="144" name="Drill_legend" color="7" fill="1" visible="yes" active="yes"/>
+<layer number="145" name="DrillLegend_01-02" color="7" fill="1" visible="yes" active="yes"/>
+<layer number="146" name="DrillLegend_01-15" color="7" fill="1" visible="yes" active="yes"/>
+<layer number="147" name="DrillLegend_01-16" color="7" fill="1" visible="yes" active="yes"/>
+<layer number="148" name="DrillLegend_01-20" color="7" fill="1" visible="yes" active="yes"/>
+<layer number="149" name="DrillLegend_02-15" color="7" fill="1" visible="yes" active="yes"/>
 <layer number="150" name="Notes" color="7" fill="1" visible="yes" active="yes"/>
 <layer number="151" name="HeatSink" color="7" fill="1" visible="yes" active="yes"/>
@@
 <part name="GND11" library="supply1" library_urn="urn:adsk.eagle:library:371" deviceset="GND" device=""/>
 <part name="C4" library="adafruit" deviceset="C-US" device="C0805" value="10uF"/>
+<part name="U$4" library="NR_connectors" deviceset="MICRO_SD" device=""/>
+<part name="GND12" library="supply1" deviceset="GND" device=""/>
+<part name="+3V4" library="supply1@1" deviceset="+3V3" device=""/>
+<part name="GND13" library="supply1" deviceset="GND" device=""/>
 </parts>
 <sheets>
 <sheet>
 <plain>
+<text x="209.55" y="137.414" size="6.4516" layer="97">SD Card</text>
 </plain>
 <instances>
@@
 <attribute name="NAME" x="196.596" y="24.765" size="1.778" layer="95"/>
 <attribute name="VALUE" x="196.596" y="19.939" size="1.778" layer="96"/>
+</instance>
+<instance part="U$4" gate="G$1" x="229.87" y="112.014" smashed="yes"/>
+<instance part="GND12" gate="1" x="247.65" y="96.774" smashed="yes">
+<attribute name="VALUE" x="241.3" y="97.536" size="1.778" layer="96"/>
+</instance>
+<instance part="+3V4" gate="G$1" x="207.01" y="119.634" smashed="yes">
+<attribute name="VALUE" x="204.724" y="115.062" size="1.778" layer="96"/>
+</instance>
+<instance part="GND13" gate="1" x="207.01" y="104.394" smashed="yes">
+<attribute name="VALUE" x="205.994" y="107.188" size="1.778" layer="96"/>
 </instance>
 </instances>
@@
 <wire x1="137.16" y1="35.56" x2="152.4" y2="35.56" width="0.1524" layer="91"/>
 </segment>
+<segment>
+<pinref part="U$4" gate="G$1" pin="G1"/>
+<wire x1="245.11" y1="132.334" x2="247.65" y2="132.334" width="0.1524" layer="91"/>
+<wire x1="247.65" y1="132.334" x2="247.65" y2="127.254" width="0.1524" layer="91"/>
+<pinref part="U$4" gate="G$1" pin="G2"/>
+<wire x1="247.65" y1="127.254" x2="247.65" y2="122.174" width="0.1524" layer="91"/>
+<wire x1="247.65" y1="122.174" x2="247.65" y2="117.094" width="0.1524" layer="91"/>
+<wire x1="247.65" y1="117.094" x2="247.65" y2="112.014" width="0.1524" layer="91"/>
+<wire x1="247.65" y1="112.014" x2="247.65" y2="99.314" width="0.1524" layer="91"/>
+<wire x1="245.11" y1="127.254" x2="247.65" y2="127.254" width="0.1524" layer="91"/>
+<pinref part="U$4" gate="G$1" pin="G3"/>
+<wire x1="245.11" y1="122.174" x2="247.65" y2="122.174" width="0.1524" layer="91"/>
+<pinref part="U$4" gate="G$1" pin="G4"/>
+<wire x1="245.11" y1="117.094" x2="247.65" y2="117.094" width="0.1524" layer="91"/>
+<pinref part="U$4" gate="G$1" pin="CD1"/>
+<wire x1="245.11" y1="112.014" x2="247.65" y2="112.014" width="0.1524" layer="91"/>
+<pinref part="GND12" gate="1" pin="GND"/>
+<junction x="247.65" y="112.014"/>
+<junction x="247.65" y="117.094"/>
+<junction x="247.65" y="122.174"/>
+<junction x="247.65" y="127.254"/>
+</segment>
+<segment>
+<pinref part="U$4" gate="G$1" pin="VSS"/>
+<wire x1="214.63" y1="106.934" x2="207.01" y2="106.934" width="0.1524" layer="91"/>
+<pinref part="GND13" gate="1" pin="GND"/>
+</segment>
 </net>
 <net name="N$2" class="0">
@@
 <wire x1="20.32" y1="83.82" x2="22.86" y2="83.82" width="0.1524" layer="91"/>
 </segment>
+<segment>
+<pinref part="U$4" gate="G$1" pin="VDD"/>
+<wire x1="207.01" y1="117.094" x2="214.63" y2="117.094" width="0.1524" layer="91"/>
+<pinref part="+3V4" gate="G$1" pin="+3V3"/>
+</segment>
 </net>
 <net name="N$3" class="0">
@@
 <label x="20.32" y="43.18" size="1.27" layer="95" rot="R180" xref="yes"/>
 </segment>
+<segment>
+<pinref part="U$4" gate="G$1" pin="CLK"/>
+<wire x1="214.63" y1="112.014" x2="212.09" y2="112.014" width="0.1524" layer="91"/>
+<label x="212.09" y="112.014" size="1.016" layer="95" rot="R180" xref="yes"/>
+</segment>
 </net>
 <net name="MOSI" class="0">
@@
 <label x="20.32" y="45.72" size="1.27" layer="95" rot="R180" xref="yes"/>
 </segment>
+<segment>
+<pinref part="U$4" gate="G$1" pin="CMD"/>
+<wire x1="214.63" y1="122.174" x2="212.09" y2="122.174" width="0.1524" layer="91"/>
+<label x="212.09" y="122.174" size="1.016" layer="95" rot="R180" xref="yes"/>
+</segment>
 </net>
 <net name="MISO" class="0">
@@
 <wire x1="99.06" y1="58.42" x2="101.6" y2="58.42" width="0.1524" layer="91"/>
 <label x="101.6" y="58.42" size="1.27" layer="95" xref="yes"/>
+</segment>
+<segment>
+<pinref part="U$4" gate="G$1" pin="DAT0"/>
+<wire x1="214.63" y1="101.854" x2="212.09" y2="101.854" width="0.1524" layer="91"/>
+<label x="212.09" y="101.854" size="1.016" layer="95" rot="R180" xref="yes"/>
 </segment>
 </net>
@@
 </segment>
 </net>
+<net name="SD_CS" class="0">
+<segment>
+<pinref part="U$4" gate="G$1" pin="CD"/>
+<wire x1="214.63" y1="127.254" x2="212.09" y2="127.254" width="0.1524" layer="91"/>
+<label x="212.09" y="127.254" size="1.016" layer="95" rot="R180" xref="yes"/>
+</segment>
+</net>
