File: Boards/BITSv5/BITSv5/BITSv5.kicad_sch (KiCad schematic)
At the start: 58 parts, among them J1 Conn_01x10_Pin, J2 USB_BOOT, J3 USB_C_Receptacle_USB2.0, U1 MCU_RaspberryPi_RP2040_RP2040, U2 W25Q128JVS, U3 MAX-M10S, U4 MAX77857, U5 TPS610997YFFR, U6 XBee_SMT, Y1 ABLS-12.000MHZ-B4-T

Commit message: BITSv5 updates
Parts:
- removed J2: USB_BOOT, symbol Connector:Conn_01x02_Pin
- added D1: LED, symbol Device:LED
- added J4: Conn_02x05_Counter_Clockwise, symbol Connector_Generic:Conn_02x05_Counter_Clockwise
- added Q1: Q_NMOS_GSD, symbol Device:Q_NMOS_GSD
- added R14: 10K, symbol Device:R
- added R15: R, symbol Device:R
- added SW1, SW2: PTM, symbol Switch:SW_Push
- C30: symbol Device:C -> Device:C_Polarized
- J1: symbol Connector:Conn_01x10_Pin -> Connector_Generic:Conn_01x10
- J3: footprint (none) -> Connector_USB:USB_C_Receptacle_GCT_USB4085
- U4: footprint (none) -> MAX77857:MAX77857-35WLP
- Y1: footprint (none) -> Crystal:Crystal_SMD_HC49-SD
Connections:
- net +3V3: now also R3.2, Q1.3 (D), R14.1; no longer R3.1
- net GND: now also U1.19 (TESTEN), D1.1 (K), SW1.1, SW2.1
- net QSPI_SS: now also R3.1; no longer R3.2
- net at R4.1: now also SW2.2
- net XBEE_DTR: now reaches U6.10 (DIO8/SLEEP_REQUEST)
- net XBEE_RTS: now reaches U6.29 (DIO6/~{RTS})
- net XBEE_DOUT: now reaches U6.3 (DIO13/UART_TX)
- net XBEE_DIN: now reaches U6.4 (DIO14/UART_RX/~{CONFIG})
- net RP2040_SWCLK: now reaches U1.24 (SWCLK)
- net RP2040_SWDIO: now reaches U1.25 (SWD)
- net at U1.26 (RUN): now also R14.2, SW1.2
- new net: Q1.2 (S), R15.1
- new net: D1.2 (A), R15.2
- new net LED: Q1.1 (G)
- no-connect marks 13 -> 32
Other:
- note added: "Debugging Headers"
- note added: "GPS"
- note added: "LED"
- note added: "XBee"
- moved on the sheet: AE1, C1, C10, C11, C12, C2, C23, C24, C25, C26, C27, C28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

Commit message: BITSv5 sch almost done
Parts:
- removed C30: 680uF, symbol Device:C_Polarized
- removed JP1: SolderJumper_3_Open, symbol Jumper:SolderJumper_3_Open
- removed R10: 2.2K, symbol Device:R
- removed R12: R, symbol Device:R
- removed U5: TPS610997YFFR, YFF0006AFAD, symbol TPS610997:TPS610997YFFR
- added C30: 10pF, Capacitor_SMD:C_0402_1005Metric, symbol Device:C
- added C31: 22uF, Capacitor_SMD:C_0805_2012Metric, symbol Device:C
- added C32, C33: 10nF, Capacitor_SMD:C_0603_1608Metric, symbol Device:C
- added C34, C35: 10uF, Capacitor_SMD:C_0603_1608Metric, symbol Device:C
- added C36, C37: 1uF, Capacitor_SMD:C_0603_1608Metric, symbol Device:C
- added J4: Conn_01x02, symbol Connector_Generic:Conn_01x02
- added R14: 20K, Resistor_SMD:R_0603_1608Metric, symbol Device:R
- added R15, R22: 23.7K, Resistor_SMD:R_0603_1608Metric, symbol Device:R_Small
- added R16, R23: 5K, Resistor_SMD:R_0603_1608Metric, symbol Device:R_Small
- added R17: 51.1K, Resistor_SMD:R_0603_1608Metric, symbol Device:R
- added R18: 1.05M, Resistor_SMD:R_0603_1608Metric, symbol Device:R
- added R19: 154K, Resistor_SMD:R_0603_1608Metric, symbol Device:R
- added R20: 510K, Resistor_SMD:R_0603_1608Metric, symbol Device:R
- added R21, R24: 10K, symbol Device:R
- added U10: USBLC6-2SC6, SOT23-6L_STM, symbol USBLC6-2SC6:USBLC6-2SC6
- added U5: TPS61232DRCR, TPS61232:DRC0010G, symbol TPS61232:TPS61232DRCR
- added U7: TPS2121RUXR, RUX0012A, symbol TPS2121:TPS2121RUXR
- added U8: LT6703CDC-3, DFN-3_DC_LIT, symbol LTC6703:LT6703CDC-3-TRPBF
- added U9: TVS1800DRVR, DRV0006A, symbol TVS1800:TVS1800DRVR
- BT1: footprint (none) -> GHOULFootPrints:XT30PW-M
- C1, C10, C11, C12, C15, C16, C2, C26, C27, C28, C29, C3, C4, C5, C6, C7, C8, C9: footprint (none) -> Capacitor_SMD:C_0603_1608Metric
- C13, C14: value 26uF -> 10pF; footprint (none) -> Capacitor_SMD:C_0603_1608Metric
- C17, C18, C20, C21: footprint (none) -> Capacitor_SMD:C_0805_2012Metric
- C19: value 2.2uF -> 470nF; footprint (none) -> Capacitor_SMD:C_0402_1005Metric
- C22: value 470uF -> 2.2uF; footprint (none) -> Capacitor_SMD:C_0402_1005Metric
- C23, C24, C25: value 10uF -> 22uF; footprint (none) -> Capacitor_SMD:C_0805_2012Metric
- D1: footprint (none) -> LED_SMD:LED_0603_1608Metric
- J1: footprint (none) -> Connector_Molex:Molex_PicoBlade_53047-1010_1x10_P1.25mm_Vertical
- J3: renamed from J4; value Conn_02x05_Counter_Clockwise -> Conn_01x06; symbol Connector_Generic:Conn_02x05_Counter_Clockwise -> Connector_Generic:Conn_01x06
- L1: value 1.5uH -> 1uH; footprint (none) -> Inductor_SMD:L_1008_2520Metric
- L2: value 2.2uH -> 1uH; footprint (none) -> 1616_Inductor:IND_XAL4020_4X4_COC-M
- R1, R2, R3, R4, R5, R6, R7, R8: footprint (none) -> Resistor_SMD:R_0603_1608Metric
- R10: renamed from R11; value R -> 50K; footprint (none) -> Resistor_SMD:R_0603_1608Metric
- R11: renamed from R14; footprint (none) -> Resistor_SMD:R_0603_1608Metric
- R12: renamed from R15; value R -> 270; footprint (none) -> Resistor_SMD:R_0603_1608Metric
- R13: value R -> 178K; footprint (none) -> Resistor_SMD:R_0603_1608Metric
- R9: value 2.2K -> 1M; footprint (none) -> Resistor_SMD:R_0603_1608Metric
- Y1: value ABLS-12.000MHZ-B4-T -> 12MHz; footprint Crystal:Crystal_SMD_HC49-SD -> Crystal:Crystal_SMD_2520-4Pin_2.5x2.0mm
- renumbered J3 to J2
Connections:
- net BUCKBOOST_VIO is gone; now on an unnamed net: C22.1, U4.A2 (VIO)
- net IRIDIUM_5V is gone; now on net +5V: J1.8 (Pin_8)
- net +3V3: now also R12.1, R13.1, C30.1, R21.1, R24.1; no longer Q1.3 (D), U4.E1 (FB)
- net +5V: now also C23.1, R9.1, C31.1, U5.3 (VOUT), U5.4 (VOUT), U5.7 (FB); no longer C24.1
- net GND: now also J3.6 (Pin_6), Q1.2 (S), C31.2, C32.2, C33.2, C34.2, C35.2, C36.2, C37.2, R14.2, R16.2, R17.2, R19.2, R23.2, U10.2, U5.11 (GND), U7.12 (GND), U7.3 (CP2), U7.6 (PR1), U7.9 (ST), U8.4 (V-), U9.1 (GND), U9.2 (GND), U9.3 (GND), U9.7 (PAD); no longer D1.1 (K), R13.2
- net GPS_SCL: now also U1.28 (GPIO17), R24.2; no longer R9.2
- net GPS_SDA: now also U1.27 (GPIO16), R21.2
- net IRIDIUM_CTS: now also U1.4 (GPIO2)
- net IRIDIUM_NETAV: now also U1.8 (GPIO6)
- net IRIDIUM_ON/OFF: now also U1.7 (GPIO5)
- net IRIDIUM_RING: now also U1.6 (GPIO4)
- net IRIDIUM_RTS: now also U1.5 (GPIO3)
- net IRIDIUM_RXD: now also U1.3 (GPIO1)
- net IRIDIUM_TXD: now also U1.2 (GPIO0)
- net USB_D+: now also U10.1; no longer J2.A6 (D+), J2.B6 (D+)
- net USB_D-: now also U10.3; no longer J2.A7 (D-), J2.B7 (D-)
- net VCC: now also C24.1, C36.1, U5.10 (VIN), U7.1 (OUT), U7.8 (OUT); no longer BT1.1 (+), C23.1, J2.A4 (VBUS), J2.A9 (VBUS), J2.B4 (VBUS), J2.B9 (VBUS)
- net XBEE_DIN: now also J3.4 (Pin_4), U1.36 (GPIO24)
- net XBEE_DOUT: now also J3.5 (Pin_5), U1.37 (GPIO25)
- net XBEE_DTR: now also J3.3 (Pin_3)
- net XBEE_RTS: now also J3.1 (Pin_1), U1.34 (GPIO22)
- net at L2.2: now also U5.1 (SW), U5.2 (SW)
- net XBEE_DIO4: now reaches J3.2 (Pin_2)
- net XBEE_DIO4: now also U6.24 (DIO4)
- net at C19.1, U4.C1 (VL): now also U4.A1 (SCL), U4.B1 (SDA)
- net XBEE_RESET: now reaches U6.6 (RESET/OD_OUT)
- net XBEE_CTS: now reaches U1.35 (GPIO23)
- net BUCKBOOST_EN renamed LVC_CUTOFF
- net LVC_CUTOFF: now also R20.2, U5.9 (EN), U8.1 (OUT)
- net IRIDIUM_3V7: no longer names the net of J1.9 (Pin_9)
- net RP2040_SWCLK: no longer names the net of U1.24 (SWCLK)
- net RP2040_SWCLK: now also J4.1 (Pin_1)
- net RP2040_SWDIO: no longer names the net of U1.25 (SWD)
- net RP2040_SWDIO: now also J4.2 (Pin_2)
- new net: R22.2, R23.1, U7.4 (OV2)
- new net: C30.2, R13.2, R14.1, U4.E1 (FB)
- new net: R17.1, U7.10 (ILM)
- new net: C33.1, U7.11 (SS)
- new net: R15.2, R16.1, U7.5 (OV1)
- new net: R18.2, R19.1, U8.3 (IN+)
- new net: J2.A7 (D-), J2.B7 (D-), U10.4
- new net: J2.A6 (D+), J2.B6 (D+), U10.6
- new net: R9.2, U5.5 (PG)
- new net: C32.1, U5.6 (SS)
- new net: D1.1 (K), Q1.3 (D)
- new net +BATT: BT1.1 (+), C34.1, C37.1, R18.1, R20.1, R22.1, U7.2 (IN2), U8.2 (V+), U9.4 (IN), U9.5 (IN), U9.6 (IN)
- new net VBUS: C35.1, J2.A4 (VBUS), J2.A9 (VBUS), J2.B4 (VBUS), J2.B9 (VBUS), R15.1, U10.5, U7.7 (IN1)
- no-connect marks 32 -> 31
Other:
- note added: "LVC"
- note added: "Power Mux"
- note added: "RockBlock Connector"
- note added: "XBee Debug"
- note removed: "Debugging Headers"
- note removed: "LiPo"
- note removed: "Rockblock Connector"
- moved on the sheet: AE1, C1, C10, C11, C13, C14, C15, C16, C17, C18, C2, C20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

Commit message: more bits updates
Parts:
- added R25: 15K, Resistor_SMD:R_0603_1608Metric, symbol Device:R
- added R26: 5K, Resistor_SMD:R_0603_1608Metric, symbol Device:R
- added SW3: ~, symbol Switch:SW_SPDT
- R10: footprint Resistor_SMD:R_0603_1608Metric -> Resistor_SMD:R_0402_1005Metric
- R12: value 270 -> 470
Connections:
- net +BATT: now also R25.1
- net GND: now also R26.1, SW3.1 (A)
- net LED: now also U1.9 (GPIO7)
- net LVC_CUTOFF: now also SW3.2 (B); no longer R20.2, U8.1 (OUT)
- net VBAT: now reaches U1.38 (GPIO26_ADC0)
- net VBAT: now also R25.2, R26.2
- new net: R20.2, SW3.3 (C), U8.1 (OUT)
Other:
- note added: "Voltage Divider"
- note added: "XBee Pro SX 900"
- note removed: "XBee"
- moved on the sheet: AE1, BT1, C1, C10, C11, C2, C3, C37, C4, C5, C6, C7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

Commit message: bits v5 board nearly done
Parts:
- removed SW1: PTM, symbol Switch:SW_Push
- added Q2: Q_PMOS_GSD, Package_TO_SOT_SMD:SOT-23, symbol Device:Q_PMOS_GSD
- C1, C10, C11, C2, C3, C4, C5, C6, C7, C8, C9: footprint Capacitor_SMD:C_0603_1608Metric -> Capacitor_SMD:C_0402_1005Metric_Pad0.74x0.62mm_HandSolder
- C12, C13, C14, C15, C16, C26, C27, C28, C29, C32, C33, C34, C35, C36, C37: footprint Capacitor_SMD:C_0603_1608Metric -> Capacitor_SMD:C_0603_1608Metric_Pad1.08x0.95mm_HandSolder
- C17, C18, C20, C21, C23, C24, C25, C31: footprint Capacitor_SMD:C_0805_2012Metric -> Capacitor_SMD:C_0805_2012Metric_Pad1.18x1.45mm_HandSolder
- C19, C22, C30: footprint Capacitor_SMD:C_0402_1005Metric -> Capacitor_SMD:C_0402_1005Metric_Pad0.74x0.62mm_HandSolder
- J1: footprint Connector_Molex:Molex_PicoBlade_53047-1010_1x10_P1.25mm_Vertical -> Connector_Molex:Molex_PicoBlade_53261-1071_1x10-1MP_P1.25mm_Horizontal
- J3: footprint (none) -> Connector_JST:JST_EH_B5B-EH-A_1x05_P2.50mm_Vertical; symbol Connector_Generic:Conn_01x06 -> Connector_Generic:Conn_01x05
- L1: footprint Inductor_SMD:L_1008_2520Metric -> Inductor_SMD:L_1008_2520Metric_Pad1.43x2.20mm_HandSolder
- Q1: footprint (none) -> Package_TO_SOT_SMD:SOT-23-3
- R1, R2, R25, R26, R5: footprint Resistor_SMD:R_0603_1608Metric -> Resistor_SMD:R_0402_1005Metric_Pad0.72x0.64mm_HandSolder
- R10: value 50K -> 48.7K; footprint Resistor_SMD:R_0402_1005Metric -> Resistor_SMD:R_0402_1005Metric_Pad0.72x0.64mm_HandSolder
- R11, R12, R13, R14, R15, R16, R17, R18, R19, R20, R22, R23, R3, R4, R6, R7, R8, R9: footprint Resistor_SMD:R_0603_1608Metric -> Resistor_SMD:R_0603_1608Metric_Pad0.98x0.95mm_HandSolder
- R21, R24: footprint (none) -> Resistor_SMD:R_0603_1608Metric_Pad0.98x0.95mm_HandSolder
- SW2: footprint (none) -> Button_Switch_SMD:SW_Push_1P1T_NO_CK_KMR2
- SW3: value ~ -> SLIDE; footprint (none) -> BITSv5:CL-SB-12B-01_NDC
- U6: footprint RF_Module:Digi_XBee_SMT -> BITSv5:XCVR_XBP9X-DMUS-001; symbol RF_ZigBee:XBee_SMT -> BITSv5:XBP9X-DMUS-001; Check_prices (none) -> https://www.snapeda.com/parts/XBP9X-DMUS-001/Digi+Internati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; DigiKey_Part_Number (none) -> 602-1890-ND; MANUFACTURER (none) -> Digi; MAXIMUM_PACKAGE_HEIGHT (none) -> 3.556mm; MF (none) -> Digi International; MP (none) -> XBP9X-DMUS-001; PARTREV (none) -> K; Package (none) -> Module Digi International; Purchase-URL (none) -> https://pricing.snapeda.com/search?q=XBP9X-DMUS-001&ref=eda; STANDARD (none) -> Manufacturer recommendations; SnapEDA_Link (none) -> https://www.snapeda.com/parts/XBP9X-DMUS-001/Digi+Internati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
- U7: footprint RUX0012A -> BITSv5:TPS2121
- U9: footprint DRV0006A -> BITSv5:TVS1800
- Y1: symbol Device:Crystal -> Device:Crystal_GND24
Connections:
- net +BATT: no longer C37.1, R18.1, R20.1, U8.2 (V+)
- net GND: now also J3.1 (Pin_1), U6.38 (GND), Y1.2, Y1.4, Q2.2 (S); no longer J3.6 (Pin_6)
- net LED: now also U1.29 (GPIO18); no longer U1.9 (GPIO7)
- net VBAT: now also U1.40 (GPIO28_ADC2); no longer U1.38 (GPIO26_ADC0)
- net VCC: now also C37.1, R18.1, R20.1, U8.2 (V+)
- net XBEE_RESET: now also Q2.1 (G)
- net XBEE_RTS: now also J3.2 (Pin_2); no longer J3.1 (Pin_1)
- net XIN: now also Y1.3; no longer Y1.2
- net at R11.2, U1.26 (RUN): now also Q2.3 (D)
- net XBEE_CTS: no longer names the net of U1.35 (GPIO23)
- net XBEE_DIO4: no longer names the net of U6.24 (DIO4)
- net XBEE_DIO4: no longer J3.2 (Pin_2)
- no-connect marks 31 -> 47
Other:
- moved on the sheet: BT1, C1, C10, C11, C14, C2, C23, C24, C25, C26, C27, C28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

Commit message: several hundred bits v5 errors later
Parts:
- removed J4: Conn_01x02, symbol Connector_Generic:Conn_01x02
- BT1: footprint GHOULFootPrints:XT30PW-M -> BITSv5:XT30PW-M
- J3: value Conn_01x06 -> Conn_01x07; footprint Connector_JST:JST_EH_B5B-EH-A_1x05_P2.50mm_Vertical -> Connector_PinSocket_2.54mm:PinSocket_1x07_P2.54mm_Vertical; symbol Connector_Generic:Conn_01x05 -> Connector_Generic:Conn_01x07
- L2: footprint 1616_Inductor:IND_XAL4020_4X4_COC-M -> BITSv5:IND_XAL4020_4X4_COC-M
- U1: footprint RP2040_minimal:RP2040-QFN-56 -> BITSv5:RP2040-QFN-56
- U4: footprint MAX77857:MAX77857-35WLP -> BITSv5:MAX77857-35WLP
- U5: footprint TPS61232:DRC0010G -> BITSv5:TPS61232
- U8: footprint DFN-3_DC_LIT -> BITSv5:DFN-3_DC_LIT
Connections:
- net RP_SWCLK: now reaches U1.24 (SWCLK)
- net RP_SWCLK: now also J3.6 (Pin_6)
- net RP_SWD: now reaches U1.25 (SWD)
- net RP_SWD: now also J3.7 (Pin_7)
Other:
- note added: "Debug Headers"
- note removed: "XBee Debug"
Changed lines of the file:
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@@
     (stroke (width 0) (type default))
   )
-  (wire (pts (xy 336.55 74.93) (xy 349.25 74.93))
-    (stroke (width 0) (type default))
-  )
   (wire (pts (xy 287.02 81.28) (xy 287.02 78.74))
     (stroke (width 0) (type default))
@@
     (stroke (width 0) (type default))
   )
-  (wire (pts (xy 332.74 71.12) (xy 332.74 69.85))
+  (wire (pts (xy 332.74 68.58) (xy 332.74 67.31))
     (stroke (width 0) (type default))
   )
@@
     (stroke (width 0) (type default))
   )
-  (wire (pts (xy 336.55 77.47) (xy 349.25 77.47))
-    (stroke (width 0) (type default))
-  )
   (wire (pts (xy 29.21 219.71) (xy 29.21 220.98))
     (stroke (width 0) (type default))
@@
     (stroke (width 0) (type default))
   )
+  (wire (pts (xy 336.55 69.85) (xy 349.25 69.85))
+    (stroke (width 0) (type default))
+  )
   (wire (pts (xy 374.65 83.82) (xy 387.35 83.82))
     (stroke (width 0) (type default))
@@
     (stroke (width 0) (type default))
   )
-  (wire (pts (xy 332.74 69.85) (xy 349.25 69.85))
-    (stroke (width 0) (type default))
-  )
   (polyline (pts (xy 328.93 64.77) (xy 229.87 64.77))
     (stroke (width 0) (type dash_dot))
@@
     (stroke (width 0) (type dash_dot))
   )
+  (wire (pts (xy 336.55 72.39) (xy 349.25 72.39))
+    (stroke (width 0) (type default))
+  )
   (wire (pts (xy 93.98 21.59) (xy 93.98 36.83))
     (stroke (width 0) (type default))
@@
     (stroke (width 0) (type default))
   )
+  (wire (pts (xy 336.55 80.01) (xy 349.25 80.01))
+    (stroke (width 0) (type default))
+  )
   (wire (pts (xy 391.16 30.48) (xy 391.16 33.02))
     (stroke (width 0) (type default))
@@
     (stroke (width 0) (type default))
   )
-  (wire (pts (xy 336.55 80.01) (xy 349.25 80.01))
-    (stroke (width 0) (type default))
-  )
   (wire (pts (xy 86.36 36.83) (xy 86.36 21.59))
     (stroke (width 0) (type default))
@@
     (stroke (width 0) (type default))
   )
+  (wire (pts (xy 336.55 74.93) (xy 349.25 74.93))
+    (stroke (width 0) (type default))
+  )
   (wire (pts (xy 320.04 121.92) (xy 330.2 121.92))
     (stroke (width 0) (type default))
@@
     (stroke (width 0) (type default))
   )
+  (wire (pts (xy 336.55 82.55) (xy 349.25 82.55))
+    (stroke (width 0) (type default))
+  )
   (wire (pts (xy 285.75 250.19) (xy 285.75 252.73))
     (stroke (width 0) (type default))
@@
     (stroke (width 0) (type default))
   )
+  (wire (pts (xy 332.74 67.31) (xy 349.25 67.31))
+    (stroke (width 0) (type default))
+  )
   (wire (pts (xy 271.78 181.61) (xy 271.78 172.72))
     (stroke (width 0) (type default))
@@
     (stroke (width 0) (type default))
   )
-  (wire (pts (xy 336.55 72.39) (xy 349.25 72.39))
-    (stroke (width 0) (type default))
-  )
   (wire (pts (xy 59.69 21.59) (xy 57.15 21.59))
     (stroke (width 0) (type default))
@@
     (stroke (width 0) (type default))
   )
-  (wire (pts (xy 41.91 125.73) (xy 45.72 125.73))
+  (wire (pts (xy 29.21 125.73) (xy 45.72 125.73))
     (stroke (width 0) (type default))
   )
@@
     (stroke (width 0) (type default))
   )
+  (wire (pts (xy 336.55 77.47) (xy 349.25 77.47))
+    (stroke (width 0) (type default))
+  )
   (wire (pts (xy 119.38 210.82) (xy 119.38 212.09))
     (stroke (width 0) (type default))
@@
     (stroke (width 0) (type default))
   )
-  (wire (pts (xy 41.91 123.19) (xy 45.72 123.19))
+  (wire (pts (xy 29.21 123.19) (xy 45.72 123.19))
     (stroke (width 0) (type default))
   )
@@
     (effects (font (size 4 4)) (justify left bottom))
   )
-  (text "XBee Debug" (at 317.5 95.25 0)
+  (text "Debug\nHeaders" (at 317.5 95.25 0)
     (effects (font (size 4 4)) (justify left bottom))
   )
@@
     (effects (font (size 1.27 1.27)) (justify left bottom))
   )
-  (label "XBEE_DTR" (at 336.55 74.93 0) (fields_autoplaced)
+  (label "XBEE_DTR" (at 336.55 72.39 0) (fields_autoplaced)
     (effects (font (size 1.27 1.27)) (justify left bottom))
   )
@@
     (effects (font (size 1.27 1.27)) (justify left bottom))
   )
-  (label "XBEE_DOUT" (at 336.55 80.01 0) (fields_autoplaced)
+  (label "XBEE_DOUT" (at 336.55 77.47 0) (fields_autoplaced)
+    (effects (font (size 1.27 1.27)) (justify left bottom))
+  )
+  (label "RP_SWCLK" (at 336.55 80.01 0) (fields_autoplaced)
+    (effects (font (size 1.27 1.27)) (justify left bottom))
+  )
+  (label "RP_SWD" (at 336.55 82.55 0) (fields_autoplaced)
     (effects (font (size 1.27 1.27)) (justify left bottom))
   )
@@
     (effects (font (size 1.27 1.27)) (justify left bottom))
   )
-  (label "XBEE_RTS" (at 336.55 72.39 0) (fields_autoplaced)
+  (label "XBEE_RTS" (at 336.55 69.85 0) (fields_autoplaced)
     (effects (font (size 1.27 1.27)) (justify left bottom))
   )
@@
     (effects (font (size 1.27 1.27)) (justify left bottom))
   )
-  (label "XBEE_DIN" (at 336.55 77.47 0) (fields_autoplaced)
+  (label "XBEE_DIN" (at 336.55 74.93 0) (fields_autoplaced)
     (effects (font (size 1.27 1.27)) (justify left bottom))
   )
@@
     (effects (font (size 1.27 1.27)) (justify right bottom))
   )
+  (label "RP_SWCLK" (at 29.21 123.19 0) (fields_autoplaced)
+    (effects (font (size 1.27 1.27)) (justify left bottom))
+  )
   (label "XBEE_DOUT" (at 326.39 207.01 0) (fields_autoplaced)
     (effects (font (size 1.27 1.27)) (justify left bottom))
@@
     (effects (font (size 1.27 1.27)) (justify right bottom))
   )
+  (label "RP_SWD" (at 29.21 125.73 0) (fields_autoplaced)
+    (effects (font (size 1.27 1.27)) (justify left bottom))
+  )
   (label "QSPI_SD2" (at 353.06 43.18 0) (fields_autoplaced)
     (effects (font (size 1.27 1.27)) (justify left bottom))
@@
     )
   )
-  (symbol (lib_id "Connector_Generic:Conn_01x05") (at 354.33 74.93 0) (unit 1)
+  (symbol (lib_id "Connector_Generic:Conn_01x07") (at 354.33 74.93 0) (unit 1)
     (in_bom yes) (on_board yes) (dnp no)
-    (property "Reference" "J3" (at 341.63 83.82 0)
+    (property "Reference" "J3" (at 350.52 87.63 0)
       (effects (font (size 1.27 1.27)) (justify left))
     )
-    (property "Value" "Conn_01x06" (at 336.55 86.36 0)
+    (property "Value" "Conn_01x07" (at 345.44 90.17 0)
       (effects (font (size 1.27 1.27)) (justify left))
     )
-    (property "Footprint" "Connector_JST:JST_EH_B5B-EH-A_1x05_P2.50mm_Vertical" (at 354.33 74.93 0)
+    (property "Footprint" "Connector_PinSocket_2.54mm:PinSocket_1x07_P2.54mm_Vertical" (at 354.33 74.93 0)
       (effects (font (size 1.27 1.27)) hide)
     )
@@
     (pin "4")
     (pin "5")
+    (pin "6")
+    (pin "7")
     (instances
       (project "BITSv5"
@@
       (effects (font (size 1.27 1.27)))
     )
-    (property "Footprint" "1616_Inductor:IND_XAL4020_4X4_COC-M" (at 250.19 172.72 0)
+    (property "Footprint" "BITSv5:IND_XAL4020_4X4_COC-M" (at 250.19 172.72 0)
       (effects (font (size 1.27 1.27)) hide)
     )
@@
       (effects (font (size 1.27 1.27)) (justify left) hide)
     )
-    (property "Footprint" "GHOULFootPrints:XT30PW-M" (at 199.39 22.606 90)
+    (property "Footprint" "BITSv5:XT30PW-M" (at 199.39 22.606 90)
       (effects (font (size 1.27 1.27)) hide)
     )
@@
       (effects (font (size 1.524 1.524)))
     )
-    (property "Footprint" "DFN-3_DC_LIT" (at 260.35 25.4 0)
+    (property "Footprint" "BITSv5:DFN-3_DC_LIT" (at 260.35 25.4 0)
       (effects (font (size 1.27 1.27) italic) hide)
     )
@@
     )
   )
-  (symbol (lib_id "Connector_Generic:Conn_01x02") (at 36.83 123.19 0) (mirror y) (unit 1)
-    (in_bom yes) (on_board yes) (dnp no)
-    (property "Reference" "J4" (at 38.1 129.54 0)
-      (effects (font (size 1.27 1.27)) (justify left))
-    )
-    (property "Value" "Conn_01x02" (at 43.18 132.08 0)
-      (effects (font (size 1.27 1.27)) (justify left))
-    )
-    (property "Footprint" "" (at 36.83 123.19 0)
-      (effects (font (size 1.27 1.27)) hide)
-    )
-    (property "Datasheet" "~" (at 36.83 123.19 0)
-      (effects (font (size 1.27 1.27)) hide)
-    )
-    (pin "1")
-    (pin "2")
-    (instances
-      (project "BITSv5"
-        (path "/55a258d3-b7da-466a-a6cc-38d8142826fc"
-          (reference "J4") (unit 1)
-        )
-      )
-    )
-  )
   (symbol (lib_id "power:+5V") (at 302.26 186.69 0) (unit 1)
     (in_bom yes) (on_board yes) (dnp no) (fields_autoplaced)
@@
     )
   )
-  (symbol (lib_id "power:GND") (at 332.74 71.12 0) (unit 1)
+  (symbol (lib_id "power:GND") (at 332.74 68.58 0) (unit 1)
     (in_bom yes) (on_board yes) (dnp no)
-    (property "Reference" "#PWR062" (at 332.74 77.47 0)
+    (property "Reference" "#PWR062" (at 332.74 74.93 0)
       (effects (font (size 1.27 1.27)) hide)
     )
-    (property "Value" "GND" (at 332.74 74.93 0)
+    (property "Value" "GND" (at 332.74 72.39 0)
       (effects (font (size 1.27 1.27)))
     )
-    (property "Footprint" "" (at 332.74 71.12 0)
+    (property "Footprint" "" (at 332.74 68.58 0)
       (effects (font (size 1.27 1.27)) hide)
     )
-    (property "Datasheet" "" (at 332.74 71.12 0)
+    (property "Datasheet" "" (at 332.74 68.58 0)
       (effects (font (size 1.27 1.27)) hide)
     )
@@
       (effects (font (size 1.27 1.27)) (justify left))
     )
-    (property "Footprint" "RP2040_minimal:RP2040-QFN-56" (at 58.42 87.63 0)
+    (property "Footprint" "BITSv5:RP2040-QFN-56" (at 58.42 87.63 0)
       (effects (font (size 1.27 1.27)) hide)
     )
@@
       (effects (font (size 1.524 1.524)))
     )
-    (property "Footprint" "TPS61232:DRC0010G" (at 250.19 191.77 0)
+    (property "Footprint" "BITSv5:TPS61232" (at 250.19 191.77 0)
       (effects (font (size 1.27 1.27) italic) hide)
     )
@@
       (effects (font (size 1.524 1.524)))
     )
-    (property "Footprint" "MAX77857:MAX77857-35WLP" (at 39.37 201.93 0)
+    (property "Footprint" "BITSv5:MAX77857-35WLP" (at 39.37 201.93 0)
       (effects (font (size 1.27 1.27) italic) hide)
     )
