File: Boards/BITSv5/BITSv5/BITSv5.kicad_sch (KiCad schematic)
At the start: 86 parts, among them J1 Conn_01x10_Pin, J2 USB_C_Receptacle_USB2.0, J3 Conn_01x07, Q1 Q_NMOS_GSD, Q2 Q_PMOS_GSD, SW2 PTM, SW3 SLIDE, U1 MCU_RaspberryPi_RP2040_RP2040, U10 USBLC6-2SC6, U2 W25Q128JVS, U3 MAX-M10S, U4 MAX77857, U5 TPS61232DRCR, U6 XBee_SMT, U7 TPS2121RUXR, U8 LT6703CDC-3, U9 TVS1800DRVR, Y1 12MHz

Commit message: bits v5 board feedback added
Parts:
- AE1: footprint (none) -> BITSv5:ANT_1575AT_JOT-M
- BT1: footprint BITSv5:XT30PW-M -> Connector_AMASS:AMASS_XT30PW-M_1x02_P2.50mm_Horizontal
- SW2: value PTM -> ~; footprint Button_Switch_SMD:SW_Push_1P1T_NO_CK_KMR2 -> BITSv5:CAS-120TB_NDC-M; symbol Switch:SW_Push -> Switch:SW_SPDT
- U10: footprint SOT23-6L_STM -> BITSv5:SOT23-6L_STM-M
Connections:
- net GND: now also SW2.3 (C); no longer SW2.1
- net XBEE_DTR: now also J3.2 (Pin_2); no longer J3.3 (Pin_3)
- net XBEE_RTS: now also J3.3 (Pin_3); no longer J3.2 (Pin_2)
- no-connect marks 47 -> 48
Changed lines of the file:
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@@
   (no_connect (at 391.16 224.79))
   (no_connect (at 196.85 260.35))
+  (no_connect (at 347.98 30.48))
   (no_connect (at 391.16 199.39))
   (no_connect (at 109.22 113.03))
@@
     (stroke (width 0) (type dash_dot))
   )
-  (wire (pts (xy 347.98 30.48) (xy 347.98 31.75))
-    (stroke (width 0) (type default))
-  )
   (wire (pts (xy 19.05 210.82) (xy 29.21 210.82))
     (stroke (width 0) (type default))
@@
     (stroke (width 0) (type default))
   )
+  (wire (pts (xy 336.55 72.39) (xy 349.25 72.39))
+    (stroke (width 0) (type default))
+  )
   (wire (pts (xy 257.81 26.67) (xy 257.81 27.94))
     (stroke (width 0) (type default))
@@
     (stroke (width 0) (type default))
   )
-  (wire (pts (xy 336.55 69.85) (xy 349.25 69.85))
-    (stroke (width 0) (type default))
-  )
   (wire (pts (xy 374.65 83.82) (xy 387.35 83.82))
     (stroke (width 0) (type default))
@@
     (stroke (width 0) (type dash_dot))
   )
+  (wire (pts (xy 342.9 30.48) (xy 342.9 33.02))
+    (stroke (width 0) (type default))
+  )
   (wire (pts (xy 92.71 228.6) (xy 92.71 227.33))
     (stroke (width 0) (type default))
@@
     (stroke (width 0) (type default))
   )
-  (wire (pts (xy 347.98 19.05) (xy 354.33 19.05))
+  (wire (pts (xy 345.44 19.05) (xy 354.33 19.05))
     (stroke (width 0) (type default))
   )
@@
     (stroke (width 0) (type dash_dot))
   )
-  (wire (pts (xy 336.55 72.39) (xy 349.25 72.39))
-    (stroke (width 0) (type default))
-  )
   (wire (pts (xy 93.98 21.59) (xy 93.98 36.83))
     (stroke (width 0) (type default))
@@
     (stroke (width 0) (type default))
   )
-  (wire (pts (xy 347.98 20.32) (xy 347.98 19.05))
+  (wire (pts (xy 345.44 20.32) (xy 345.44 19.05))
     (stroke (width 0) (type default))
   )
@@
     (stroke (width 0) (type default))
   )
+  (wire (pts (xy 336.55 69.85) (xy 349.25 69.85))
+    (stroke (width 0) (type default))
+  )
   (wire (pts (xy 109.22 115.57) (xy 130.81 115.57))
     (stroke (width 0) (type default))
@@
     (effects (font (size 1.27 1.27)) (justify left bottom))
   )
-  (label "XBEE_DTR" (at 336.55 72.39 0) (fields_autoplaced)
+  (label "XBEE_DTR" (at 336.55 69.85 0) (fields_autoplaced)
     (effects (font (size 1.27 1.27)) (justify left bottom))
   )
@@
     (effects (font (size 1.27 1.27)) (justify left bottom))
   )
-  (label "XBEE_RTS" (at 336.55 69.85 0) (fields_autoplaced)
+  (label "XBEE_RTS" (at 336.55 72.39 0) (fields_autoplaced)
     (effects (font (size 1.27 1.27)) (justify left bottom))
   )
@@
     )
   )
-  (symbol (lib_id "power:GND") (at 347.98 31.75 0) (unit 1)
+  (symbol (lib_id "power:GND") (at 342.9 33.02 0) (unit 1)
     (in_bom yes) (on_board yes) (dnp no) (fields_autoplaced)
-    (property "Reference" "#PWR010" (at 347.98 38.1 0)
+    (property "Reference" "#PWR010" (at 342.9 39.37 0)
       (effects (font (size 1.27 1.27)) hide)
     )
-    (property "Value" "GND" (at 347.98 36.83 0)
+    (property "Value" "GND" (at 342.9 38.1 0)
       (effects (font (size 1.27 1.27)))
     )
-    (property "Footprint" "" (at 347.98 31.75 0)
+    (property "Footprint" "" (at 342.9 33.02 0)
       (effects (font (size 1.27 1.27)) hide)
     )
-    (property "Datasheet" "" (at 347.98 31.75 0)
+    (property "Datasheet" "" (at 342.9 33.02 0)
       (effects (font (size 1.27 1.27)) hide)
     )
@@
       (effects (font (size 1.27 1.27)) (justify left) hide)
     )
-    (property "Footprint" "BITSv5:XT30PW-M" (at 199.39 22.606 90)
+    (property "Footprint" "Connector_AMASS:AMASS_XT30PW-M_1x02_P2.50mm_Horizontal" (at 199.39 22.606 90)
       (effects (font (size 1.27 1.27)) hide)
     )
@@
       (effects (font (size 1.524 1.524)))
     )
-    (property "Footprint" "SOT23-6L_STM" (at 355.6 135.89 0)
+    (property "Footprint" "BITSv5:SOT23-6L_STM-M" (at 355.6 135.89 0)
       (effects (font (size 1.27 1.27) italic) hide)
     )
@@
     )
   )
-  (symbol (lib_id "Switch:SW_Push") (at 347.98 25.4 90) (unit 1)
+  (symbol (lib_id "Switch:SW_SPDT") (at 345.44 25.4 270) (unit 1)
     (in_bom yes) (on_board yes) (dnp no)
     (property "Reference" "SW2" (at 340.36 24.13 90)
       (effects (font (size 1.27 1.27)) (justify right))
     )
-    (property "Value" "PTM" (at 340.36 26.67 90)
-      (effects (font (size 1.27 1.27)) (justify right))
+    (property "Value" "~" (at 339.09 22.86 90)
+      (effects (font (size 1.27 1.27)) (justify right) hide)
     )
-    (property "Footprint" "Button_Switch_SMD:SW_Push_1P1T_NO_CK_KMR2" (at 342.9 25.4 0)
+    (property "Footprint" "BITSv5:CAS-120TB_NDC-M" (at 345.44 25.4 0)
       (effects (font (size 1.27 1.27)) hide)
     )
-    (property "Datasheet" "~" (at 342.9 25.4 0)
+    (property "Datasheet" "~" (at 345.44 25.4 0)
       (effects (font (size 1.27 1.27)) hide)
     )
     (pin "1")
     (pin "2")
+    (pin "3")
     (instances
       (project "BITSv5"
@@
       (effects (font (size 1.27 1.27)) (justify left))
     )
-    (property "Footprint" "" (at 201.93 232.41 0)
+    (property "Footprint" "BITSv5:ANT_1575AT_JOT-M" (at 201.93 232.41 0)
       (effects (font (size 1.27 1.27)) hide)
     )
@@
   (symbol (lib_id "Device:Q_PMOS_GSD") (at 34.29 102.87 270) (unit 1)
     (in_bom yes) (on_board yes) (dnp no)
-    (property "Reference" "Q2" (at 36.83 111.76 90)
+    (property "Reference" "Q2" (at 36.83 110.49 90)
       (effects (font (size 1.27 1.27)))
     )
-    (property "Value" "Q_PMOS_GSD" (at 36.83 114.3 90)
+    (property "Value" "Q_PMOS_GSD" (at 36.83 113.03 90)
       (effects (font (size 1.27 1.27)))
     )
