File: Boards/BITSv5/BITSv5/BITSv5.kicad_sch (KiCad schematic)
At the start: 90 parts, among them J1 Conn_01x03_Pin, J2 USB_C_Receptacle_USB2.0, J3 XT30, J4 PicoBlade_53261-1071, J6 U.FL, Q1 Q_NMOS_GSD, SW3 SLIDE, U1 MCU_RaspberryPi_RP2040_RP2040, U10 USBLC6-2SC6, U11 MS5607-02BA, U2 W25Q128JVS, U3 MAX-M10S, U4 DRF1262TL, U6 TPS2121RUXR, U7 MB85RS1MT, U8 LT6703CDC-3, U9 TVS1800DRVR, Y1 12MHz

Commit message: BITSv5.2 new power system laid out
Parts:
- removed AE1: Antenna, BPP_Lib:ANT_1575AT_JOT-M, symbol Device:Antenna
- removed C37: 1uF, Capacitor_SMD:C_0402_1005Metric, symbol Device:C_Small
- removed H4: M2, MountingHole:MountingHole_2.2mm_M2_Pad, symbol Mechanical:MountingHole
- removed R18: 1.5M, Resistor_SMD:R_0402_1005Metric, symbol Device:R_Small
- removed R19: 100K, Resistor_SMD:R_0402_1005Metric, symbol Device:R_Small
- removed TP3: TestPoint, symbol Connector:TestPoint
- removed U8: LT6703CDC-3, BITSv5:DFN-3_DC_LIT, symbol LTC6703:LT6703CDC-3-TRPBF
- added C17, C24: 1uF, Capacitor_SMD:C_0603_1608Metric, symbol Device:C_Small
- added C18, C20: 47uF, Capacitor_SMD:C_1206_3216Metric, symbol Device:C_Small
- added C19, C23: 100nF, Capacitor_SMD:C_0603_1608Metric, symbol Device:C_Small
- added C21: 4.7uF, Capacitor_SMD:C_0805_2012Metric, symbol Device:C_Small
- added C25, C31: 22uF, Capacitor_SMD:C_0805_2012Metric, symbol Device:C_Small
- added H1: M2, MountingHole:MountingHole_2.2mm_M2_Pad, symbol Mechanical:MountingHole
- added J5: U.FL, Connector_Coaxial:U.FL_Molex_MCRF_73412-0110_Vertical, symbol Connector:Conn_Coaxial
- added JP1: SolderJumper_2_Open, Jumper:SolderJumper-2_P1.3mm_Open_RoundedPad1.0x1.5mm, symbol Jumper:SolderJumper_2_Open
- added R15: 332k, Resistor_SMD:R_0603_1608Metric, symbol Device:R_Small
- added R16, R31: 100k, Resistor_SMD:R_0603_1608Metric, symbol Device:R_Small
- added R32: 25.5k, Resistor_SMD:R_0603_1608Metric, symbol Device:R_Small
- added R33: 43.2k, Resistor_SMD:R_0603_1608Metric, symbol Device:R_Small
- added TP6: TestPoint, TestPoint:TestPoint_Keystone_5000-5004_Miniature, symbol Connector:TestPoint
- added U5, U8: TPSM33625FRDNR, BPP_Lib:RDN0011A-MFG-NO-VIA, symbol BPP_Lib:TPSM33625
- C16: footprint (none) -> Capacitor_SMD:C_0603_1608Metric
- J3: footprint (none) -> Connector_AMASS:AMASS_XT30PW-M_1x02_P2.50mm_Horizontal
- R20: value 510K -> 100k; footprint Resistor_SMD:R_0402_1005Metric -> Resistor_SMD:R_0603_1608Metric
- R22, R23, R25, R26, R27, R28, R29, R30: footprint (none) -> Resistor_SMD:R_0603_1608Metric
- R5: footprint Capacitor_SMD:C_0402_1005Metric -> Resistor_SMD:R_0402_1005Metric
- TP4, TP5: footprint (none) -> TestPoint:TestPoint_Keystone_5000-5004_Miniature
Connections:
- net +5V: now also C23.1, JP1.2 (B), U8.2 (EN), U8.3 (VIN); no longer C26.1, C27.1, U4.6 (VDD), U4.7 (VDD)
- net +BATT: now also C19.1, C21.1, R15.1, U5.3 (VIN)
- net EXTINT: now also U1.29 (GPIO18); no longer U1.28 (GPIO17)
- net GND: now also C17.2, C18.2, C19.2, C20.2, C21.2, C23.2, C24.2, C25.2, C31.2, J5.2 (Ext), R16.2, R32.2, R33.2, U5.10 (GND), U5.11 (MODE), U8.10 (GND), U8.11 (MODE)
- net TIMEPULSE: now also U1.28 (GPIO17); no longer U1.29 (GPIO18)
- net VBUS: now also J2.A4 (VBUS), J2.A9 (VBUS), J2.B4 (VBUS), J2.B9 (VBUS), U10.5
- net at SW3.3 (C): now also R16.1; no longer R20.2
- net BATT_REG: now reaches C34.1, R25.1, R27.1, U6.2 (IN2)
- net BATT_REG: now also C18.1, C20.1, R31.1, TP6.1, U5.4 (VOUT)
- net at R20.1: now also L3.2, R10.2, C25.1, C31.1, U8.4 (VOUT)
- net at U3.11 (RF_IN): now also J5.1 (In)
- net at U3.2 (TXD): now also J1.1 (Pin_1); no longer J1.2 (Pin_2)
- net at U3.3 (RXD): now also J1.2 (Pin_2); no longer J1.1 (Pin_1)
- net LVC_CUTOFF: no longer names the net of SW3.2 (B)
- net LVC_CUTOFF: now also R15.2, U5.2 (EN)
- new net: C26.1, C27.1, JP1.1 (A), U4.6 (VDD), U4.7 (VDD)
- new net: U3.10 (GND), U3.12 (GND)
- new net: C24.1, U8.8 (VCC)
- new net: R31.2, R32.1, U5.9 (FB)
- new net: R20.2, R33.1, U8.9 (FB)
- new net: C17.1, U5.8 (VCC)
- no-connect marks 22 -> 24
Other:
- note added: "3.3v Power"
- note added: "5v Power"
- note added: "Power Train"
- note removed: "LVC"
- note removed: "SOICbite"
- note removed: "TPSM33625FRDNR"
- title: UMDBPP Command BITSv5.1 -> UMDBPP Command BITSv5.2
- moved on the sheet: C15, C16, C28, C33, C34, C38, L3, L4, R10, R13, R17, R22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
