File: Boards/BITSv5/BITSv5/sch1_BITSv5.kicad_sch (KiCad schematic)
At the start: 81 parts, among them J1 Conn_01x10_Pin, J2 USB_C_Receptacle_USB2.0, J3 Conn_01x07, Q1 Q_NMOS_GSD, Q2 Q_PMOS_GSD, SW3 SLIDE, U1 MCU_RaspberryPi_RP2040_RP2040, U10 USBLC6-2SC6, U2 W25Q128JVS, U3 MAX-M10S, U4 MAX25255AFDA/VY+, U6 XBee_SMT, U7 TPS2121RUXR, U8 LT6703CDC-3, U9 TVS1800DRVR, Y1 12MHz

Commit message: BITSv5 layout changes
Parts:
- removed C15, C31: 0.1uF, Capacitor_SMD:C_0603_1608Metric_Pad1.08x0.95mm_HandSolder, symbol Device:C_Small
- removed C16, C29, C30: 4.7uF, Capacitor_SMD:C_0603_1608Metric_Pad1.08x0.95mm_HandSolder, symbol Device:C_Small
- removed C25: 2.2uF, Capacitor_SMD:C_0603_1608Metric_Pad1.08x0.95mm_HandSolder, symbol Device:C_Small
- removed R10, R9: 10K, Resistor_SMD:R_0603_1608Metric_Pad0.98x0.95mm_HandSolder, symbol Device:R_Small
- removed U4: MAX25255AFDA/VY+, BITSv5:21-100477_90-100168_MXM, symbol BITSv5:MAX25255DAFDG_VY+
- added C15, C16: 220nF, Capacitor_SMD:C_0603_1608Metric_Pad1.08x0.95mm_HandSolder, symbol Device:C
- added C25, C31: 22uF, Capacitor_SMD:C_0805_2012Metric_Pad1.18x1.45mm_HandSolder, symbol Device:C
- added C29: 10uF, Capacitor_SMD:C_0603_1608Metric_Pad1.08x0.95mm_HandSolder, symbol Device:C
- added C30: 10pF, Capacitor_SMD:C_0402_1005Metric_Pad0.74x0.62mm_HandSolder, symbol Device:C
- added R10: 48.7K, Resistor_SMD:R_0402_1005Metric_Pad0.72x0.64mm_HandSolder, symbol Device:R
- added R13: 178K, Resistor_SMD:R_0603_1608Metric_Pad0.98x0.95mm_HandSolder, symbol Device:R
- added R14: 20K, Resistor_SMD:R_0603_1608Metric_Pad0.98x0.95mm_HandSolder, symbol Device:R
- added R25: 15K, Resistor_SMD:R_0402_1005Metric_Pad0.72x0.64mm_HandSolder, symbol Device:R
- added R26: 5K, Resistor_SMD:R_0402_1005Metric_Pad0.72x0.64mm_HandSolder, symbol Device:R
- added R9: 1M, Resistor_SMD:R_0603_1608Metric_Pad0.98x0.95mm_HandSolder, symbol Device:R
- added U4: MAX77857, BITSv5:MAX77857-35WLP, symbol MAX77857:MAX77857BEWB+
- added U5: TPS61232DRCR, BITSv5:TPS61232, symbol TPS61232:TPS61232DRCR
- C17, C18: footprint Capacitor_SMD:C_0603_1608Metric_Pad1.08x0.95mm_HandSolder -> Capacitor_SMD:C_0805_2012Metric_Pad1.18x1.45mm_HandSolder
- C19: value 22uF -> 470nF; footprint Capacitor_SMD:C_0603_1608Metric_Pad1.08x0.95mm_HandSolder -> Capacitor_SMD:C_0402_1005Metric_Pad0.74x0.62mm_HandSolder
- C20, C21: value 22uF -> 10uF; footprint Capacitor_SMD:C_0603_1608Metric_Pad1.08x0.95mm_HandSolder -> Capacitor_SMD:C_0805_2012Metric_Pad1.18x1.45mm_HandSolder
- C22: value 22uF -> 2.2uF; footprint Capacitor_SMD:C_0603_1608Metric_Pad1.08x0.95mm_HandSolder -> Capacitor_SMD:C_0402_1005Metric_Pad0.74x0.62mm_HandSolder
- C23, C24: value 0.1uF -> 22uF; footprint Capacitor_SMD:C_0402_1005Metric_Pad0.74x0.62mm_HandSolder -> Capacitor_SMD:C_0805_2012Metric_Pad1.18x1.45mm_HandSolder
- C26: value 100pF -> 8.2pF
- C27: value 1uF -> 47pF
- C28: value 10uF -> 100nF
- C32: value 100nF -> 10nF; footprint Capacitor_SMD:C_0402_1005Metric_Pad0.74x0.62mm_HandSolder -> Capacitor_SMD:C_0603_1608Metric_Pad1.08x0.95mm_HandSolder
- J1: footprint Connector_Molex:Molex_PicoBlade_53048-1010_1x10_P1.25mm_Horizontal -> Connector_Molex:Molex_PicoBlade_53261-1071_1x10-1MP_P1.25mm_Horizontal
- L1: value 0.47uH -> 1uH
- L2: value 0.47uH -> 1uH; footprint Inductor_SMD:L_1008_2520Metric_Pad1.43x2.20mm_HandSolder -> BITSv5:IND_XAL4020_4X4_COC-M
Connections:
- net +3V3: now also C17.1, C18.1, C29.1, C30.1, R13.1, U4.D4 (OUT), U4.E4 (OUT), U4.E5 (OUT), U4.E6 (OUT); no longer C20.2, C21.2, C22.2, C32.1, L2.2
- net +5V: now also C23.1, C25.1, C31.1, R9.1, U5.3 (VOUT), U5.4 (VOUT), U5.7 (FB); no longer C17.2, C18.2, C19.2, L1.1
- net +BATT: now also R25.1
- net GND: now also C17.2, C18.2, C19.2, C20.2, C21.2, C22.2, C23.2, C24.2, C25.2, C29.2, C31.2, R10.2, R14.2, R26.1, U4.C3 (PGND), U4.C4 (PGND), U4.C5 (PGND), U4.C6 (PGND), U4.C7 (PGND), U4.D2 (PGND), U4.D3 (PGND), U4.E2 (AGND), U5.11 (GND); no longer C17.1, C18.1, C19.1, C20.1, C21.1, C22.1
- net GPS_SCL: now also U1.28 (GPIO17); no longer U1.32 (GPIO21)
- net GPS_SDA: now also U1.27 (GPIO16); no longer U1.31 (GPIO20)
- net LVC_CUTOFF: now also U4.B2 (EN), U4.B3 (EN), U5.9 (EN)
- net RP_SWCLK: now also J3.6 (Pin_6); no longer J3.7 (Pin_7)
- net RP_SWD: now also J3.7 (Pin_7); no longer J3.6 (Pin_6)
- net VBAT: now also R25.2, R26.2
- net VCC: now also C20.1, C21.1, C24.1, L2.1, U4.A4 (IN), U4.A5 (IN), U4.A6 (IN), U4.B4 (IN), U5.10 (VIN)
- net at L1.2: now also C16.1, U4.D5 (LX2), U4.D6 (LX2), U4.D7 (LX2), U4.E7 (LX2); no longer C23.2
- new net: C30.2, R13.2, R14.1, U4.E1 (FB)
- new net: C15.1, U4.A3 (BST1)
- new net: C15.2, L1.1, U4.A7 (LX1), U4.B5 (LX1), U4.B6 (LX1), U4.B7 (LX1)
- new net: R10.1, U4.D1 (SEL)
- new net: L2.2, U5.1 (SW), U5.2 (SW)
- new net: C16.2, U4.E3 (BST2)
- new net: C19.1, C22.1, U4.A1 (SCL), U4.A2 (VIO), U4.B1 (SDA), U4.C1 (VL)
- new net: R9.2, U5.5 (PG)
- new net: C32.1, U5.6 (SS)
- no-connect marks 51 -> 48
Other:
- note added: "3.3V Buck-Boost"
- note added: "5V Boost"
- note added: "Voltage Divider"
- note removed: "Dual Buck Regulator"
- moved on the sheet: BT1, C26, C27, C33, C34, C35, C36, J3, R15, R16, R17, R22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
