File: Boards/BITSv5/BITSv5/BITSv5.kicad_pcb (KiCad board)
At the start: 2 copper layers, 8 parts, among them J3 USB_C_Receptacle_USB2.0, U1 MCU_RaspberryPi_RP2040_RP2040, U2 W25Q128JVS, U3 MAX-M10S, U4 MAX77857, U5 TPS610997YFFR, U6 XBee_SMT, Y1 ABLS-12.000MHZ-B4-T

Commit message: BITSv5 sch almost done
Parts:
- added BT1: 1S1P LiPo, GHOULFootPrints:XT30PW-M, F.Cu at (162.1, 35.2)
- added C1: 1uF, Capacitor_SMD:C_0603_1608Metric, F.Cu at (94.0, 24.0)
- added C10: 100nF, Capacitor_SMD:C_0603_1608Metric, F.Cu at (98.0, 26.6)
- added C11: 100nF, Capacitor_SMD:C_0603_1608Metric, F.Cu at (98.0, 29.1)
- added C12: 100nF, Capacitor_SMD:C_0603_1608Metric, F.Cu at (98.0, 31.6)
- added C13: 10pF, Capacitor_SMD:C_0603_1608Metric, F.Cu at (98.0, 34.1)
- added C14: 10pF, Capacitor_SMD:C_0603_1608Metric, F.Cu at (98.0, 36.6)
- added C15: 220nF, Capacitor_SMD:C_0603_1608Metric, F.Cu at (85.3, 97.3)
- added C16: 220nF, Capacitor_SMD:C_0603_1608Metric, F.Cu at (105.9, 96.3)
- added C17: 22uF, Capacitor_SMD:C_0805_2012Metric, F.Cu at (100.3, 109.0)
- added C18: 22uF, Capacitor_SMD:C_0805_2012Metric, F.Cu at (102.4, 109.0)
- added C19: 470nF, Capacitor_SMD:C_0402_1005Metric, F.Cu at (93.6, 119.3)
- added C2: 1uF, Capacitor_SMD:C_0603_1608Metric, F.Cu at (94.0, 26.6)
- added C20: 10uF, Capacitor_SMD:C_0805_2012Metric, F.Cu at (93.1, 109.0)
- added C21: 10uF, Capacitor_SMD:C_0805_2012Metric, F.Cu at (95.2, 109.0)
- added C22: 2.2uF, Capacitor_SMD:C_0402_1005Metric, F.Cu at (93.6, 121.3)
- added C23: 22uF, Capacitor_SMD:C_0805_2012Metric, F.Cu at (89.8, 36.3)
- added C24: 22uF, Capacitor_SMD:C_0805_2012Metric, F.Cu at (89.8, 39.3)
- added C25: 22uF, Capacitor_SMD:C_0805_2012Metric, F.Cu at (89.8, 42.4)
- added C26: 8.2pF, Capacitor_SMD:C_0603_1608Metric, F.Cu at (59.3, 21.6)
- added C27: 47pF, Capacitor_SMD:C_0603_1608Metric, F.Cu at (59.3, 24.1)
- added C28: 100nF, Capacitor_SMD:C_0603_1608Metric, F.Cu at (59.3, 26.6)
- added C29: 10uF, Capacitor_SMD:C_0603_1608Metric, F.Cu at (59.3, 29.1)
- added C3: 100nF, Capacitor_SMD:C_0603_1608Metric, F.Cu at (94.0, 29.1)
- added C30: 10pF, Capacitor_SMD:C_0402_1005Metric, F.Cu at (103.3, 120.9)
- added C31: 22uF, Capacitor_SMD:C_0805_2012Metric, F.Cu at (89.8, 45.4)
- added C32: 10nF, Capacitor_SMD:C_0603_1608Metric, F.Cu at (59.3, 31.6)
- added C33: 10nF, Capacitor_SMD:C_0603_1608Metric, F.Cu at (175.0, 24.0)
- added C34: 10uF, Capacitor_SMD:C_0603_1608Metric, F.Cu at (175.0, 26.5)
- added C35: 10uF, Capacitor_SMD:C_0603_1608Metric, F.Cu at (175.0, 29.0)
- added C36: 1uF, Capacitor_SMD:C_0603_1608Metric, F.Cu at (175.0, 31.5)
- added C37: 1uF, Capacitor_SMD:C_0603_1608Metric, F.Cu at (175.0, 34.0)
- added C4: 100nF, Capacitor_SMD:C_0603_1608Metric, F.Cu at (94.0, 31.6)
- added C5: 100nF, Capacitor_SMD:C_0603_1608Metric, F.Cu at (94.0, 34.1)
- added C6: 100nF, Capacitor_SMD:C_0603_1608Metric, F.Cu at (94.0, 36.6)
- added C7: 100nF, Capacitor_SMD:C_0603_1608Metric, F.Cu at (94.0, 39.1)
- added C8: 100nF, Capacitor_SMD:C_0603_1608Metric, F.Cu at (98.0, 24.0)
- added C9: 100nF, Capacitor_SMD:C_0603_1608Metric, F.Cu at (59.3, 35.6)
- added D1: LED, LED_SMD:LED_0603_1608Metric, F.Cu at (175.1, 36.6)
- added J1: Conn_01x10_Pin, Connector_Molex:Molex_PicoBlade_53047-1010_1x10_P1.25mm_Vertical, F.Cu at (149.5, 53.0)
- added L1: 1uH, Inductor_SMD:L_1008_2520Metric, F.Cu at (98.3, 103.3)
- added L2: 1uH, 1616_Inductor:IND_XAL4020_4X4_COC-M, F.Cu at (96.8, 43.4)
- added R1: 27Ω, Resistor_SMD:R_0603_1608Metric, F.Cu at (102.0, 26.6)
- added R10: 50K, Resistor_SMD:R_0603_1608Metric, F.Cu at (133.5, 114.4)
- added R11: 10K, Resistor_SMD:R_0603_1608Metric, F.Cu at (106.0, 29.1)
- added R12: 270, Resistor_SMD:R_0603_1608Metric, F.Cu at (106.0, 31.6)
- added R13: 178K, Resistor_SMD:R_0603_1608Metric, F.Cu at (113.4, 116.0)
- added R14: 20K, Resistor_SMD:R_0603_1608Metric, F.Cu at (113.4, 118.5)
- added R15: 23.7K, Resistor_SMD:R_0603_1608Metric, F.Cu at (179.0, 24.0)
- added R16: 5K, Resistor_SMD:R_0603_1608Metric, F.Cu at (179.0, 26.5)
- added R17: 51.1K, Resistor_SMD:R_0603_1608Metric, F.Cu at (179.0, 29.0)
- added R18: 1.05M, Resistor_SMD:R_0603_1608Metric, F.Cu at (179.0, 31.5)
- added R19: 154K, Resistor_SMD:R_0603_1608Metric, F.Cu at (179.0, 34.0)
- added R2: 27Ω, Resistor_SMD:R_0603_1608Metric, F.Cu at (102.0, 29.1)
- added R20: 510K, Resistor_SMD:R_0603_1608Metric, F.Cu at (183.1, 24.0)
- added R22: 23.7K, Resistor_SMD:R_0603_1608Metric, F.Cu at (183.1, 26.5)
- added R23: 5K, Resistor_SMD:R_0603_1608Metric, F.Cu at (183.1, 29.0)
- added R3: 10K, Resistor_SMD:R_0603_1608Metric, F.Cu at (102.0, 31.6)
- added R4: 1K, Resistor_SMD:R_0603_1608Metric, F.Cu at (102.0, 34.1)
- added R5: 1K, Resistor_SMD:R_0603_1608Metric, F.Cu at (102.0, 36.6)
- added R6: 1M, Resistor_SMD:R_0603_1608Metric, F.Cu at (102.0, 39.1)
- added R7: 5.1K, Resistor_SMD:R_0603_1608Metric, F.Cu at (111.0, 32.9)
- added R8: 5.1K, Resistor_SMD:R_0603_1608Metric, F.Cu at (111.0, 35.4)
- added R9: 1M, Resistor_SMD:R_0603_1608Metric, F.Cu at (106.0, 24.0)
- U5: value TPS610997YFFR -> TPS61232DRCR; footprint TPS610997:YFF0006AFAD -> TPS61232:DRC0010G
- Y1: value ABLS-12.000MHZ-B4-T -> 12MHz; footprint Crystal:Crystal_SMD_HC49-SD -> Crystal:Crystal_SMD_2520-4Pin_2.5x2.0mm
- moved U4 74.2 mm to (97.8, 110.4), turned to 90 degrees
- moved U5 27.2 mm to (107.5, 43.0)
- moved U2 2.24 mm to (109.6, 68.4)
- renumbered J3 to J2
Connections:
- net /RP2040_SWCLK renamed Net-(J4-Pin_1)
- net /RP2040_SWDIO renamed Net-(J4-Pin_2)
- net /USB_D+ renamed Net-(J2-D+-PadA6)
- net /USB_D- renamed Net-(J2-D--PadA7)
- J2 pad A4: VCC -> VBUS
- J2 pad A9: VCC -> VBUS
- J2 pad B4: VCC -> VBUS
- J2 pad B9: VCC -> VBUS
- U1 pad 2: unconnected-(U1-GPIO0-Pad2) -> /IRIDIUM_TXD
- U1 pad 3: unconnected-(U1-GPIO1-Pad3) -> /IRIDIUM_RXD
- U1 pad 4: unconnected-(U1-GPIO2-Pad4) -> /IRIDIUM_CTS
- U1 pad 5: unconnected-(U1-GPIO3-Pad5) -> /IRIDIUM_RTS
- U1 pad 6: unconnected-(U1-GPIO4-Pad6) -> /IRIDIUM_RING
- U1 pad 7: unconnected-(U1-GPIO5-Pad7) -> /IRIDIUM_ON/OFF
- U1 pad 8: unconnected-(U1-GPIO6-Pad8) -> /IRIDIUM_NETAV
- U3 pad 16: /GPS_SDA -> unconnected-(U3-SDA-Pad16)
- U3 pad 17: /GPS_SCL -> unconnected-(U3-SCL-Pad17)
- U3 pad 2: unconnected-(U3-TXD-Pad2) -> /GPS_TX
- U3 pad 3: unconnected-(U3-RXD-Pad3) -> /GPS_RX
- U4 pad A1: unconnected-(U4-SCL-PadA1) -> Net-(U4-SCL)
- U4 pad A2: /BUCKBOOST_VIO -> Net-(U4-SCL)
- U4 pad B1: unconnected-(U4-SDA-PadB1) -> Net-(U4-SCL)
- U4 pad B2: /BUCKBOOST_EN -> /LVC_CUTOFF
- U4 pad B3: /BUCKBOOST_EN -> /LVC_CUTOFF
- U4 pad C1: Net-(U4-VL) -> Net-(U4-SCL)
- U4 pad E1: +3V3 -> Net-(U4-FB)
- U6 pad 6: unconnected-(U6-RESET/OD_OUT-Pad6) -> /XBEE_RESET
Routing:
- net Net-(C16-Pad1): vias 0 -> 3
- net Net-(C15-Pad2): vias 0 -> 3
- added copper zone on F.Cu, net +3V3
- added copper zone on F.Cu, net GND
- added copper zone on F.Cu, net Net-(C15-Pad2)
- added copper zone on F.Cu, net Net-(C16-Pad1)
- added copper zone on F.Cu, net VCC
Other:
- copper layers 2 -> 4

Commit message: more bits updates
Parts:
- added R25: 15K, Resistor_SMD:R_0603_1608Metric, F.Cu at (125.2, 32.6)
- added R26: 5K, Resistor_SMD:R_0603_1608Metric, F.Cu at (125.2, 35.1)
- added U10: USBLC6-2SC6, BITSv5:SOT23-6L_STM, F.Cu at (132.4, 62.6)
- added U8: LT6703CDC-3, BITSv5:DFN-3_DC_LIT, F.Cu at (77.4, 127.3)
- BT1: moved to B.Cu
- R10: footprint Resistor_SMD:R_0603_1608Metric -> Resistor_SMD:R_0402_1005Metric
- R12: value 270 -> 470
- moved C37 135.8 mm to (73.2, 124.0)
- moved R18 135.8 mm to (77.2, 121.5)
- moved R19 135.8 mm to (77.2, 124.0)
- moved R20 135.8 mm to (81.3, 113.9)
- moved BT1 134.6 mm to (60.0, 122.8), turned to 90 degrees
- moved R9 99.6 mm to (102.2, 123.6), turned to 180 degrees
- moved C32 96.8 mm to (103.5, 117.7)
- moved C23 85.4 mm to (103.0, 120.7), turned to 90 degrees
- moved L2 81.2 mm to (94.2, 124.6)
- moved C24 80.2 mm to (95.0, 119.4), turned to -90 degrees
- moved C25 79.9 mm to (105.4, 120.7), turned to 90 degrees
- moved C31 77.4 mm to (107.8, 120.7), turned to 90 degrees
- moved U5 76.5 mm to (98.8, 119.0), turned to 90 degrees
- moved R10 34.4 mm to (99.2, 113.6), turned to -90 degrees
- moved C15 17.1 mm to (94.4, 111.8), turned to 180 degrees
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Connections:
- R20 pad 2: /LVC_CUTOFF -> Net-(SW3-C)
- U1 pad 27: unconnected-(U1-GPIO16-Pad27) -> /GPS_SDA
- U1 pad 28: unconnected-(U1-GPIO17-Pad28) -> /GPS_SCL
- U1 pad 34: unconnected-(U1-GPIO22-Pad34) -> /XBEE_RTS
- U1 pad 35: unconnected-(U1-GPIO23-Pad35) -> /XBEE_CTS
- U1 pad 36: unconnected-(U1-GPIO24-Pad36) -> /XBEE_DIN
- U1 pad 37: unconnected-(U1-GPIO25-Pad37) -> /XBEE_DOUT
- U1 pad 38: unconnected-(U1-GPIO26_ADC0-Pad38) -> /VBAT
- U1 pad 9: unconnected-(U1-GPIO7-Pad9) -> /LED
- U3 pad 16: unconnected-(U3-SDA-Pad16) -> /GPS_SDA
- U3 pad 17: unconnected-(U3-SCL-Pad17) -> /GPS_SCL
- U3 pad 2: /GPS_TX -> unconnected-(U3-TXD-Pad2)
- U3 pad 3: /GPS_RX -> unconnected-(U3-RXD-Pad3)
- U6 pad 24: unconnected-(U6-DIO4-Pad24) -> /XBEE_DIO4
Routing:
- net Net-(U4-FB): track 0.00 -> 10.7 mm, vias 0 -> 3
- net +5V: track 0.00 -> 7.11 mm, vias 0 -> 2
- net GND: track 0.00 -> 6.15 mm, vias 0 -> 30
- net Net-(U5-PG): track 0.00 -> 4.10 mm, vias 0 -> 2
- net VCC: track 0.00 -> 3.18 mm
- net Net-(U5-SS): track 0.00 -> 2.95 mm
- net Net-(U4-SEL): track 0.00 -> 2.02 mm, vias 0 -> 2
- net Net-(C16-Pad1): vias 3 -> 9
- net Net-(C15-Pad2): vias 3 -> 10
- net /LVC_CUTOFF: vias 0 -> 2
- added copper zone on F.Cu, net +5V
- added copper zone on In1.Cu, net /LVC_CUTOFF
- added copper zone on In1.Cu, net Net-(C15-Pad2)
- added copper zone on In1.Cu, net Net-(C16-Pad1)
- added copper zone on F.Cu, net Net-(L2-Pad2)
- added copper zone on F.Cu, net Net-(U4-BST1)
- added copper zone on F.Cu, net Net-(U4-BST2)
- added copper zone on F.Cu, net Net-(U4-SCL)
- added copper zone on F.Cu, net Net-(U5-PG)

Commit message: bits v5 board nearly done
Parts:
- added J3: Conn_01x06, Connector_JST:JST_EH_B5B-EH-A_1x05_P2.50mm_Vertical, F.Cu at (188.2, 119.2)
- added Q1: Q_NMOS_GSD, Package_TO_SOT_SMD:SOT-23-3, F.Cu at (173.4, 98.8)
- added Q2: Q_PMOS_GSD, Package_TO_SOT_SMD:SOT-23, F.Cu at (171.3, 117.8)
- added R21: 10K, Resistor_SMD:R_0603_1608Metric_Pad0.98x0.95mm_HandSolder, F.Cu at (192.9, 107.6)
- added R24: 10K, Resistor_SMD:R_0603_1608Metric_Pad0.98x0.95mm_HandSolder, F.Cu at (192.9, 105.6)
- added SW2: PTM, Button_Switch_SMD:SW_Push_1P1T_NO_CK_KMR2, F.Cu at (190.5, 112.8)
- added SW3: SLIDE, BITSv5:CL-SB-12B-01_NDC, F.Cu at (137.4, 105.3)
- added U7: TPS2121RUXR, BITSv5:TPS2121, F.Cu at (156.9, 80.0)
- added U9: TVS1800DRVR, BITSv5:TVS1800, F.Cu at (156.2, 69.2)
- C1, C10, C11, C2, C3, C4, C5, C6, C7, C8, C9: footprint Capacitor_SMD:C_0603_1608Metric -> Capacitor_SMD:C_0402_1005Metric_Pad0.74x0.62mm_HandSolder
- C12, C13, C14, C15, C16, C26, C27, C28, C29, C32, C33, C34, C35, C36, C37: footprint Capacitor_SMD:C_0603_1608Metric -> Capacitor_SMD:C_0603_1608Metric_Pad1.08x0.95mm_HandSolder
- C17, C18, C20, C21, C23, C24, C25, C31: footprint Capacitor_SMD:C_0805_2012Metric -> Capacitor_SMD:C_0805_2012Metric_Pad1.18x1.45mm_HandSolder
- C19, C22, C30: footprint Capacitor_SMD:C_0402_1005Metric -> Capacitor_SMD:C_0402_1005Metric_Pad0.74x0.62mm_HandSolder
- J1: footprint Connector_Molex:Molex_PicoBlade_53047-1010_1x10_P1.25mm_Vertical -> Connector_Molex:Molex_PicoBlade_53261-1071_1x10-1MP_P1.25mm_Horizontal
- L1: footprint Inductor_SMD:L_1008_2520Metric -> Inductor_SMD:L_1008_2520Metric_Pad1.43x2.20mm_HandSolder
- R1, R2, R25, R26, R5: footprint Resistor_SMD:R_0603_1608Metric -> Resistor_SMD:R_0402_1005Metric_Pad0.72x0.64mm_HandSolder
- R10: value 50K -> 48.7K; footprint Resistor_SMD:R_0402_1005Metric -> Resistor_SMD:R_0402_1005Metric_Pad0.72x0.64mm_HandSolder
- R11, R12, R13, R14, R15, R16, R17, R18, R19, R20, R22, R23, R3, R4, R6, R7, R8, R9: footprint Resistor_SMD:R_0603_1608Metric -> Resistor_SMD:R_0603_1608Metric_Pad0.98x0.95mm_HandSolder
- U6: footprint RF_Module:Digi_XBee_SMT -> BITSv5:XCVR_XBP9X-DMUS-001
- moved C26 133.8 mm to (181.7, 75.5), turned to 180 degrees
- moved C27 131.9 mm to (181.7, 73.0), turned to 180 degrees
- moved C28 130.1 mm to (181.7, 70.5), turned to 180 degrees
- moved C9 129.2 mm to (169.5, 103.1), turned to 90 degrees
- moved C29 128.5 mm to (181.7, 68.0), turned to 180 degrees
- moved C4 112.0 mm to (166.0, 117.4), turned to -90 degrees
- moved C11 110.6 mm to (164.6, 117.4), turned to -90 degrees
- moved C5 109.8 mm to (171.6, 111.7)
- moved U6 108.5 mm to (197.3, 84.4)
- moved R11 108.5 mm to (168.1, 118.0), turned to 90 degrees
- moved U3 108.4 mm to (201.6, 114.4), turned to 90 degrees
- moved C8 108.2 mm to (159.2, 113.3), turned to -90 degrees
- moved C1 107.5 mm to (166.8, 103.0), turned to 90 degrees
- moved C2 106.5 mm to (168.2, 103.0), turned to 90 degrees
- moved R19 103.6 mm to (165.9, 70.3), turned to 90 degrees
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Connections:
- C37 pad 1: +BATT -> VCC
- R18 pad 1: +BATT -> VCC
- R20 pad 1: +BATT -> VCC
- U1 pad 29: unconnected-(U1-GPIO18-Pad29) -> /LED
- U1 pad 35: /XBEE_CTS -> unconnected-(U1-GPIO23-Pad35)
- U1 pad 38: /VBAT -> unconnected-(U1-GPIO26_ADC0-Pad38)
- U1 pad 40: unconnected-(U1-GPIO28_ADC2-Pad40) -> /VBAT
- U1 pad 9: /LED -> unconnected-(U1-GPIO7-Pad9)
- U6 pad 18: unconnected-(U6-NC-Pad18) -> (no net)
- U6 pad 19: unconnected-(U6-NC-Pad19) -> (no net)
- U6 pad 20: unconnected-(U6-NC-Pad20) -> (no net)
- U6 pad 21: unconnected-(U6-NC-Pad21) -> (no net)
- U6 pad 23: unconnected-(U6-NC-Pad23) -> (no net)
- U6 pad 24: /XBEE_DIO4 -> unconnected-(U6-DIO4-Pad24)
- U6 pad 27: unconnected-(U6-VREF-Pad27) -> (no net)
- U6 pad 34: unconnected-(U6-NC-Pad34) -> (no net)
- U6 pad 37: unconnected-(U6-NC-Pad37) -> (no net)
- U6 pad 9: unconnected-(U6-NC-Pad9) -> (no net)
- U8 pad 2: +BATT -> VCC
- Y1 pad 2: /XIN -> GND
- Y1 pad 3: (no net) -> /XIN
- Y1 pad 4: (no net) -> GND
Routing:
- net +3V3: track 0.00 -> 211.5 mm, vias 0 -> 25
- net +5V: track 7.11 -> 96.6 mm, vias 2 -> 13
- net /XBEE_RTS: track 0.00 -> 89.0 mm, vias 0 -> 1
- net +BATT: track 0.00 -> 63.1 mm, vias 0 -> 1
- net /XBEE_DOUT: track 0.00 -> 57.9 mm, vias 0 -> 1
- net /LVC_CUTOFF: track 0.00 -> 57.9 mm, vias 2 -> 3
- net Net-(R4-Pad1): track 0.00 -> 54.5 mm, vias 0 -> 2
- net Net-(SW3-C): track 0.00 -> 54.3 mm, vias 0 -> 2
- net /XBEE_DIN: track 0.00 -> 52.6 mm, vias 0 -> 1
- net /XBEE_RESET: track 0.00 -> 45.5 mm
- net /GPS_SDA: track 0.00 -> 40.2 mm, vias 0 -> 2
- net /GPS_SCL: track 0.00 -> 39.4 mm, vias 0 -> 2
- net VCC: track 3.18 -> 41.4 mm
- net +1V1: track 0.00 -> 30.3 mm, vias 0 -> 4
- net /IRIDIUM_RXD: track 0.00 -> 29.5 mm
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- added copper zone on F.Cu, net +1V1
- added copper zone on F.Cu, net +BATT
- added copper zone on F.Cu, net /LVC_CUTOFF
- added copper zone on B.Cu, net GND
- added copper zone on F.Cu, net Net-(J2-D+-PadA6)
- added copper zone on F.Cu, net Net-(R4-Pad1)
- added copper zone on F.Cu, net Net-(SW3-C)
- added copper zone on F.Cu, net VBUS

Commit message: several hundred bits v5 errors later
Parts:
- BT1: footprint GHOULFootPrints:XT30PW-M -> BITSv5:XT30PW-M
- J3: value Conn_01x06 -> Conn_01x07; footprint Connector_JST:JST_EH_B5B-EH-A_1x05_P2.50mm_Vertical -> Connector_PinSocket_2.54mm:PinSocket_1x07_P2.54mm_Vertical
- L2: footprint 1616_Inductor:IND_XAL4020_4X4_COC-M -> BITSv5:IND_XAL4020_4X4_COC-M
- U1: footprint RP2040_minimal:RP2040-QFN-56 -> BITSv5:RP2040-QFN-56
- U4: footprint MAX77857:MAX77857-35WLP -> BITSv5:MAX77857-35WLP
- U5: footprint TPS61232:DRC0010G -> BITSv5:TPS61232
- moved J3 3.83 mm to (192.0, 119.3), turned to -90 degrees
Connections:
- U1 pad 24: Net-(J4-Pin_1) -> /RP_SWCLK
- U1 pad 25: Net-(J4-Pin_2) -> /RP_SWD
Routing:
- net GND: track 27.2 -> 50.0 mm, vias 108 -> 98
- net /RP_SWCLK: track 0.00 -> 17.1 mm, vias 0 -> 1
- net /RP_SWD: track 0.00 -> 13.8 mm, vias 0 -> 1
- net VBUS: track 14.0 -> 27.7 mm
- net /XBEE_RTS: track 89.0 -> 93.5 mm
- net /XBEE_DIN: track 52.6 -> 56.5 mm
- net +3V3: track 211.5 -> 214.3 mm
- net /XBEE_DTR: track 27.2 -> 29.7 mm
- net /XBEE_DOUT: track 57.9 -> 59.7 mm
- net /XBEE_RESET: track 45.5 -> 46.4 mm
- net Net-(C16-Pad1): track 4.62 -> 4.83 mm, vias 10 -> 7
- net Net-(C15-Pad2): track 4.24 -> 4.38 mm, vias 10 -> 7
- net Net-(U4-SEL): track 1.86 -> 1.82 mm, vias 2 -> 0
- added copper zone on In2.Cu, net +5V
Other:
- board outline added: 82.9 x 59.4 mm

Commit message: bits v5 board feedback added
Parts:
- added AE1: Antenna, BITSv5:ANT_1575AT_JOT-M, F.Cu at (213.0, 112.3)
- BT1: footprint BITSv5:XT30PW-M -> Connector_AMASS:AMASS_XT30PW-M_1x02_P2.50mm_Horizontal
- SW2: value PTM -> ~; footprint Button_Switch_SMD:SW_Push_1P1T_NO_CK_KMR2 -> BITSv5:CAS-120TB_NDC-M
- U10: footprint BITSv5:SOT23-6L_STM -> BITSv5:SOT23-6L_STM-M
- moved J3 18.9 mm to (180.4, 104.4), turned to 0 degrees
- moved SW2 5.99 mm to (186.9, 117.6)
- moved R21 5.88 mm to (188.1, 110.9)
- moved R24 5.88 mm to (188.1, 109.0)
- moved C24 3.73 mm to (167.3, 79.8), turned to -90 degrees
- moved U3 3.50 mm to (198.1, 114.5)
- moved BT1 2.61 mm to (146.2, 79.7), turned to -90 degrees
- moved C11 1.84 mm to (164.5, 119.2)
- moved C4 1.84 mm to (165.8, 119.2)
- moved L2 1.81 mm to (176.0, 79.8)
- moved J1 1.24 mm to (144.4, 119.5)
- moved R5 1.02 mm to (163.1, 116.8)
- moved Q1 0.99 mm to (172.4, 99.0)
- moved D1 0.99 mm to (175.6, 98.4)
- moved R12 0.99 mm to (175.6, 102.1)
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Connections:
- J3 pad 2: /XBEE_RTS -> /XBEE_DTR
- J3 pad 3: /XBEE_DTR -> /XBEE_RTS
- SW2 pad 1: GND -> unconnected-(SW2-A-Pad1)
Routing:
- net +3V3: track 214.3 -> 45.8 mm
- net +5V: track 96.4 -> 1.92 mm
- net VCC: track 41.4 -> 14.9 mm, vias 0 -> 15
- net /XBEE_RTS: track 93.5 -> 71.6 mm
- net /XBEE_DTR: track 29.7 -> 16.9 mm
- net Net-(SW2-B): track 54.5 -> 66.9 mm
- net +1V1: track 30.3 -> 41.8 mm, vias 4 -> 3
- net GND: track 50.0 -> 39.1 mm, vias 98 -> 94
- net /XBEE_DIN: track 56.5 -> 48.4 mm
- net /GPS_SCL: track 39.4 -> 32.7 mm
- net /RP_SWD: track 13.8 -> 19.4 mm
- net /GPS_SDA: track 39.8 -> 34.6 mm
- net /XBEE_DOUT: track 59.7 -> 55.2 mm
- net /LVC_CUTOFF: track 57.9 -> 53.5 mm
- net +BATT: track 63.0 -> 66.4 mm, vias 1 -> 2
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- added copper zone on In2.Cu, net +3V3
- added copper zone on B.Cu, net /LVC_CUTOFF
- added copper zone on In1.Cu, net GND
- added copper zone on In2.Cu, net GND
- added copper zone on B.Cu, net Net-(C15-Pad2)
- added copper zone on B.Cu, net Net-(C16-Pad1)
- added copper zone on In2.Cu, net VCC
- removed copper zone on In1.Cu, net /LVC_CUTOFF
- removed copper zone on In1.Cu, net Net-(C15-Pad2)
- removed copper zone on In1.Cu, net Net-(C16-Pad1)
Other:
- outline, holes or cut-outs redrawn
- board text added: "BITSv5.0 Sept. '23"
- board text added: "J. Bishop, M. Shipman, & A. Takeuchi"

Commit message: no more 5 am commits
Routing:
- net Net-(AE1-A): track 3.10 -> 14.4 mm
- net Net-(U4-FB): track 13.3 -> 10.4 mm
