File: Boards/XBee Joint/XBee_Joint/XBee_Joint.kicad_pcb (KiCad board)
At the start: 4 copper layers, 67.4 x 98.5 mm, 64 parts, among them J1 Conn_01x07, J2 USB_C_Receptacle_USB2.0, Q1 Q_NMOS_GSD, SW2 SW_SPDT, SW3 SLIDE, U1 MCU_RaspberryPi_RP2040_RP2040, U2 XBee_SMT, U3 W25Q128JVS, U4 USBLC6-2SC6, U5 TPS63021DSJR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

Commit message: xbee joint board updates
Parts:
- removed R10: 1.05M, Resistor_SMD:R_0603_1608Metric_Pad0.98x0.95mm_HandSolder
- removed SW3: SLIDE, BITSv5:CL-SB-12B-01_NDC
- added R18: 510K, Resistor_SMD:R_0603_1608Metric_Pad0.98x0.95mm_HandSolder, F.Cu at (88.3, 113.9)
- BT1, U2: moved to F.Cu
- C1, C11, C5, C6, R1: moved to B.Cu
- C21: value 10nF -> 1uF
- R11: value 154K -> 1.05M
- R12: value 510K -> 154K
- R13: value 51.1K -> 46.4K
- R14, R16: value 23.7K -> 10K
- R15: value 5K -> 10K
- R17: value 5K -> 22K
- SW2: value SW_SPDT -> SLIDE; footprint BITSv5:CAS-120TB_NDC-M -> BITSv5:CL-SB-12B-01_NDC
- moved C16 109.9 mm to (116.6, 115.0), turned to -90 degrees
- moved R5 91.9 mm to (116.9, 98.4), turned to 90 degrees
- moved U3 90.8 mm to (114.5, 106.5), turned to -90 degrees
- moved R4 90.5 mm to (116.9, 94.1), turned to -90 degrees
- moved R11 88.8 mm to (83.7, 107.7)
- moved R8 88.6 mm to (99.6, 111.7), turned to 90 degrees
- moved R12 88.1 mm to (83.7, 109.5), turned to 180 degrees
- moved C17 87.5 mm to (114.3, 88.5), turned to -90 degrees
- moved R7 87.1 mm to (91.3, 111.7), turned to -90 degrees
- moved C22 86.1 mm to (88.6, 102.3), turned to -90 degrees
- moved C23 84.8 mm to (90.8, 102.3), turned to -90 degrees
- moved C1 84.8 mm to (108.6, 102.6), turned to -90 degrees
- moved C21 83.4 mm to (84.8, 98.6), turned to 180 degrees
- moved C19 82.0 mm to (87.6, 108.5), turned to 90 degrees
- moved C8 81.9 mm to (114.1, 94.9)
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Connections:
- C20 pad 1: VBUS -> +BATT
- C23 pad 1: +BATT -> VBUS
- R1 pad 2: Net-(SW2-B) -> Net-(U1-RUN)
- R11 pad 1: Net-(U6-IN+) -> VCC
- R11 pad 2: GND -> Net-(U6-IN+)
- R12 pad 1: VCC -> Net-(U6-IN+)
- R12 pad 2: Net-(SW3-C) -> GND
- R14 pad 1: VBUS -> +BATT
- R14 pad 2: Net-(U8-OV1) -> Net-(U8-PR1)
- R15 pad 1: Net-(U8-OV1) -> Net-(U8-PR1)
- R16 pad 1: +BATT -> VBUS
- R16 pad 2: Net-(U8-OV2) -> Net-(U8-CP2)
- R17 pad 1: Net-(U8-OV2) -> Net-(U8-CP2)
- R9 pad 1: +3V3 -> VCC
- SW2 pad 1: unconnected-(SW2-A-Pad1) -> GND
- SW2 pad 2: Net-(SW2-B) -> /LVC_CUTOFF
- SW2 pad 3: GND -> Net-(SW2-C)
- U1 pad 26: Net-(SW2-B) -> Net-(U1-RUN)
- U6 pad 1: Net-(SW3-C) -> Net-(SW2-C)
- U8 pad 2: +BATT -> VBUS
- U8 pad 3: GND -> Net-(U8-CP2)
- U8 pad 4: Net-(U8-OV2) -> GND
- U8 pad 5: Net-(U8-OV1) -> GND
- U8 pad 6: GND -> Net-(U8-PR1)
- U8 pad 7: VBUS -> +BATT
Routing:
- net GND: track 0.00 -> 78.6 mm, vias 0 -> 68
- net /XBEE_DOUT: track 0.00 -> 73.3 mm
- net /XBEE_DIN: track 0.00 -> 71.6 mm
- net /XBEE_RTS: track 0.00 -> 68.5 mm
- net /LVC_CUTOFF: track 0.00 -> 47.2 mm, vias 0 -> 2
- net /RP_SWD: track 0.00 -> 41.1 mm, vias 0 -> 1
- net +3V3: track 0.00 -> 33.1 mm, vias 0 -> 17
- net /RP_SWCLK: track 0.00 -> 32.5 mm, vias 0 -> 1
- net /XBEE_DTR: track 0.00 -> 28.2 mm
- net Net-(SW2-C): track 0.00 -> 27.2 mm
- net /LED: track 0.00 -> 21.4 mm, vias 0 -> 2
- net /QSPI_SS: track 0.00 -> 19.4 mm
- net /QSPI_SD3: track 0.00 -> 19.3 mm
- net /USB_D-: track 0.00 -> 18.3 mm
- net /USB_D+: track 0.00 -> 18.2 mm
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- added copper zone on F.Cu, net +3V3
- added copper zone on In2.Cu, net +3V3
- added copper zone on F.Cu, net +BATT
- added copper zone on In2.Cu, net +BATT
- added copper zone on F.Cu, net VBUS
- added copper zone on In2.Cu, net VBUS
- added copper zone on F.Cu, net VCC
- added copper zone on In2.Cu, net VCC
