File: Boards/XBee Joint/XBee_Joint/_autosave-XBee_Joint.kicad_pcb (KiCad board)
At the start: 4 copper layers, 67.4 x 98.5 mm, 63 parts, among them J1 Conn_01x07, J2 USB_C_Receptacle_USB2.0, Q1 Q_NMOS_GSD, SW2 SLIDE, U1 MCU_RaspberryPi_RP2040_RP2040, U2 XBee_SMT, U3 W25Q128JVS, U4 USBLC6-2SC6, U5 TPS63021DSJR, U6 LT6703CDC-3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

Commit message: xbee joint and bits updates
Changed lines of the file:
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@@
   (segment (start 83.1475 93.85) (end 83.1475 93.2025) (width 0.5) (layer "F.Cu") (net 11))
   (segment (start 84.8375 91.5125) (end 84.8375 91.18) (width 0.5) (layer "F.Cu") (net 11))
+  (segment (start 105.46 64.87) (end 93.85 64.87) (width 0.2) (layer "F.Cu") (net 12))
+  (segment (start 93.01 55.35) (end 92.2525 54.5925) (width 0.2) (layer "F.Cu") (net 12))
   (segment (start 106.99 68.055) (end 106.99 66.4) (width 0.2) (layer "F.Cu") (net 12))
-  (segment (start 93.52 64.54) (end 93.52 55.86) (width 0.2) (layer "F.Cu") (net 12))
-  (segment (start 93.85 64.87) (end 93.52 64.54) (width 0.2) (layer "F.Cu") (net 12))
+  (segment (start 93.85 64.87) (end 93.01 64.03) (width 0.2) (layer "F.Cu") (net 12))
+  (segment (start 106.99 66.4) (end 105.46 64.87) (width 0.2) (layer "F.Cu") (net 12))
   (segment (start 92.2525 54.5925) (end 90.46 54.5925) (width 0.2) (layer "F.Cu") (net 12))
-  (segment (start 93.52 55.86) (end 92.2525 54.5925) (width 0.2) (layer "F.Cu") (net 12))
-  (segment (start 106.99 66.4) (end 105.46 64.87) (width 0.2) (layer "F.Cu") (net 12))
-  (segment (start 105.46 64.87) (end 93.85 64.87) (width 0.2) (layer "F.Cu") (net 12))
+  (segment (start 93.01 64.03) (end 93.01 55.35) (width 0.2) (layer "F.Cu") (net 12))
   (segment (start 102.681041 95.65) (end 102.22 95.65) (width 0.2) (layer "F.Cu") (net 13))
   (segment (start 102.22 95.65) (end 101.72 95.15) (width 0.2) (layer "F.Cu") (net 13))
