File: Boards/XBee Joint/XBee_Joint/XBee_Joint.kicad_sch (KiCad schematic)
At the start: 64 parts, among them J2 USB_C_Receptacle_USB2.0, J3 Conn_01x07, Q1 Q_NMOS_GSD, SW2 SW_SPDT, SW3 SLIDE, U1 MCU_RaspberryPi_RP2040_RP2040, U10 USBLC6-2SC6, U2 W25Q128JVS, U5 TPS63021DSJR, U6 XBee_SMT, U7 TPS2121RUXR, U8 LT6703CDC-3, U9 TVS1800DRVR, Y1 12MHz

Commit message: xbee joint board updates
Parts:
- removed SW2: SW_SPDT, BITSv5:CAS-120TB_NDC-M, symbol Switch:SW_SPDT
- C33: value 10nF -> 1uF; symbol Device:C -> Device:C_Small
- C36: symbol Device:C -> Device:C_Small
- R15, R22: value 23.7K -> 10K
- R16: value 5K -> 10K
- R17: value 51.1K -> 46.4K
- R23: value 5K -> 22K
Connections:
- net +3V3: no longer R12.1
- net +BATT: now also C35.1, R15.1, U7.7 (IN1); no longer C34.1, R22.1, U7.2 (IN2)
- net GND: now also U7.4 (OV2), U7.5 (OV1); no longer U7.3 (CP2), U7.6 (PR1)
- net VBUS: now also C34.1, R22.1, U7.2 (IN2); no longer C35.1, R15.1, U7.7 (IN1)
- net VCC: now also R12.1
- net at R15.2, R16.1: now also U7.6 (PR1); no longer U7.5 (OV1)
- net at R22.2, R23.1: now also U7.3 (CP2); no longer U7.4 (OV2)
- no-connect marks 40 -> 48
Other:
- note removed: "LVC"
- moved on the sheet: C12, C13, C14, C24, C25, C26, C27, C28, C29, C33, C35, C36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

Commit message: xbee joint and bits updates
Parts:
- removed C24, C25, C34, C35: 10uF, Capacitor_SMD:C_0603_1608Metric_Pad1.08x0.95mm_HandSolder, symbol Device:C
- removed C26: 100nF, Capacitor_SMD:C_0603_1608Metric_Pad1.08x0.95mm_HandSolder, symbol Device:C
- removed C27, C28, C29: 22uF, Capacitor_SMD:C_0603_1608Metric_Pad1.08x0.95mm_HandSolder, symbol Device:C
- removed C33, C36: 1uF, Capacitor_SMD:C_0603_1608Metric_Pad1.08x0.95mm_HandSolder, symbol Device:C_Small
- removed C37: 1uF, Capacitor_SMD:C_0603_1608Metric_Pad1.08x0.95mm_HandSolder, symbol Device:C
- removed R15, R16, R22: 10K, Resistor_SMD:R_0603_1608Metric_Pad0.98x0.95mm_HandSolder, symbol Device:R_Small
- removed R17: 46.4K, Resistor_SMD:R_0603_1608Metric_Pad0.98x0.95mm_HandSolder, symbol Device:R
- removed R18: 1.05M, Resistor_SMD:R_0603_1608Metric_Pad0.98x0.95mm_HandSolder, symbol Device:R
- removed R19: 154K, Resistor_SMD:R_0603_1608Metric_Pad0.98x0.95mm_HandSolder, symbol Device:R
- removed R20: 510K, Resistor_SMD:R_0603_1608Metric_Pad0.98x0.95mm_HandSolder, symbol Device:R
- removed R23: 22K, Resistor_SMD:R_0603_1608Metric_Pad0.98x0.95mm_HandSolder, symbol Device:R_Small
- removed SW3: SLIDE, BITSv5:CL-SB-12B-01_NDC, symbol Switch:SW_SPDT
- removed U5: TPS63021DSJR, IC_TPS63021DSJR, symbol BITSv5:TPS63021DSJR
- removed U7: TPS2121RUXR, BITSv5:TPS2121, symbol TPS2121:TPS2121RUXR
- removed U8: LT6703CDC-3, BITSv5:DFN-3_DC_LIT, symbol LTC6703:LT6703CDC-3-TRPBF
- removed U9: TVS1800DRVR, BITSv5:TVS1800, symbol TVS1800:TVS1800DRVR
- added C19: C_Small, symbol Device:C_Small
- added U5: MAX25232ATCB/V+, 21-0664_TD12_2C_MXM, symbol BITSv5:MAX25232ATCB_V+
- L1: value 1.5uH -> L; footprint Inductor_SMD:L_Coilcraft_XxL4040 -> (none)
Connections:
- no-connect marks 48 -> 47
Other:
- note removed: "Power Mux"

Commit message: working on xbee joint
Parts:
- removed BT1: 1S1P LiPo, BITSv5:1042_KEY, symbol Device:Battery_Cell
- removed C19: C_Small, symbol Device:C_Small
- removed L1: L, symbol Device:L
- removed U5: MAX25232ATCB/V+, 21-0664_TD12_2C_MXM, symbol BITSv5:MAX25232ATCB_V+
- added U6: AP7361C-33E, Package_TO_SOT_SMD:SOT-223-3_TabPin2, symbol Regulator_Linear:AP7361C-33E
Connections:
- net +3V3: now also U6.3 (VO)
- net GND: now also U6.2 (GND)
- net VBUS: now also U6.1 (VI)
- net USB_D+ renamed D+
- net USB_D- renamed D-
- net XIN: no longer names the net of C13.2, U1.20 (XIN), Y1.3
- net XOUT: no longer names the net of R5.2, U1.21 (XOUT)
Other:
- note added: "Regulator"
- note removed: "3.3V Buck-Boost Regulator"
- note removed: "Crystal"
- note removed: "LED"
- note removed: "USB-C Port"
- moved on the sheet: C1, C10, C11, C12, C13, C14, C2, C26, C27, C28, C3, C32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

Commit message: xbee joint layout almost complete
Connections:
- net VCC is gone; now on net +3V3: R12.1
- net XIN: now reaches C13.2, U1.20 (XIN), Y1.3
- net XOUT: now reaches R5.2, U1.21 (XOUT)
Changed lines of the file:
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@@
+    (effects (font (size 1.27 1.27)) (justify left bottom))
+  )
+  (label "XOUT" (at 64.77 134.62 0) (fields_autoplaced)
     (effects (font (size 1.27 1.27)) (justify left bottom))
   )
@@
   )
   (label "QSPI_SD1" (at 342.9 194.31 0) (fields_autoplaced)
+    (effects (font (size 1.27 1.27)) (justify left bottom))
+  )
+  (label "XIN" (at 64.77 129.54 0) (fields_autoplaced)
     (effects (font (size 1.27 1.27)) (justify left bottom))
   )
@@
     )
   )
-  (symbol (lib_id "power:VCC") (at 190.5 135.89 0) (unit 1)
-    (in_bom yes) (on_board yes) (dnp no) (fields_autoplaced)
-    (property "Reference" "#PWR028" (at 190.5 139.7 0)
-      (effects (font (size 1.27 1.27)) hide)
-    )
-    (property "Value" "VCC" (at 190.5 132.08 0)
+  (symbol (lib_id "power:+3V3") (at 190.5 135.89 0) (unit 1)
+    (in_bom yes) (on_board yes) (dnp no)
+    (property "Reference" "#PWR02" (at 190.5 139.7 0)
+      (effects (font (size 1.27 1.27)) hide)
+    )
+    (property "Value" "+3V3" (at 190.5 132.08 0)
       (effects (font (size 1.27 1.27)))
     )
@@
       (project "XBee_Joint"
         (path "/8a7ed02c-ffe8-4f4c-89c1-18f4e0aa059d"
-          (reference "#PWR028") (unit 1)
-        )
-      )
+          (reference "#PWR02") (unit 1)
+        )
+      )

Commit message: updates
Parts:
- removed U6: AP7361C-33E, Package_TO_SOT_SMD:SOT-223-3_TabPin2, symbol Regulator_Linear:AP7361C-33E
- added R10: 166k, Resistor_SMD:R_0603_1608Metric_Pad0.98x0.95mm_HandSolder, symbol Device:R_Small
- added R11: 100k, Resistor_SMD:R_0603_1608Metric_Pad0.98x0.95mm_HandSolder, symbol Device:R_Small
- added R12: 330, Resistor_SMD:R_1210_3225Metric_Pad1.30x2.65mm_HandSolder, symbol Device:R_Small
- added U7: MIC29302WU, Package_TO_SOT_SMD:TO-263-5_TabPin3, symbol Regulator_Linear:MIC29302WU
Connections:
- net +3V3: now also R10.1, R12.1, U7.4 (VOUT)
- net GND: now also R11.2, R12.2, U7.3 (GND)
- net VBUS: now also U7.1 (EN), U7.2 (VIN)
- net XBEE_DIN: no longer U6.4 (DIO14/DIN/~{CONFIG})
- net XBEE_DOUT: no longer U6.3 (DIO13/DOUT)
- net XBEE_DTR: no longer U6.10 (DIO8/~{DTR~{/SLEEP_RQ})
- net XBEE_RTS: no longer U6.29 (DIO6/~{RTS})
- new net: R10.2, R11.1, U7.5 (ADJ)
- new net XBEE_PRO_DIN: U6.4 (DIO14/DIN/~{CONFIG})
- new net XBEE_PRO_DOUT: U6.3 (DIO13/DOUT)
- new net XBEE_PRO_DTR: U6.10 (DIO8/~{DTR~{/SLEEP_RQ})
- new net XBEE_PRO_RTS: U6.29 (DIO6/~{RTS})
Other:
- note added: "Pre-load for minimum load current requirement"
- title: (none) -> Xbee Joint
- moved on the sheet: C26, C27, D1, J2, Q1, R12, R7, R8, U10

Commit message: dorji joint?
Parts:
- removed C1, C2: 1uF, Capacitor_SMD:C_0402_1005Metric_Pad0.74x0.62mm_HandSolder, symbol Device:C
- removed C10, C11, C3, C32, C4, C5, C6, C7, C8, C9: 100nF, Capacitor_SMD:C_0402_1005Metric_Pad0.74x0.62mm_HandSolder, symbol Device:C
- removed C12: 100nF, Capacitor_SMD:C_0603_1608Metric_Pad1.08x0.95mm_HandSolder, symbol Device:C
- removed C13, C14: 10pF, Capacitor_SMD:C_0603_1608Metric_Pad1.08x0.95mm_HandSolder, symbol Device:C
- removed C26: 100pF, Capacitor_SMD:C_0603_1608Metric_Pad1.08x0.95mm_HandSolder, symbol Device:C
- removed C27: 1uF, Capacitor_SMD:C_0603_1608Metric_Pad1.08x0.95mm_HandSolder, symbol Device:C
- removed C28: 10uF, Capacitor_SMD:C_0603_1608Metric_Pad1.08x0.95mm_HandSolder, symbol Device:C
- removed J3: Conn_01x07, Connector_PinSocket_2.54mm:PinSocket_1x07_P2.54mm_Vertical, symbol Connector_Generic:Conn_01x07
- removed Q1: Q_NMOS_GSD, Package_TO_SOT_SMD:SOT-23-3, symbol Device:Q_NMOS_GSD
- removed R1, R2: 27Ω, Resistor_SMD:R_0402_1005Metric_Pad0.72x0.64mm_HandSolder, symbol Device:R
- removed R10: 166k, Resistor_SMD:R_0603_1608Metric_Pad0.98x0.95mm_HandSolder, symbol Device:R_Small
- removed R11: 100k, Resistor_SMD:R_0603_1608Metric_Pad0.98x0.95mm_HandSolder, symbol Device:R_Small
- removed R11, R3: 10K, Resistor_SMD:R_0603_1608Metric_Pad0.98x0.95mm_HandSolder, symbol Device:R
- removed R12: 470, Resistor_SMD:R_0603_1608Metric_Pad0.98x0.95mm_HandSolder, symbol Device:R
- removed R4: 1K, Resistor_SMD:R_0603_1608Metric_Pad0.98x0.95mm_HandSolder, symbol Device:R
- removed R5: 1K, Resistor_SMD:R_0402_1005Metric_Pad0.72x0.64mm_HandSolder, symbol Device:R
- removed R7, R8: 5.1K, Resistor_SMD:R_0603_1608Metric_Pad0.98x0.95mm_HandSolder, symbol Device:R
- removed U1: MCU_RaspberryPi_RP2040_RP2040, BITSv5:RP2040-QFN-56, symbol RP2040_minimal-cache:MCU_RaspberryPi_RP2040_RP2040
- removed U10: USBLC6-2SC6, BITSv5:SOT23-6L_STM-M, symbol USBLC6-2SC6:USBLC6-2SC6
- removed U6: XBee_SMT, BITSv5:XCVR_XBP9X-DMUS-001, symbol BITSv5:XBP9X-DMUS-001
- removed U7: MIC29302WU, Package_TO_SOT_SMD:TO-263-5_TabPin3, symbol Regulator_Linear:MIC29302WU
- removed Y1: 12MHz, Crystal:Crystal_SMD_2520-4Pin_2.5x2.0mm, symbol Device:Crystal_GND24
- added AE2: Antenna, Connector_Coaxial:SMA_Molex_73251-1153_EdgeMount_Horizontal, symbol Device:Antenna
- added C1, C2: 1uF, Capacitor_SMD:C_0402_1005Metric, symbol Device:C_Small
- added C10, C11, C12, C3, C32, C4, C5, C6, C7, C8, C9: 100nF, Capacitor_SMD:C_0402_1005Metric, symbol Device:C_Small
- added C13, C14: 10pF, Capacitor_SMD:C_0402_1005Metric, symbol Device:C_Small
- added C26: 1uF, Capacitor_SMD:C_0603_1608Metric, symbol Device:C_Small
- added C26: 10uF, Capacitor_SMD:C_0603_1608Metric, symbol Device:C_Small
- added C27: 100nF, Capacitor_SMD:C_0603_1608Metric, symbol Device:C_Small
- added H1, H2: M2, MountingHole:MountingHole_2.2mm_M2_Pad, symbol Mechanical:MountingHole
- added J3: SOICbite, BITSv5:SOIC_clipProgSmall, symbol Connector:Conn_01x08_Socket
- added R1, R2: 27, Resistor_SMD:R_0402_1005Metric, symbol Device:R_Small
- added R3: DNF, Resistor_SMD:R_0603_1608Metric, symbol Device:R_Small
- added R4: 10K, Resistor_SMD:R_0603_1608Metric, symbol Device:R_Small
- added R4: 1K, Resistor_SMD:R_0603_1608Metric, symbol Device:R_Small
- added R5: 1K, Capacitor_SMD:C_0402_1005Metric, symbol Device:R_Small
- added R7, R8: 5.1K, Resistor_SMD:R_0603_1608Metric_Pad0.98x0.95mm_HandSolder, symbol Device:R_Small
- added U1: MCU_RaspberryPi_RP2040_RP2040, BITSv5:RP2040-QFN-56, symbol BITSv5:MCU_RaspberryPi_RP2040
- added U10: USBLC6-2SC6, SOT23-6L_STM, symbol BITSv5:USBLC6-2SC6
- added U2: AP2114H-3.3TRG1, Package_TO_SOT_SMD:SOT-223-3_TabPin2, symbol Regulator_Linear:AP1117-33
- added U4: DRF1262TL, BITSv5:DRF1262TL, symbol BITSv5:DRF1262TL
- added Y1: 12MHz, Crystal:Crystal_SMD_2520-4Pin_2.5x2.0mm, symbol Device:Crystal_GND24_Small
- J2: footprint Connector_USB:USB_C_Receptacle_GCT_USB4085 -> Connector_USB:USB_C_Receptacle_GCT_USB4105-xx-A_16P_TopMnt_Horizontal
- R12: value 330 -> 470; footprint Resistor_SMD:R_1210_3225Metric_Pad1.30x2.65mm_HandSolder -> Resistor_SMD:R_0603_1608Metric
- U2: footprint Package_SO:SOIC-8_5.23x5.23mm_P1.27mm -> BITSv5:WSON_128JVPIQ_WIN
Connections:
- net +1V1: now also C1.1, C3.1, C4.1, U1.23 (DVDD), U1.45 (VREG_VOUT), U1.50 (DVDD)
- net +3V3: now also C10.1, C11.1, C12.1, C2.1, C32.1, C5.1, C6.1, C7.1, C8.1, C9.1, R3.2, R4.1, U1.1 (IOVDD), U1.10 (IOVDD), U1.22 (IOVDD), U1.33 (IOVDD), U1.42 (IOVDD), U1.43 (ADC_AVDD), U1.44 (VREG_IN), U1.48 (USB_VDD), U1.49 (IOVDD), U2.2 (VO)
- net GND: now also D1.1 (K), C1.2, C10.2, C11.2, C12.2, C13.2, C14.2, C2.2, C26.2, C26.2, C27.2, C3.2, C32.2, C4.2, C5.2, C6.2, C7.2, C8.2, C9.2, J3.8 (Pin_8), R7.1, R8.2, U1.19 (TESTEN), U1.57 (GND), U10.2, U2.1 (GND), U4.15 (GND), U4.17 (GND), U4.2 (GND), U4.4 (GND), U4.5 (GND), Y1.2, Y1.4; no longer R12.2
- net QSPI_SCLK: now also U1.52 (QSPI_SCLK)
- net QSPI_SD0: now also U1.53 (QSPI_SD0)
- net QSPI_SD1: now also U1.55 (QSPI_SD1)
- net QSPI_SD2: now also U1.54 (QSPI_SD2)
- net QSPI_SD3: now also U1.51 (QSPI_SD3)
- net QSPI_SS: now also R3.1, R4.2, U1.56 (QSPI_SS)
- net RP_SWCLK: now also J3.1 (Pin_1), U1.24 (SWCLK)
- net RP_SWD: now also J3.2 (Pin_2), U1.25 (SWD)
- net VBUS: now also C26.1, C26.1, C27.1, U10.5, U2.3 (VI), U4.6 (VDD), U4.7 (VDD)
- net at D1.2 (A): now also R12.2
- net at J2.A5 (CC1): now also R7.2
- net at J2.A6 (D+), J2.B6 (D+): now also U10.6
- net at J2.A7 (D-), J2.B7 (D-): now also U10.4
- net at J2.B5 (CC2): now also R8.1
- net at SW2.2 (B): now also R4.1
- new net: AE2.1 (A), U4.16 (ANT)
- new net: R4.2, U1.26 (RUN)
- new net: C14.1, R5.1, Y1.1
- new net: C13.1, U1.20 (XIN), Y1.3
- new net: R2.2, U1.47 (USB_DP)
- new net: R5.2, U1.21 (XOUT)
- new net: R1.2, U1.46 (USB_DM)
- new net DRF_BUSY: U1.8 (GPIO6), U4.9 (BUSY)
- new net DRF_CLK: U1.29 (GPIO18), U4.13 (SCK)
- new net DRF_CS: U1.32 (GPIO21), U4.14 (NSS)
- new net DRF_DIO1: U1.5 (GPIO3), U4.8 (DIO1)
- new net DRF_MISO: U1.31 (GPIO20), U4.11 (MISO)
- new net DRF_MOSI: U1.30 (GPIO19), U4.12 (MOSI)
- new net DRF_SW: U1.12 (GPIO9), U4.1 (SW)
- new net DRF_TXEN: U1.3 (GPIO1), U4.3 (TXEN)
- new net USB_D+: R2.1, U10.1
- new net USB_D-: R1.1, U10.3
- no-connect marks 47 -> 30
Other:
- note added: "LED"
- note added: "MCU"
- note added: "Radio"
- note added: "SOICbite"
- note removed: "Debug Headers"
- note removed: "Pre-load for minimum load current requirement"
- note removed: "Regulator"
- note removed: "XBee Pro SX 900"
